File: hardware/colibri-v2/mems.sch (KiCad schematic (older format))
At the start: 9 parts, among them U2 L3GD20, U3 LSM303D

Commit message: Re-annotated schematic
Parts:
- renumbered C35 to C33, C36 to C34, C37 to C35, C38 to C36, C39 to C37, C40 to C38, C41 to C39
Changed lines of the file:
@@
 $EndComp
 $Comp
-L C C36
+L C C34
 U 1 1 55865EFE
 P 6100 3450
-F 0 "C36" H 6125 3550 50  0000 L CNN
+F 0 "C34" H 6125 3550 50  0000 L CNN
 F 1 "10nF/25V" H 6125 3350 50  0000 L CNN
 F 2 "" H 6138 3300 30  0000 C CNN
@@
 $EndComp
 $Comp
-L C C38
+L C C36
 U 1 1 55865F5E
 P 6750 3200
-F 0 "C38" H 6775 3300 50  0000 L CNN
+F 0 "C36" H 6775 3300 50  0000 L CNN
 F 1 "10nF" H 6775 3100 50  0000 L CNN
 F 2 "" H 6788 3050 30  0000 C CNN
@@
 $EndComp
 $Comp
-L C C40
+L C C38
 U 1 1 55865F9A
 P 7350 3200
-F 0 "C40" H 7375 3300 50  0000 L CNN
+F 0 "C38" H 7375 3300 50  0000 L CNN
 F 1 "10uF" H 7375 3100 50  0000 L CNN
 F 2 "" H 7388 3050 30  0000 C CNN
@@
 $EndComp
 $Comp
-L GND #PWR037
+L GND #PWR36
 U 1 1 55865FDB
 P 6750 3950
-F 0 "#PWR037" H 6750 3700 50  0001 C CNN
+F 0 "#PWR36" H 6750 3700 50  0001 C CNN
 F 1 "GND" H 6750 3800 50  0000 C CNN
 F 2 "" H 6750 3950 60  0000 C CNN
@@
 $EndComp
 $Comp
-L GND #PWR038
+L GND #PWR34
 U 1 1 558661BB
 P 3950 3950
-F 0 "#PWR038" H 3950 3700 50  0001 C CNN
+F 0 "#PWR34" H 3950 3700 50  0001 C CNN
 F 1 "GND" H 3950 3800 50  0000 C CNN
 F 2 "" H 3950 3950 60  0000 C CNN
@@
 MEMS_ACC_INT1
 $Comp
-L GND #PWR039
+L GND #PWR37
 U 1 1 5587241A
 P 6750 5950
-F 0 "#PWR039" H 6750 5700 50  0001 C CNN
+F 0 "#PWR37" H 6750 5700 50  0001 C CNN
 F 1 "GND" H 6750 5800 50  0000 C CNN
 F 2 "" H 6750 5950 60  0000 C CNN
@@
 $EndComp
 $Comp
-L C C37
+L C C35
 U 1 1 55872576
 P 6100 5350
-F 0 "C37" H 5950 5250 50  0000 L CNN
+F 0 "C35" H 5950 5250 50  0000 L CNN
 F 1 "4.7uF" H 5850 5450 50  0000 L CNN
 F 2 "" H 6138 5200 30  0000 C CNN
@@
 $EndComp
 $Comp
-L C C39
+L C C37
 U 1 1 55873CA6
 P 6750 5150
-F 0 "C39" H 6775 5250 50  0000 L CNN
+F 0 "C37" H 6775 5250 50  0000 L CNN
 F 1 "10nF" H 6775 5050 50  0000 L CNN
 F 2 "" H 6788 5000 30  0000 C CNN
@@
 $EndComp
 $Comp
-L C C41
+L C C39
 U 1 1 55873CAC
 P 7350 5150
-F 0 "C41" H 7375 5250 50  0000 L CNN
+F 0 "C39" H 7375 5250 50  0000 L CNN
 F 1 "10uF" H 7375 5050 50  0000 L CNN
 F 2 "" H 7388 5000 30  0000 C CNN
@@
 MEMS_ACC_NCS
 $Comp
-L C C35
+L C C33
 U 1 1 55878EB4
 P 3700 5500
-F 0 "C35" V 3750 5350 50  0000 L CNN
+F 0 "C33" V 3750 5350 50  0000 L CNN
 F 1 "0.22uF" V 3750 5600 50  0000 L CNN
 F 2 "" H 3738 5350 30  0000 C CNN
@@
 $EndComp
 Wire Wire Line
-	5500 3700 5650 3700
-Wire Wire Line
-	5650 3700 6100 3700
-Wire Wire Line
-	6100 3700 6750 3700
-Wire Wire Line
-	6750 3700 7350 3700
+	5500 3700 7350 3700
 Wire Wire Line
 	7350 3700 7350 3350
 Wire Wire Line
-	6750 3350 6750 3700
-Wire Wire Line
-	6750 3700 6750 3950
+	6750 3350 6750 3950
 Connection ~ 6750 3700
 Wire Wire Line
@@
 	5500 3300 5650 3300
 Wire Wire Line
-	5650 3300 5650 3400
-Wire Wire Line
-	5650 3400 5650 3500
-Wire Wire Line
-	5650 3500 5650 3600
-Wire Wire Line
-	5650 3600 5650 3700
+	5650 3300 5650 3700
 Connection ~ 5650 3700
 Wire Wire Line
@@
 	5500 3000 5650 3000
 Wire Wire Line
-	5650 2700 5650 3000
-Wire Wire Line
-	5650 3000 5650 3100
-Wire Wire Line
-	5650 2700 6750 2700
-Wire Wire Line
-	6750 2700 7350 2700
-Wire Wire Line
-	7350 2700 8250 2700
+	5650 2700 5650 3100
+Wire Wire Line
+	5650 2700 8250 2700
 Wire Wire Line
 	5650 3100 5500 3100
@@
 	3950 3700 4100 3700
 Wire Wire Line
-	1500 3100 3050 3100
-Wire Wire Line
-	3050 3100 4100 3100
-Wire Wire Line
-	1500 3200 2950 3200
-Wire Wire Line
-	2950 3200 4100 3200
-Wire Wire Line
-	1500 3300 2850 3300
-Wire Wire Line
-	2850 3300 4100 3300
+	1500 3100 4100 3100
+Wire Wire Line
+	1500 3200 4100 3200
+Wire Wire Line
+	1500 3300 4100 3300
 Wire Wire Line
 	1500 3400 4100 3400
@@
 Connection ~ 5650 5500
 Wire Wire Line
-	5500 5600 5650 5600
-Wire Wire Line
-	5650 5600 6100 5600
-Wire Wire Line
-	6100 5600 6750 5600
-Wire Wire Line
-	6750 5600 7350 5600
+	5500 5600 7350 5600
 Connection ~ 5650 5600
 Wire Wire Line
@@
 Connection ~ 6100 5600
 Wire Wire Line
-	6750 5300 6750 5600
-Wire Wire Line
-	6750 5600 6750 5950
+	6750 5300 6750 5950
 Connection ~ 6750 5600
 Wire Wire Line
 	6100 4600 6100 5000
 Wire Wire Line
-	5650 5200 5650 5300
-Wire Wire Line
-	5650 5300 5650 5400
-Wire Wire Line
-	5650 5400 5650 5500
-Wire Wire Line
-	5650 5500 5650 5600
-Wire Wire Line
-	8250 4600 7350 4600
-Wire Wire Line
-	7350 4600 6750 4600
-Wire Wire Line
-	6750 4600 6100 4600
+	5650 5200 5650 5600
+Wire Wire Line
+	8250 4600 6100 4600
 Wire Wire Line
 	7350 4600 7350 5000
@@
 Connection ~ 6750 2700
 Wire Wire Line
-	8250 2300 8250 2700
-Wire Wire Line
-	8250 2700 8250 4600
+	8250 2300 8250 4600
 Connection ~ 7350 2700
 Connection ~ 7350 4600
@@
 V_SENS1
 Wire Wire Line
-	1500 2300 1950 2300
-Wire Wire Line
-	1950 2300 8250 2300
-$Comp
-L PWR_FLAG #FLG040
+	1500 2300 8250 2300
+$Comp
+L PWR_FLAG #FLG1
 U 1 1 55FF3EA5
 P 1950 2100
-F 0 "#FLG040" H 1950 2195 50  0001 C CNN
+F 0 "#FLG1" H 1950 2195 50  0001 C CNN
 F 1 "PWR_FLAG" H 1950 2280 50  0000 C CNN
 F 2 "" H 1950 2100 60  0000 C CNN
@@
 Connection ~ 1950 2300
 $Comp
-L +3V3 #PWR041
+L +3V3 #PWR35
 U 1 1 5622ED95
 P 5800 4550
-F 0 "#PWR041" H 5800 4400 50  0001 C CNN
+F 0 "#PWR35" H 5800 4400 50  0001 C CNN
 F 1 "+3V3" H 5800 4690 50  0000 C CNN
 F 2 "" H 5800 4550 60  0000 C CNN
@@
 	5800 4900 5800 4550
 $Comp
-L +3V3 #PWR042
+L +3V3 #PWR33
 U 1 1 5622EE37
 P 3950 2700
-F 0 "#PWR042" H 3950 2550 50  0001 C CNN
+F 0 "#PWR33" H 3950 2550 50  0001 C CNN
 F 1 "+3V3" H 3950 2840 50  0000 C CNN
 F 2 "" H 3950 2700 60  0000 C CNN

Commit message: Associated footprints for R and some of the C
Parts:
- C33, C34, C35: footprint (none) -> Capacitors_SMD:C_0603
- C36, C37, C38, C39: footprint (none) -> Capacitors_SMD:C_0805
Changed lines of the file:
@@
 F 0 "U2" H 5200 3850 60  0000 C CNN
 F 1 "L3GD20" H 4500 2850 60  0000 C CNN
-F 2 "" H 4800 3500 60  0000 C CNN
+F 2 "" H 4800 3500 60  0001 C CNN
 F 3 "" H 4800 3500 60  0000 C CNN
 	1    4800 3350
@@
 F 0 "C34" H 6125 3550 50  0000 L CNN
 F 1 "10nF/25V" H 6125 3350 50  0000 L CNN
-F 2 "" H 6138 3300 30  0000 C CNN
+F 2 "Capacitors_SMD:C_0603" H 6138 3300 30  0001 C CNN
 F 3 "" H 6100 3450 60  0000 C CNN
 	1    6100 3450
@@
 F 0 "C36" H 6775 3300 50  0000 L CNN
 F 1 "10nF" H 6775 3100 50  0000 L CNN
-F 2 "" H 6788 3050 30  0000 C CNN
+F 2 "Capacitors_SMD:C_0805" H 6788 3050 30  0001 C CNN
 F 3 "" H 6750 3200 60  0000 C CNN
 	1    6750 3200
@@
 F 0 "C38" H 7375 3300 50  0000 L CNN
 F 1 "10uF" H 7375 3100 50  0000 L CNN
-F 2 "" H 7388 3050 30  0000 C CNN
+F 2 "Capacitors_SMD:C_0805" H 7388 3050 30  0001 C CNN
 F 3 "" H 7350 3200 60  0000 C CNN
 	1    7350 3200
@@
 $EndComp
 $Comp
-L GND #PWR36
+L GND #PWR033
 U 1 1 55865FDB
 P 6750 3950
-F 0 "#PWR36" H 6750 3700 50  0001 C CNN
+F 0 "#PWR033" H 6750 3700 50  0001 C CNN
 F 1 "GND" H 6750 3800 50  0000 C CNN
 F 2 "" H 6750 3950 60  0000 C CNN
@@
 $EndComp
 $Comp
-L GND #PWR34
+L GND #PWR034
 U 1 1 558661BB
 P 3950 3950
-F 0 "#PWR34" H 3950 3700 50  0001 C CNN
+F 0 "#PWR034" H 3950 3700 50  0001 C CNN
 F 1 "GND" H 3950 3800 50  0000 C CNN
 F 2 "" H 3950 3950 60  0000 C CNN
@@
 F 0 "U3" H 5200 5750 60  0000 C CNN
 F 1 "LSM303D" H 4550 4750 60  0000 C CNN
-F 2 "" H 4800 5400 60  0000 C CNN
+F 2 "" H 4800 5400 60  0001 C CNN
 F 3 "" H 4800 5400 60  0000 C CNN
 	1    4800 5250
@@
 MEMS_ACC_INT1
 $Comp
-L GND #PWR37
+L GND #PWR035
 U 1 1 5587241A
 P 6750 5950
-F 0 "#PWR37" H 6750 5700 50  0001 C CNN
+F 0 "#PWR035" H 6750 5700 50  0001 C CNN
 F 1 "GND" H 6750 5800 50  0000 C CNN
 F 2 "" H 6750 5950 60  0000 C CNN
@@
 F 0 "C35" H 5950 5250 50  0000 L CNN
 F 1 "4.7uF" H 5850 5450 50  0000 L CNN
-F 2 "" H 6138 5200 30  0000 C CNN
+F 2 "Capacitors_SMD:C_0603" H 6138 5200 30  0001 C CNN
 F 3 "" H 6100 5350 60  0000 C CNN
 	1    6100 5350
@@
 F 0 "C37" H 6775 5250 50  0000 L CNN
 F 1 "10nF" H 6775 5050 50  0000 L CNN
-F 2 "" H 6788 5000 30  0000 C CNN
+F 2 "Capacitors_SMD:C_0805" H 6788 5000 30  0001 C CNN
 F 3 "" H 6750 5150 60  0000 C CNN
 	1    6750 5150
@@
 F 0 "C39" H 7375 5250 50  0000 L CNN
 F 1 "10uF" H 7375 5050 50  0000 L CNN
-F 2 "" H 7388 5000 30  0000 C CNN
+F 2 "Capacitors_SMD:C_0805" H 7388 5000 30  0001 C CNN
 F 3 "" H 7350 5150 60  0000 C CNN
 	1    7350 5150
@@
 F 0 "C33" V 3750 5350 50  0000 L CNN
 F 1 "0.22uF" V 3750 5600 50  0000 L CNN
-F 2 "" H 3738 5350 30  0000 C CNN
+F 2 "Capacitors_SMD:C_0603" H 3738 5350 30  0001 C CNN
 F 3 "" H 3700 5500 60  0000 C CNN
 	1    3700 5500
@@
 	1500 2300 8250 2300
 $Comp
-L PWR_FLAG #FLG1
+L PWR_FLAG #FLG036
 U 1 1 55FF3EA5
 P 1950 2100
-F 0 "#FLG1" H 1950 2195 50  0001 C CNN
+F 0 "#FLG036" H 1950 2195 50  0001 C CNN
 F 1 "PWR_FLAG" H 1950 2280 50  0000 C CNN
 F 2 "" H 1950 2100 60  0000 C CNN
@@
 Connection ~ 1950 2300
 $Comp
-L +3V3 #PWR35
+L +3V3 #PWR037
 U 1 1 5622ED95
 P 5800 4550
-F 0 "#PWR35" H 5800 4400 50  0001 C CNN
+F 0 "#PWR037" H 5800 4400 50  0001 C CNN
 F 1 "+3V3" H 5800 4690 50  0000 C CNN
 F 2 "" H 5800 4550 60  0000 C CNN
@@
 	5800 4900 5800 4550
 $Comp
-L +3V3 #PWR33
+L +3V3 #PWR038
 U 1 1 5622EE37
 P 3950 2700
-F 0 "#PWR33" H 3950 2550 50  0001 C CNN
+F 0 "#PWR038" H 3950 2550 50  0001 C CNN
 F 1 "+3V3" H 3950 2840 50  0000 C CNN
 F 2 "" H 3950 2700 60  0000 C CNN
