File: hardware/colibri-v2/receiver_pwm_input.sch (KiCad schematic (older format))
At the start: 11 parts, among them P18 CONN_01X03, P19 CONN_01X03, P20 CONN_01X03, P21 CONN_01X03, P22 CONN_01X03, U19 SN74LVC162244A

Commit message: Associated footprints for R and some of the C
Parts:
- R136, R137, R138, R139, R140: footprint (none) -> Resistors_SMD:R_0603
Changed lines of the file:
@@
 F 0 "P18" H 7250 1750 50  0000 C CNN
 F 1 "CONN_01X03" V 7350 1550 50  0000 C CNN
-F 2 "" H 7250 1550 60  0000 C CNN
+F 2 "" H 7250 1550 60  0001 C CNN
 F 3 "" H 7250 1550 60  0000 C CNN
 	1    7250 1550
@@
 $EndComp
 $Comp
-L +5V #PWR183
+L +5V #PWR0182
 U 1 1 5624B1E0
 P 6900 1350
-F 0 "#PWR183" H 6900 1200 50  0001 C CNN
+F 0 "#PWR0182" H 6900 1200 50  0001 C CNN
 F 1 "+5V" H 6900 1490 50  0000 C CNN
 F 2 "" H 6900 1350 60  0000 C CNN
@@
 $EndComp
 $Comp
-L GND #PWR184
+L GND #PWR0183
 U 1 1 5624B1E6
 P 6900 1750
-F 0 "#PWR184" H 6900 1500 50  0001 C CNN
+F 0 "#PWR0183" H 6900 1500 50  0001 C CNN
 F 1 "GND" H 6900 1600 50  0000 C CNN
 F 2 "" H 6900 1750 60  0000 C CNN
@@
 F 0 "R136" V 6580 1450 50  0000 C CNN
 F 1 "100" V 6500 1450 50  0000 C CNN
-F 2 "" V 6430 1450 30  0000 C CNN
+F 2 "Resistors_SMD:R_0603" V 6430 1450 30  0001 C CNN
 F 3 "" H 6500 1450 30  0000 C CNN
 	1    6500 1450
@@
 F 0 "P19" H 7250 2650 50  0000 C CNN
 F 1 "CONN_01X03" V 7350 2450 50  0000 C CNN
-F 2 "" H 7250 2450 60  0000 C CNN
+F 2 "" H 7250 2450 60  0001 C CNN
 F 3 "" H 7250 2450 60  0000 C CNN
 	1    7250 2450
@@
 $EndComp
 $Comp
-L +5V #PWR185
+L +5V #PWR0184
 U 1 1 5624B200
 P 6900 2250
-F 0 "#PWR185" H 6900 2100 50  0001 C CNN
+F 0 "#PWR0184" H 6900 2100 50  0001 C CNN
 F 1 "+5V" H 6900 2390 50  0000 C CNN
 F 2 "" H 6900 2250 60  0000 C CNN
@@
 $EndComp
 $Comp
-L GND #PWR186
+L GND #PWR0185
 U 1 1 5624B206
 P 6900 2650
-F 0 "#PWR186" H 6900 2400 50  0001 C CNN
+F 0 "#PWR0185" H 6900 2400 50  0001 C CNN
 F 1 "GND" H 6900 2500 50  0000 C CNN
 F 2 "" H 6900 2650 60  0000 C CNN
@@
 F 0 "R137" V 6580 2350 50  0000 C CNN
 F 1 "100" V 6500 2350 50  0000 C CNN
-F 2 "" V 6430 2350 30  0000 C CNN
+F 2 "Resistors_SMD:R_0603" V 6430 2350 30  0001 C CNN
 F 3 "" H 6500 2350 30  0000 C CNN
 	1    6500 2350
@@
 F 0 "P20" H 7250 3550 50  0000 C CNN
 F 1 "CONN_01X03" V 7350 3350 50  0000 C CNN
-F 2 "" H 7250 3350 60  0000 C CNN
+F 2 "" H 7250 3350 60  0001 C CNN
 F 3 "" H 7250 3350 60  0000 C CNN
 	1    7250 3350
@@
 $EndComp
 $Comp
-L +5V #PWR187
+L +5V #PWR0186
 U 1 1 5624B220
 P 6900 3150
-F 0 "#PWR187" H 6900 3000 50  0001 C CNN
+F 0 "#PWR0186" H 6900 3000 50  0001 C CNN
 F 1 "+5V" H 6900 3290 50  0000 C CNN
 F 2 "" H 6900 3150 60  0000 C CNN
@@
 $EndComp
 $Comp
-L GND #PWR188
+L GND #PWR0187
 U 1 1 5624B226
 P 6900 3550
-F 0 "#PWR188" H 6900 3300 50  0001 C CNN
+F 0 "#PWR0187" H 6900 3300 50  0001 C CNN
 F 1 "GND" H 6900 3400 50  0000 C CNN
 F 2 "" H 6900 3550 60  0000 C CNN
@@
 F 0 "R138" V 6580 3250 50  0000 C CNN
 F 1 "100" V 6500 3250 50  0000 C CNN
-F 2 "" V 6430 3250 30  0000 C CNN
+F 2 "Resistors_SMD:R_0603" V 6430 3250 30  0001 C CNN
 F 3 "" H 6500 3250 30  0000 C CNN
 	1    6500 3250
@@
 F 0 "P21" H 7250 4450 50  0000 C CNN
 F 1 "CONN_01X03" V 7350 4250 50  0000 C CNN
-F 2 "" H 7250 4250 60  0000 C CNN
+F 2 "" H 7250 4250 60  0001 C CNN
 F 3 "" H 7250 4250 60  0000 C CNN
 	1    7250 4250
@@
 $EndComp
 $Comp
-L +5V #PWR189
+L +5V #PWR0188
 U 1 1 5624B240
 P 6900 4050
-F 0 "#PWR189" H 6900 3900 50  0001 C CNN
+F 0 "#PWR0188" H 6900 3900 50  0001 C CNN
 F 1 "+5V" H 6900 4190 50  0000 C CNN
 F 2 "" H 6900 4050 60  0000 C CNN
@@
 $EndComp
 $Comp
-L GND #PWR190
+L GND #PWR0189
 U 1 1 5624B246
 P 6900 4450
-F 0 "#PWR190" H 6900 4200 50  0001 C CNN
+F 0 "#PWR0189" H 6900 4200 50  0001 C CNN
 F 1 "GND" H 6900 4300 50  0000 C CNN
 F 2 "" H 6900 4450 60  0000 C CNN
@@
 F 0 "R139" V 6580 4150 50  0000 C CNN
 F 1 "100" V 6500 4150 50  0000 C CNN
-F 2 "" V 6430 4150 30  0000 C CNN
+F 2 "Resistors_SMD:R_0603" V 6430 4150 30  0001 C CNN
 F 3 "" H 6500 4150 30  0000 C CNN
 	1    6500 4150
@@
 F 0 "U19" H 5150 3600 60  0000 C CNN
 F 1 "SN74LVC162244A" H 4950 2500 60  0000 C CNN
-F 2 "" H 4950 2900 60  0000 C CNN
+F 2 "" H 4950 2900 60  0001 C CNN
 F 3 "" H 4950 2900 60  0000 C CNN
 	4    4950 3050
@@
 F 0 "P22" H 7250 5500 50  0000 C CNN
 F 1 "CONN_01X03" V 7350 5300 50  0000 C CNN
-F 2 "" H 7250 5300 60  0000 C CNN
+F 2 "" H 7250 5300 60  0001 C CNN
 F 3 "" H 7250 5300 60  0000 C CNN
 	1    7250 5300
@@
 $EndComp
 $Comp
-L +5V #PWR191
+L +5V #PWR0190
 U 1 1 5624BF5C
 P 6900 5100
-F 0 "#PWR191" H 6900 4950 50  0001 C CNN
+F 0 "#PWR0190" H 6900 4950 50  0001 C CNN
 F 1 "+5V" H 6900 5240 50  0000 C CNN
 F 2 "" H 6900 5100 60  0000 C CNN
@@
 $EndComp
 $Comp
-L GND #PWR192
+L GND #PWR0191
 U 1 1 5624BF62
 P 6900 5500
-F 0 "#PWR192" H 6900 5250 50  0001 C CNN
+F 0 "#PWR0191" H 6900 5250 50  0001 C CNN
 F 1 "GND" H 6900 5350 50  0000 C CNN
 F 2 "" H 6900 5500 60  0000 C CNN
@@
 F 0 "R140" V 6580 5200 50  0000 C CNN
 F 1 "100" V 6500 5200 50  0000 C CNN
-F 2 "" V 6430 5200 30  0000 C CNN
+F 2 "Resistors_SMD:R_0603" V 6430 5200 30  0001 C CNN
 F 3 "" H 6500 5200 30  0000 C CNN
 	1    6500 5200
@@
 $EndComp
 $Comp
-L GND #PWR180
+L GND #PWR0192
 U 1 1 5624BFB9
 P 4400 8350
-F 0 "#PWR180" H 4400 8100 50  0001 C CNN
+F 0 "#PWR0192" H 4400 8100 50  0001 C CNN
 F 1 "GND" H 4400 8200 50  0000 C CNN
 F 2 "" H 4400 8350 60  0000 C CNN
@@
 F 0 "U19" H 5150 5950 60  0000 C CNN
 F 1 "SN74LVC162244A" H 4950 4850 60  0000 C CNN
-F 2 "" H 4950 5250 60  0000 C CNN
+F 2 "" H 4950 5250 60  0001 C CNN
 F 3 "" H 4950 5250 60  0000 C CNN
 	5    4950 5400
@@
 $EndComp
 $Comp
-L GND #PWR182
+L GND #PWR0193
 U 1 1 5624BFE2
 P 5650 5000
-F 0 "#PWR182" H 5650 4750 50  0001 C CNN
+F 0 "#PWR0193" H 5650 4750 50  0001 C CNN
 F 1 "GND" H 5650 4850 50  0000 C CNN
 F 2 "" H 5650 5000 60  0000 C CNN
@@
 	5400 5000 5650 5000
 $Comp
-L GND #PWR181
+L GND #PWR0194
 U 1 1 5624F657
 P 5650 2650
-F 0 "#PWR181" H 5650 2400 50  0001 C CNN
+F 0 "#PWR0194" H 5650 2400 50  0001 C CNN
 F 1 "GND" H 5650 2500 50  0000 C CNN
 F 2 "" H 5650 2650 60  0000 C CNN
