File: hardware/colibri-v2/servo_pwm_output.sch (KiCad schematic (older format))
At the start: 18 parts, among them P10 CONN_01X03, P11 CONN_01X03, P12 CONN_01X03, P13 CONN_01X03, P14 CONN_01X03, P15 CONN_01X03, P16 CONN_01X03, P17 CONN_01X03, U19 SN74LVC162244A

Commit message: Associated footprints for R and some of the C
Parts:
- R128, R129, R130, R131, R132, R133, R134, R135: footprint (none) -> Resistors_SMD:R_0603
Changed lines of the file:
@@
 F 0 "P14" H 5050 4750 50  0000 C CNN
 F 1 "CONN_01X03" V 5150 4550 50  0000 C CNN
-F 2 "" H 5050 4550 60  0000 C CNN
+F 2 "" H 5050 4550 60  0001 C CNN
 F 3 "" H 5050 4550 60  0000 C CNN
 	1    5050 4550
@@
 $EndComp
 $Comp
-L +5V #PWR169
+L +5V #PWR0161
 U 1 1 561914C0
 P 4700 4350
-F 0 "#PWR169" H 4700 4200 50  0001 C CNN
+F 0 "#PWR0161" H 4700 4200 50  0001 C CNN
 F 1 "+5V" H 4700 4490 50  0000 C CNN
 F 2 "" H 4700 4350 60  0000 C CNN
@@
 $EndComp
 $Comp
-L GND #PWR170
+L GND #PWR0162
 U 1 1 56191507
 P 4700 4750
-F 0 "#PWR170" H 4700 4500 50  0001 C CNN
+F 0 "#PWR0162" H 4700 4500 50  0001 C CNN
 F 1 "GND" H 4700 4600 50  0000 C CNN
 F 2 "" H 4700 4750 60  0000 C CNN
@@
 F 0 "R132" V 4380 4450 50  0000 C CNN
 F 1 "22" V 4300 4450 50  0000 C CNN
-F 2 "" V 4230 4450 30  0000 C CNN
+F 2 "Resistors_SMD:R_0603" V 4230 4450 30  0001 C CNN
 F 3 "" H 4300 4450 30  0000 C CNN
 	1    4300 4450
@@
 F 0 "P15" H 5050 5650 50  0000 C CNN
 F 1 "CONN_01X03" V 5150 5450 50  0000 C CNN
-F 2 "" H 5050 5450 60  0000 C CNN
+F 2 "" H 5050 5450 60  0001 C CNN
 F 3 "" H 5050 5450 60  0000 C CNN
 	1    5050 5450
@@
 $EndComp
 $Comp
-L +5V #PWR171
+L +5V #PWR0163
 U 1 1 56191928
 P 4700 5250
-F 0 "#PWR171" H 4700 5100 50  0001 C CNN
+F 0 "#PWR0163" H 4700 5100 50  0001 C CNN
 F 1 "+5V" H 4700 5390 50  0000 C CNN
 F 2 "" H 4700 5250 60  0000 C CNN
@@
 $EndComp
 $Comp
-L GND #PWR172
+L GND #PWR0164
 U 1 1 5619192E
 P 4700 5650
-F 0 "#PWR172" H 4700 5400 50  0001 C CNN
+F 0 "#PWR0164" H 4700 5400 50  0001 C CNN
 F 1 "GND" H 4700 5500 50  0000 C CNN
 F 2 "" H 4700 5650 60  0000 C CNN
@@
 F 0 "R133" V 4380 5350 50  0000 C CNN
 F 1 "22" V 4300 5350 50  0000 C CNN
-F 2 "" V 4230 5350 30  0000 C CNN
+F 2 "Resistors_SMD:R_0603" V 4230 5350 30  0001 C CNN
 F 3 "" H 4300 5350 30  0000 C CNN
 	1    4300 5350
@@
 F 0 "P16" H 5050 6550 50  0000 C CNN
 F 1 "CONN_01X03" V 5150 6350 50  0000 C CNN
-F 2 "" H 5050 6350 60  0000 C CNN
+F 2 "" H 5050 6350 60  0001 C CNN
 F 3 "" H 5050 6350 60  0000 C CNN
 	1    5050 6350
@@
 $EndComp
 $Comp
-L +5V #PWR173
+L +5V #PWR0165
 U 1 1 56191B28
 P 4700 6150
-F 0 "#PWR173" H 4700 6000 50  0001 C CNN
+F 0 "#PWR0165" H 4700 6000 50  0001 C CNN
 F 1 "+5V" H 4700 6290 50  0000 C CNN
 F 2 "" H 4700 6150 60  0000 C CNN
@@
 $EndComp
 $Comp
-L GND #PWR174
+L GND #PWR0166
 U 1 1 56191B2E
 P 4700 6550
-F 0 "#PWR174" H 4700 6300 50  0001 C CNN
+F 0 "#PWR0166" H 4700 6300 50  0001 C CNN
 F 1 "GND" H 4700 6400 50  0000 C CNN
 F 2 "" H 4700 6550 60  0000 C CNN
@@
 F 0 "R134" V 4380 6250 50  0000 C CNN
 F 1 "22" V 4300 6250 50  0000 C CNN
-F 2 "" V 4230 6250 30  0000 C CNN
+F 2 "Resistors_SMD:R_0603" V 4230 6250 30  0001 C CNN
 F 3 "" H 4300 6250 30  0000 C CNN
 	1    4300 6250
@@
 F 0 "P17" H 5050 7450 50  0000 C CNN
 F 1 "CONN_01X03" V 5150 7250 50  0000 C CNN
-F 2 "" H 5050 7250 60  0000 C CNN
+F 2 "" H 5050 7250 60  0001 C CNN
 F 3 "" H 5050 7250 60  0000 C CNN
 	1    5050 7250
@@
 $EndComp
 $Comp
-L +5V #PWR175
+L +5V #PWR0167
 U 1 1 56191CEC
 P 4700 7050
-F 0 "#PWR175" H 4700 6900 50  0001 C CNN
+F 0 "#PWR0167" H 4700 6900 50  0001 C CNN
 F 1 "+5V" H 4700 7190 50  0000 C CNN
 F 2 "" H 4700 7050 60  0000 C CNN
@@
 $EndComp
 $Comp
-L GND #PWR176
+L GND #PWR0168
 U 1 1 56191CF2
 P 4700 7450
-F 0 "#PWR176" H 4700 7200 50  0001 C CNN
+F 0 "#PWR0168" H 4700 7200 50  0001 C CNN
 F 1 "GND" H 4700 7300 50  0000 C CNN
 F 2 "" H 4700 7450 60  0000 C CNN
@@
 F 0 "R135" V 4380 7150 50  0000 C CNN
 F 1 "22" V 4300 7150 50  0000 C CNN
-F 2 "" V 4230 7150 30  0000 C CNN
+F 2 "Resistors_SMD:R_0603" V 4230 7150 30  0001 C CNN
 F 3 "" H 4300 7150 30  0000 C CNN
 	1    4300 7150
@@
 F 0 "P10" H 5050 1200 50  0000 C CNN
 F 1 "CONN_01X03" V 5150 1000 50  0000 C CNN
-F 2 "" H 5050 1000 60  0000 C CNN
+F 2 "" H 5050 1000 60  0001 C CNN
 F 3 "" H 5050 1000 60  0000 C CNN
 	1    5050 1000
@@
 $EndComp
 $Comp
-L +5V #PWR161
+L +5V #PWR0169
 U 1 1 56193403
 P 4700 800
-F 0 "#PWR161" H 4700 650 50  0001 C CNN
+F 0 "#PWR0169" H 4700 650 50  0001 C CNN
 F 1 "+5V" H 4700 940 50  0000 C CNN
 F 2 "" H 4700 800 60  0000 C CNN
@@
 $EndComp
 $Comp
-L GND #PWR162
+L GND #PWR0170
 U 1 1 56193409
 P 4700 1200
-F 0 "#PWR162" H 4700 950 50  0001 C CNN
+F 0 "#PWR0170" H 4700 950 50  0001 C CNN
 F 1 "GND" H 4700 1050 50  0000 C CNN
 F 2 "" H 4700 1200 60  0000 C CNN
@@
 F 0 "R128" V 4380 900 50  0000 C CNN
 F 1 "22" V 4300 900 50  0000 C CNN
-F 2 "" V 4230 900 30  0000 C CNN
+F 2 "Resistors_SMD:R_0603" V 4230 900 30  0001 C CNN
 F 3 "" H 4300 900 30  0000 C CNN
 	1    4300 900
@@
 F 0 "P11" H 5050 2100 50  0000 C CNN
 F 1 "CONN_01X03" V 5150 1900 50  0000 C CNN
-F 2 "" H 5050 1900 60  0000 C CNN
+F 2 "" H 5050 1900 60  0001 C CNN
 F 3 "" H 5050 1900 60  0000 C CNN
 	1    5050 1900
@@
 $EndComp
 $Comp
-L +5V #PWR163
+L +5V #PWR0171
 U 1 1 56193429
 P 4700 1700
-F 0 "#PWR163" H 4700 1550 50  0001 C CNN
+F 0 "#PWR0171" H 4700 1550 50  0001 C CNN
 F 1 "+5V" H 4700 1840 50  0000 C CNN
 F 2 "" H 4700 1700 60  0000 C CNN
@@
 $EndComp
 $Comp
-L GND #PWR164
+L GND #PWR0172
 U 1 1 5619342F
 P 4700 2100
-F 0 "#PWR164" H 4700 1850 50  0001 C CNN
+F 0 "#PWR0172" H 4700 1850 50  0001 C CNN
 F 1 "GND" H 4700 1950 50  0000 C CNN
 F 2 "" H 4700 2100 60  0000 C CNN
@@
 F 0 "R129" V 4380 1800 50  0000 C CNN
 F 1 "22" V 4300 1800 50  0000 C CNN
-F 2 "" V 4230 1800 30  0000 C CNN
+F 2 "Resistors_SMD:R_0603" V 4230 1800 30  0001 C CNN
 F 3 "" H 4300 1800 30  0000 C CNN
 	1    4300 1800
@@
 F 0 "P12" H 5050 3000 50  0000 C CNN
 F 1 "CONN_01X03" V 5150 2800 50  0000 C CNN
-F 2 "" H 5050 2800 60  0000 C CNN
+F 2 "" H 5050 2800 60  0001 C CNN
 F 3 "" H 5050 2800 60  0000 C CNN
 	1    5050 2800
@@
 $EndComp
 $Comp
-L +5V #PWR165
+L +5V #PWR0173
 U 1 1 5619344F
 P 4700 2600
-F 0 "#PWR165" H 4700 2450 50  0001 C CNN
+F 0 "#PWR0173" H 4700 2450 50  0001 C CNN
 F 1 "+5V" H 4700 2740 50  0000 C CNN
 F 2 "" H 4700 2600 60  0000 C CNN
@@
 $EndComp
 $Comp
-L GND #PWR166
+L GND #PWR0174
 U 1 1 56193455
 P 4700 3000
-F 0 "#PWR166" H 4700 2750 50  0001 C CNN
+F 0 "#PWR0174" H 4700 2750 50  0001 C CNN
 F 1 "GND" H 4700 2850 50  0000 C CNN
 F 2 "" H 4700 3000 60  0000 C CNN
@@
 F 0 "R130" V 4380 2700 50  0000 C CNN
 F 1 "22" V 4300 2700 50  0000 C CNN
-F 2 "" V 4230 2700 30  0000 C CNN
+F 2 "Resistors_SMD:R_0603" V 4230 2700 30  0001 C CNN
 F 3 "" H 4300 2700 30  0000 C CNN
 	1    4300 2700
@@
 F 0 "P13" H 5050 3900 50  0000 C CNN
 F 1 "CONN_01X03" V 5150 3700 50  0000 C CNN
-F 2 "" H 5050 3700 60  0000 C CNN
+F 2 "" H 5050 3700 60  0001 C CNN
 F 3 "" H 5050 3700 60  0000 C CNN
 	1    5050 3700
@@
 $EndComp
 $Comp
-L +5V #PWR167
+L +5V #PWR0175
 U 1 1 56193475
 P 4700 3500
-F 0 "#PWR167" H 4700 3350 50  0001 C CNN
+F 0 "#PWR0175" H 4700 3350 50  0001 C CNN
 F 1 "+5V" H 4700 3640 50  0000 C CNN
 F 2 "" H 4700 3500 60  0000 C CNN
@@
 $EndComp
 $Comp
-L GND #PWR168
+L GND #PWR0176
 U 1 1 5619347B
 P 4700 3900
-F 0 "#PWR168" H 4700 3650 50  0001 C CNN
+F 0 "#PWR0176" H 4700 3650 50  0001 C CNN
 F 1 "GND" H 4700 3750 50  0000 C CNN
 F 2 "" H 4700 3900 60  0000 C CNN
@@
 F 0 "R131" V 4380 3600 50  0000 C CNN
 F 1 "22" V 4300 3600 50  0000 C CNN
-F 2 "" V 4230 3600 30  0000 C CNN
+F 2 "Resistors_SMD:R_0603" V 4230 3600 30  0001 C CNN
 F 3 "" H 4300 3600 30  0000 C CNN
 	1    4300 3600
@@
 SRV_PWM_3
 $Comp
-L +3V3 #PWR177
+L +3V3 #PWR0177
 U 1 1 5619349D
 P 7600 1800
-F 0 "#PWR177" H 7600 1650 50  0001 C CNN
+F 0 "#PWR0177" H 7600 1650 50  0001 C CNN
 F 1 "+3V3" H 7600 1940 50  0000 C CNN
 F 2 "" H 7600 1800 60  0000 C CNN
@@
 $EndComp
 $Comp
-L GND #PWR178
+L GND #PWR0178
 U 1 1 561934AB
 P 7600 3400
-F 0 "#PWR178" H 7600 3150 50  0001 C CNN
+F 0 "#PWR0178" H 7600 3150 50  0001 C CNN
 F 1 "GND" H 7600 3250 50  0000 C CNN
 F 2 "" H 7600 3400 60  0000 C CNN
@@
 F 0 "C88" H 7650 3250 50  0000 L CNN
 F 1 "100n/50V" H 7200 3050 50  0000 L CNN
-F 2 "" H 7638 3000 30  0000 C CNN
+F 2 "" H 7638 3000 30  0001 C CNN
 F 3 "" H 7600 3150 60  0000 C CNN
 	1    7600 3150
@@
 F 0 "U19" H 3300 3050 60  0000 C CNN
 F 1 "SN74LVC162244A" H 3100 1950 60  0000 C CNN
-F 2 "" H 3100 2350 60  0000 C CNN
+F 2 "" H 3100 2350 60  0001 C CNN
 F 3 "" H 3100 2350 60  0000 C CNN
 	1    3100 2500
@@
 $EndComp
 $Comp
-L GND #PWR159
+L GND #PWR0179
 U 1 1 56246310
 P 2450 2100
-F 0 "#PWR159" H 2450 1850 50  0001 C CNN
+F 0 "#PWR0179" H 2450 1850 50  0001 C CNN
 F 1 "GND" H 2450 1950 50  0000 C CNN
 F 2 "" H 2450 2100 60  0000 C CNN
@@
 F 0 "U19" H 3300 6600 60  0000 C CNN
 F 1 "SN74LVC162244A" H 3100 5500 60  0000 C CNN
-F 2 "" H 3100 5900 60  0000 C CNN
+F 2 "" H 3100 5900 60  0001 C CNN
 F 3 "" H 3100 5900 60  0000 C CNN
 	2    3100 6050
@@
 F 0 "U19" H 8500 3050 60  0000 C CNN
 F 1 "SN74LVC162244A" H 8300 1950 60  0000 C CNN
-F 2 "" H 8300 2350 60  0000 C CNN
+F 2 "" H 8300 2350 60  0001 C CNN
 F 3 "" H 8300 2350 60  0000 C CNN
 	3    8300 2500
@@
 $EndComp
 $Comp
-L GND #PWR179
+L GND #PWR0180
 U 1 1 56246B43
 P 8950 3400
-F 0 "#PWR179" H 8950 3150 50  0001 C CNN
+F 0 "#PWR0180" H 8950 3150 50  0001 C CNN
 F 1 "GND" H 8950 3250 50  0000 C CNN
 F 2 "" H 8950 3400 60  0000 C CNN
@@
 $EndComp
 $Comp
-L GND #PWR160
+L GND #PWR0181
 U 1 1 5624E422
 P 2450 5650
-F 0 "#PWR160" H 2450 5400 50  0001 C CNN
+F 0 "#PWR0181" H 2450 5400 50  0001 C CNN
 F 1 "GND" H 2450 5500 50  0000 C CNN
 F 2 "" H 2450 5650 60  0000 C CNN
