File: hardware/colibri-v2/usb_otg_fs.sch (KiCad schematic (older format))
At the start: 15 parts, among them P9 USB_OTG, Q9 BSS138PW, U17 TPS2061CDBVT, U18 VBUS053CZ-HAF-G-08

Commit message: Associated footprints for R and some of the C
Parts:
- R120, R121, R122, R123, R124, R125, R126, R127: footprint (none) -> Resistors_SMD:R_0603
Changed lines of the file:
@@
 F 0 "P9" H 9625 5025 50  0000 C CNN
 F 1 "USB_OTG" H 9300 5350 50  0000 C CNN
-F 2 "" V 9250 5050 60  0000 C CNN
+F 2 "" V 9250 5050 60  0001 C CNN
 F 3 "" V 9250 5050 60  0000 C CNN
 	1    9300 5150
@@
 F 0 "U18" H 5450 4450 60  0000 C CNN
 F 1 "VBUS053CZ-HAF-G-08" H 5300 3850 60  0000 C CNN
-F 2 "" H 5250 4850 60  0000 C CNN
+F 2 "" H 5250 4850 60  0001 C CNN
 F 3 "" H 5250 4850 60  0000 C CNN
 	1    5300 4150
@@
 F 0 "R121" V 3350 5200 50  0000 C CNN
 F 1 "22" V 3400 5050 50  0000 C CNN
-F 2 "" V 3330 5050 30  0000 C CNN
+F 2 "Resistors_SMD:R_0603" V 3330 5050 30  0001 C CNN
 F 3 "" H 3400 5050 30  0000 C CNN
 	1    3400 5050
@@
 F 0 "R122" V 3350 5300 50  0000 C CNN
 F 1 "22" V 3400 5150 50  0000 C CNN
-F 2 "" V 3330 5150 30  0000 C CNN
+F 2 "Resistors_SMD:R_0603" V 3330 5150 30  0001 C CNN
 F 3 "" H 3400 5150 30  0000 C CNN
 	1    3400 5150
@@
 $EndComp
 $Comp
-L +3V3 #PWR149
+L +3V3 #PWR0151
 U 1 1 5614EDA6
 P 3100 1800
-F 0 "#PWR149" H 3100 1650 50  0001 C CNN
+F 0 "#PWR0151" H 3100 1650 50  0001 C CNN
 F 1 "+3V3" H 3100 1940 50  0000 C CNN
 F 2 "" H 3100 1800 60  0000 C CNN
@@
 F 0 "R120" V 3180 2350 50  0000 C CNN
 F 1 "10K" V 3100 2350 50  0000 C CNN
-F 2 "" V 3030 2350 30  0000 C CNN
+F 2 "Resistors_SMD:R_0603" V 3030 2350 30  0001 C CNN
 F 3 "" H 3100 2350 30  0000 C CNN
 	1    3100 2350
@@
 $EndComp
 $Comp
-L +3V3 #PWR150
+L +3V3 #PWR0152
 U 1 1 5614EDB3
 P 3450 1800
-F 0 "#PWR150" H 3450 1650 50  0001 C CNN
+F 0 "#PWR0152" H 3450 1650 50  0001 C CNN
 F 1 "+3V3" H 3450 1940 50  0000 C CNN
 F 2 "" H 3450 1800 60  0000 C CNN
@@
 F 0 "R123" V 3530 2350 50  0000 C CNN
 F 1 "47K" V 3450 2350 50  0000 C CNN
-F 2 "" V 3380 2350 30  0000 C CNN
+F 2 "Resistors_SMD:R_0603" V 3380 2350 30  0001 C CNN
 F 3 "" H 3450 2350 30  0000 C CNN
 	1    3450 2350
@@
 F 0 "D16" H 3800 2600 50  0000 C CNN
 F 1 "RED" H 3800 2400 50  0000 C CNN
-F 2 "" H 3800 2500 60  0000 C CNN
+F 2 "" H 3800 2500 60  0001 C CNN
 F 3 "" H 3800 2500 60  0000 C CNN
 	1    3800 2500
@@
 F 0 "R124" V 3880 2050 50  0000 C CNN
 F 1 "620" V 3800 2050 50  0000 C CNN
-F 2 "" V 3730 2050 30  0000 C CNN
+F 2 "Resistors_SMD:R_0603" V 3730 2050 30  0001 C CNN
 F 3 "" H 3800 2050 30  0000 C CNN
 	1    3800 2050
@@
 $EndComp
 $Comp
-L +3V3 #PWR151
+L +3V3 #PWR0153
 U 1 1 5614EDCE
 P 3800 1800
-F 0 "#PWR151" H 3800 1650 50  0001 C CNN
+F 0 "#PWR0153" H 3800 1650 50  0001 C CNN
 F 1 "+3V3" H 3800 1940 50  0000 C CNN
 F 2 "" H 3800 1800 60  0000 C CNN
@@
 F 0 "D17" H 9100 2350 50  0000 C CNN
 F 1 "GREEN" H 9100 2150 50  0000 C CNN
-F 2 "" H 9100 2250 60  0000 C CNN
+F 2 "" H 9100 2250 60  0001 C CNN
 F 3 "" H 9100 2250 60  0000 C CNN
 	1    9100 2250
@@
 F 0 "R127" V 9180 1850 50  0000 C CNN
 F 1 "620" V 9100 1850 50  0000 C CNN
-F 2 "" V 9030 1850 30  0000 C CNN
+F 2 "Resistors_SMD:R_0603" V 9030 1850 30  0001 C CNN
 F 3 "" H 9100 1850 30  0000 C CNN
 	1    9100 1850
@@
 $EndComp
 $Comp
-L +3V3 #PWR157
+L +3V3 #PWR0154
 U 1 1 5614EDE2
 P 9100 1600
-F 0 "#PWR157" H 9100 1450 50  0001 C CNN
+F 0 "#PWR0154" H 9100 1450 50  0001 C CNN
 F 1 "+3V3" H 9100 1740 50  0000 C CNN
 F 2 "" H 9100 1600 60  0000 C CNN
@@
 F 0 "Q9" H 9300 2850 50  0000 R CNN
 F 1 "BSS138PW" H 9650 2750 50  0000 R CNN
-F 2 "" H 9200 2900 29  0000 C CNN
+F 2 "" H 9200 2900 29  0001 C CNN
 F 3 "" H 9000 2800 60  0000 C CNN
 	1    9000 2800
@@
 $EndComp
 $Comp
-L GND #PWR158
+L GND #PWR0155
 U 1 1 5614EDEF
 P 9100 3250
-F 0 "#PWR158" H 9100 3000 50  0001 C CNN
+F 0 "#PWR0155" H 9100 3000 50  0001 C CNN
 F 1 "GND" H 9100 3100 50  0000 C CNN
 F 2 "" H 9100 3250 60  0000 C CNN
@@
 F 0 "R125" V 8380 2800 50  0000 C CNN
 F 1 "10K" V 8300 2800 50  0000 C CNN
-F 2 "" V 8230 2800 30  0000 C CNN
+F 2 "Resistors_SMD:R_0603" V 8230 2800 30  0001 C CNN
 F 3 "" H 8300 2800 30  0000 C CNN
 	1    8300 2800
@@
 F 0 "R126" V 8930 3100 50  0000 C CNN
 F 1 "47K" V 8850 3100 50  0000 C CNN
-F 2 "" V 8780 3100 30  0000 C CNN
+F 2 "Resistors_SMD:R_0603" V 8780 3100 30  0001 C CNN
 F 3 "" H 8850 3100 30  0000 C CNN
 	1    8850 3100
@@
 F 0 "C87" H 6525 3150 50  0000 L CNN
 F 1 "C" H 6525 2950 50  0000 L CNN
-F 2 "" H 6538 2900 30  0000 C CNN
+F 2 "" H 6538 2900 30  0001 C CNN
 F 3 "" H 6500 3050 60  0000 C CNN
 	1    6500 3050
@@
 $EndComp
 $Comp
-L GND #PWR155
+L GND #PWR0156
 U 1 1 5614EE0A
 P 6500 3250
-F 0 "#PWR155" H 6500 3000 50  0001 C CNN
+F 0 "#PWR0156" H 6500 3000 50  0001 C CNN
 F 1 "GND" H 6500 3100 50  0000 C CNN
 F 2 "" H 6500 3250 60  0000 C CNN
@@
 $EndComp
 $Comp
-L GND #PWR153
+L GND #PWR0157
 U 1 1 5614EE10
 P 6100 3250
-F 0 "#PWR153" H 6100 3000 50  0001 C CNN
+F 0 "#PWR0157" H 6100 3000 50  0001 C CNN
 F 1 "GND" H 6100 3100 50  0000 C CNN
 F 2 "" H 6100 3250 60  0000 C CNN
@@
 $EndComp
 $Comp
-L GND #PWR154
+L GND #PWR0158
 U 1 1 5614EE16
 P 6100 4500
-F 0 "#PWR154" H 6100 4250 50  0001 C CNN
+F 0 "#PWR0158" H 6100 4250 50  0001 C CNN
 F 1 "GND" H 6100 4350 50  0000 C CNN
 F 2 "" H 6100 4500 60  0000 C CNN
@@
 Connection ~ 4050 5050
 $Comp
-L GND #PWR156
+L GND #PWR0159
 U 1 1 5614EE59
 P 8900 5800
-F 0 "#PWR156" H 8900 5550 50  0001 C CNN
+F 0 "#PWR0159" H 8900 5550 50  0001 C CNN
 F 1 "GND" H 8900 5650 50  0000 C CNN
 F 2 "" H 8900 5800 60  0000 C CNN
@@
 Connection ~ 8900 5700
 $Comp
-L +5V #PWR152
+L +5V #PWR0160
 U 1 1 5614EE65
 P 4150 1800
-F 0 "#PWR152" H 4150 1650 50  0001 C CNN
+F 0 "#PWR0160" H 4150 1650 50  0001 C CNN
 F 1 "+5V" H 4150 1940 50  0000 C CNN
 F 2 "" H 4150 1800 60  0000 C CNN
@@
 F 0 "U17" H 5550 3150 60  0000 C CNN
 F 1 "TPS2061CDBVT" H 5300 2650 60  0000 C CNN
-F 2 "" H 5300 2700 60  0000 C CNN
+F 2 "" H 5300 2700 60  0001 C CNN
 F 3 "" H 5300 2700 60  0000 C CNN
 	1    5300 2900
