File: hardware/colibri-v2/usb_otg_fs.sch (KiCad schematic (older format))
At the start: 14 parts, among them CN8 629_105_150_921, U19 TPS2061CDBVT, U20 VBUS053CZ-HAF-G-08

Commit message: Added footprints
Parts:
- CN8: footprint (none) -> Sigmadrone:WURTH_629105150921
Changed lines of the file:
@@
 $Descr A4 11693 8268
 encoding utf-8
-Sheet 23 28
+Sheet 22 28
 Title ""
 Date ""
@@
 F 0 "CN8" H 10000 5500 60  0000 C CNN
 F 1 "629_105_150_921" V 10100 4700 60  0000 C CNN
-F 2 "" H 11400 6150 60  0001 C CNN
+F 2 "Sigmadrone:WURTH_629105150921" H 11400 6150 60  0001 C CNN
 F 3 "" H 11400 6150 60  0000 C CNN
 	1    9850 4850

Commit message: Added footprints
Parts:
- U19: footprint (none) -> TO_SOT_Packages_SMD:SOT-23-5
- U20: footprint (none) -> Sigmadrone:VBUS053CZ-HAF
Changed lines of the file:
@@
 F 0 "U20" H 5450 3950 60  0000 C CNN
 F 1 "VBUS053CZ-HAF-G-08" H 5300 3350 60  0000 C CNN
-F 2 "" H 5250 4350 60  0001 C CNN
+F 2 "Sigmadrone:VBUS053CZ-HAF" H 5250 4350 60  0001 C CNN
 F 3 "" H 5250 4350 60  0000 C CNN
 	1    5300 3650
@@
 F 0 "U19" H 5550 2700 60  0000 C CNN
 F 1 "TPS2061CDBVT" H 5300 2200 60  0000 C CNN
-F 2 "" H 5300 2250 60  0001 C CNN
+F 2 "TO_SOT_Packages_SMD:SOT-23-5" H 5300 2250 60  0001 C CNN
 F 3 "" H 5300 2250 60  0000 C CNN
 	1    5300 2450

Commit message: Added AP6681GMT-HF-3.kicad_mod. Fixed netlist errors
Parts:
- DL13: footprint LEDs:LED-0603 -> LEDs:LED_0603
Changed lines of the file:
@@
 F 0 "DL13" H 8300 3100 50  0000 C CNN
 F 1 "GREEN" H 8300 2900 50  0000 C CNN
-F 2 "LEDs:LED-0603" H 8300 2850 30  0001 C CNN
+F 2 "LEDs:LED_0603" H 8300 2850 30  0001 C CNN
 F 3 "" H 8300 3000 60  0000 C CNN
 F 4 "0603" H 8185 2980 30  0000 C CNN "SMT"
