File: hardware/colibri-v2/wnd_lcd.sch (KiCad schematic (older format))
At the start: 18 parts

Commit message: Work on Wandboard LCD
Parts:
- added C? (x3): 1u/10%/10V, symbol C
- added C? (x2): 47u/20%/6.3V, symbol C
- added C? (x5): 0.1u/10%/16V, symbol C
- added R? (x9): 22R, symbol R
- added R? (x2): 10K, symbol R
Connections:
- net +3V3: now also CN?.45 (VDD1), CN?.46 (VDD2), C?.1, C?.1, C?.1, C?.1, C?.1, C?.1, R?.1
- net GND: now also CN?.18 (GND), CN?.27 (GND/CNTRST), CN?.31 (GND), CN?.33 (GND), CN?.44 (GND), CN?.9 (GND), C?.2, C?.2, C?.2, C?.2, C?.2, C?.2, C?.2, C?.2, C?.2, C?.2, R?.1
- net TOUCH_X1: now also CN?.34 (X+)
- net TOUCH_X2: now also CN?.35 (X-)
- net TOUCH_Y1: now also CN?.36 (Y+)
- net TOUCH_Y2: now also CN?.37 (Y-)
- net at CN?.28 (DEN), R?.1: now also R?.1
- net at CN?.38 (SPI_CLK): now also R?.1
- net at CN?.39 (SPI_MOSI): now also R?.1
- net at CN?.40 (SPI_MISO): now also R?.1
- net at CN?.41 (CS): now also R?.1
- net at CN?.42 (I2C_CLK): now also R?.1
- net at CN?.43 (I2C_DAT): now also R?.1
- net +5V: now reaches CN?.47 (VDD3)
- net +5V: now also CN?.48 (VDD4), C?.1, C?.1, C?.1, C?.1
- net at CN?.49 (RESET): now also R?.1, R?.2
- net at CN?.50 (PWREN): now also R?.1, R?.2
- new net DISP0_CNTRST: R?.2
- new net DISP0_I2C_CLK: R?.2
- new net DISP0_I2C_SDA: R?.2
- new net DISP0_PWREN: R?.2
- new net DISP0_REST: R?.2
- new net DISP0_SPI_CLK: R?.2
- new net DISP0_SPI_CS: R?.2
- new net DISP0_SPI_MISO: R?.2
- new net DISP0_SPI_MOSI: R?.2
Other:
- note added: "mars board_V1.0.pdf\npage 12 (LCD PORT)"
- moved on the sheet: C?, CN?, R?, U?

Commit message: Annotated Components
Parts:
- gave numbers to parts that had none: 39

Commit message: Work on hardware
Other:
- note added: "27 pin 0R to GND"
- note added: "Research for capacitive \ncontroller???"
Changed lines of the file:
@@
 	3800 3400 2300 3400
 Wire Bus Line
-	2200 750  2200 800
-Wire Bus Line
-	2200 800  2200 900
-Wire Bus Line
-	2200 900  2200 1000
-Wire Bus Line
-	2200 1000 2200 1100
-Wire Bus Line
-	2200 1100 2200 1200
-Wire Bus Line
-	2200 1200 2200 1300
-Wire Bus Line
-	2200 1300 2200 1400
-Wire Bus Line
-	2200 1400 2200 1500
-Wire Bus Line
-	2200 1500 2200 1700
-Wire Bus Line
-	2200 1700 2200 1800
-Wire Bus Line
-	2200 1800 2200 1900
-Wire Bus Line
-	2200 1900 2200 2000
-Wire Bus Line
-	2200 2000 2200 2100
-Wire Bus Line
-	2200 2100 2200 2200
-Wire Bus Line
-	2200 2200 2200 2300
-Wire Bus Line
-	2200 2300 2200 2400
-Wire Bus Line
-	2200 2400 2200 2600
-Wire Bus Line
-	2200 2600 2200 2700
-Wire Bus Line
-	2200 2700 2200 2800
-Wire Bus Line
-	2200 2800 2200 2900
-Wire Bus Line
-	2200 2900 2200 3000
-Wire Bus Line
-	2200 3000 2200 3100
-Wire Bus Line
-	2200 3100 2200 3200
-Wire Bus Line
-	2200 3200 2200 3300
+	2200 750  2200 3300
 Wire Bus Line
 	2200 750  1750 750
 Wire Wire Line
-	3100 3600 3350 3600
-Wire Wire Line
-	3350 3600 3800 3600
+	3100 3600 3800 3600
 Wire Wire Line
 	3100 3700 3800 3700
@@
 	1750 4000 2800 4000
 Wire Wire Line
-	7000 4400 7000 4650
-Wire Wire Line
-	7000 4650 7000 4750
+	7000 4400 7000 4750
 Wire Wire Line
 	7000 4650 7300 4650
@@
 	9550 5250 8400 5250
 Wire Wire Line
-	9550 3850 9550 3950
-Wire Wire Line
-	9550 3950 9550 5250
-Wire Wire Line
-	9550 5250 9550 5700
+	9550 3850 9550 5700
 $Comp
 L R R103
@@
 	8550 4950 8400 4950
 Wire Wire Line
-	8850 4650 8950 4650
-Wire Wire Line
-	8950 4650 10100 4650
-Wire Wire Line
-	8850 4750 9050 4750
-Wire Wire Line
-	9050 4750 10100 4750
-Wire Wire Line
-	8850 4850 9150 4850
-Wire Wire Line
-	9150 4850 10100 4850
-Wire Wire Line
-	8850 4950 9250 4950
-Wire Wire Line
-	9250 4950 10100 4950
-Wire Wire Line
-	8400 5150 9450 5150
-Wire Wire Line
-	9450 5150 10100 5150
+	8850 4650 10100 4650
+Wire Wire Line
+	8850 4750 10100 4750
+Wire Wire Line
+	8850 4850 10100 4850
+Wire Wire Line
+	8850 4950 10100 4950
+Wire Wire Line
+	8400 5150 10100 5150
 $Comp
 L R R110
@@
 	9450 3950 9450 4050
 Wire Wire Line
-	8950 3950 9050 3950
-Wire Wire Line
-	9050 3950 9150 3950
-Wire Wire Line
-	9150 3950 9250 3950
-Wire Wire Line
-	9250 3950 9350 3950
-Wire Wire Line
-	9350 3950 9450 3950
-Wire Wire Line
-	9450 3950 9550 3950
+	8950 3950 9550 3950
 Wire Wire Line
 	8950 3950 8950 4050
@@
 $EndComp
 Wire Wire Line
-	2450 5600 3600 5600
-Wire Wire Line
-	3600 5600 3800 5600
+	2450 5600 3800 5600
 Wire Wire Line
 	3800 5700 3600 5700
@@
 Connection ~ 3600 5600
 Wire Wire Line
-	2450 5900 3600 5900
-Wire Wire Line
-	3600 5900 3800 5900
+	2450 5900 3800 5900
 Wire Wire Line
 	3800 5800 3600 5800
@@
 $EndComp
 Wire Wire Line
-	2450 5400 3600 5400
-Wire Wire Line
-	3600 5400 3800 5400
+	2450 5400 3800 5400
 Wire Wire Line
 	3600 4100 3800 4100
 Wire Wire Line
-	3600 1700 3600 2600
-Wire Wire Line
-	3600 2600 3600 3500
-Wire Wire Line
-	3600 3500 3600 3900
-Wire Wire Line
-	3600 3900 3600 4100
-Wire Wire Line
-	3600 4100 3600 5400
+	3600 1700 3600 5400
 Connection ~ 3600 5400
 Wire Wire Line
@@
 	2850 6700 2850 6850
 Wire Wire Line
-	2500 6100 2850 6100
-Wire Wire Line
-	2850 6100 3800 6100
-Wire Wire Line
-	2500 6200 3150 6200
-Wire Wire Line
-	3150 6200 3800 6200
+	2500 6100 3800 6100
+Wire Wire Line
+	2500 6200 3800 6200
 Wire Wire Line
 	1750 6100 2200 6100
@@
 	7200 950  7200 1200
 Wire Wire Line
-	6000 950  6600 950
-Wire Wire Line
-	6600 950  7200 950
-Wire Wire Line
-	7200 950  7800 950
-Wire Wire Line
-	6000 800  6000 950
-Wire Wire Line
-	6000 950  6000 1200
-Wire Wire Line
-	6000 1500 6000 1700
-Wire Wire Line
-	6000 1700 6000 1850
-Wire Wire Line
-	6000 1700 6600 1700
-Wire Wire Line
-	6600 1700 7200 1700
-Wire Wire Line
-	7200 1700 7800 1700
+	6000 950  7800 950
+Wire Wire Line
+	6000 800  6000 1200
+Wire Wire Line
+	6000 1500 6000 1850
+Wire Wire Line
+	6000 1700 7800 1700
 Wire Wire Line
 	7200 1700 7200 1500
@@
 	7200 2500 7200 2750
 Wire Wire Line
-	6000 2500 6600 2500
-Wire Wire Line
-	6600 2500 7200 2500
-Wire Wire Line
-	7200 2500 7800 2500
-Wire Wire Line
-	6000 2350 6000 2500
-Wire Wire Line
-	6000 2500 6000 2750
-Wire Wire Line
-	6000 3050 6000 3250
-Wire Wire Line
-	6000 3250 6000 3400
-Wire Wire Line
-	6000 3250 6600 3250
-Wire Wire Line
-	6600 3250 7200 3250
-Wire Wire Line
-	7200 3250 7800 3250
+	6000 2500 7800 2500
+Wire Wire Line
+	6000 2350 6000 2750
+Wire Wire Line
+	6000 3050 6000 3400
+Wire Wire Line
+	6000 3250 7800 3250
 Wire Wire Line
 	7200 3250 7200 3050
@@
 $EndComp
 Wire Wire Line
-	8850 800  8850 950
-Wire Wire Line
-	8850 950  8850 1200
-Wire Wire Line
-	8850 1500 8850 1700
-Wire Wire Line
-	8850 1700 8850 1850
+	8850 800  8850 1200
+Wire Wire Line
+	8850 1500 8850 1850
 Wire Wire Line
 	9450 1200 9450 950
@@
 	3350 3500 3350 3600
 Connection ~ 3350 3600
+Text Notes 8550 3550 0    120  ~ 24
+Research for capacitive \ncontroller???
+Text Notes 1100 3350 0    60   ~ 0
+27 pin 0R to GND
 $EndSCHEMATC

Commit message: Work on LCD module
Parts:
- added R?: NA, symbol R
- added R?: 0R, symbol R
Connections:
- net DISP0_CNTRST: now also R?.2
- net GND: now also R?.2; no longer CN4.27 (GND/CNTRST)
- new net: CN4.27 (GND/CNTRST), R?.1, R?.1
Other:
- note added: "Research for \ncapacitive controller???"
- note removed: "27 pin 0R to GND"
- note removed: "Research for capacitive \ncontroller???"
- moved on the sheet: C74, C75, C76, C77, C78, C79, C80, C81, C82, C84, CN4, R100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

Commit message: Re-annotated schematic
Parts:
- gave numbers to parts that had none: 2
- renumbered C74 to C72, C75 to C73, C76 to C74, C77 to C75, C78 to C76, C79 to C77, C80 to C78, C81 to C79, C83 to C80, C82 to C81, C85 to C82, C84 to C83, R88 to R102, R89 to R103, R90 to R104, R102 to R105, R103 to R106, R104 to R107, R105 to R108, R106 to R109, R107 to R110, R108 to R111, R109 to R112, R110 to R113, R111 to R114, R112 to R115

Commit message: Associated footprints for R and some of the C
Parts:
- R100, R101, R102, R103, R104, R105, R106, R107, R108, R109, R110, R111, R112, R113, R114, R115, R89, R90, R91, R92, R93, R94, R95, R96, R97, R98, R99: footprint (none) -> Resistors_SMD:R_0603

Commit message: Work on cortex USB connection.
Parts:
- renumbered C80 to C?, C82 to C?, C76 to C?, C72 to C?, C74 to C?, C78 to C?, C77 to C?, C73 to C?, C75 to C?, C79 to C?, C83 to C?, C81 to C?, CN4 to CN?, R92 to R?, R93 to R?, R94 to R?, R95 to R?, R106 to R?, R107 to R?, R108 to R?, R109 to R?, R113 to R?, R112 to R?, R111 to R?, R110 to R?, R114 to R?, R115 to R?, R96 to R?, R97 to R?, R98 to R?, R99 to R?, R100 to R?, R101 to R?, R103 to R?, R105 to R?, R104 to R?, R102 to R?, R91 to R?, R90 to R?, R89 to R?, U15 to U?
