File: hardware/colibri-v2/wnd_micro_sd.sch (KiCad schematic (older format))
At the start: 12 parts

Commit message: added wnd_lcd.sch
Changed lines of the file:
@@
 $Descr A4 11693 8268
 encoding utf-8
-Sheet 14 22
+Sheet 14 23
 Title ""
 Date ""
@@
 	5500 4550 5350 4550
 Wire Wire Line
-	5350 3950 5350 4550
-Wire Wire Line
-	5350 4550 5350 5050
-Wire Wire Line
-	6100 4850 6100 4950
-Wire Wire Line
-	6100 4950 6100 5050
+	5350 3950 5350 5050
+Wire Wire Line
+	6100 4850 6100 5050
 Wire Wire Line
 	6200 4850 6200 4950
@@
 Connection ~ 6100 4950
 Wire Wire Line
-	3450 3450 4400 3450
-Wire Wire Line
-	4400 3450 5500 3450
-Wire Wire Line
-	3450 3550 4500 3550
-Wire Wire Line
-	4500 3550 5500 3550
-Wire Wire Line
-	3450 4050 4700 4050
-Wire Wire Line
-	4700 4050 5500 4050
-Wire Wire Line
-	3450 4150 4800 4150
-Wire Wire Line
-	4800 4150 5500 4150
-Wire Wire Line
-	3450 4250 4900 4250
-Wire Wire Line
-	4900 4250 5500 4250
-Wire Wire Line
-	3450 4350 4300 4350
-Wire Wire Line
-	4300 4350 5500 4350
+	3450 3450 5500 3450
+Wire Wire Line
+	3450 3550 5500 3550
+Wire Wire Line
+	3450 4050 5500 4050
+Wire Wire Line
+	3450 4150 5500 4150
+Wire Wire Line
+	3450 4250 5500 4250
+Wire Wire Line
+	3450 4350 5500 4350
 Wire Wire Line
 	5500 3950 5350 3950
@@
 $EndComp
 Wire Wire Line
-	4100 3850 4600 3850
-Wire Wire Line
-	4600 3850 5500 3850
+	4100 3850 5500 3850
 Wire Wire Line
 	3800 3850 3450 3850
@@
 $EndComp
 Wire Wire Line
-	5350 1550 5350 1850
-Wire Wire Line
-	5350 1850 5350 3750
+	5350 1550 5350 3750
 Wire Wire Line
 	5350 3750 5500 3750
@@
 	4300 2050 4300 1850
 Wire Wire Line
-	4300 1850 4400 1850
-Wire Wire Line
-	4400 1850 4500 1850
-Wire Wire Line
-	4500 1850 4600 1850
-Wire Wire Line
-	4600 1850 4700 1850
-Wire Wire Line
-	4700 1850 4800 1850
-Wire Wire Line
-	4800 1850 4900 1850
-Wire Wire Line
-	4900 1850 5350 1850
-Wire Wire Line
-	5350 1850 5900 1850
-Wire Wire Line
-	5900 1850 6500 1850
+	4300 1850 6500 1850
 Connection ~ 5350 1850
 Wire Wire Line
@@
 Connection ~ 5900 1850
 Wire Wire Line
-	6500 2350 6500 2700
-Wire Wire Line
-	6500 2700 6500 2850
+	6500 2350 6500 2850
 Wire Wire Line
 	5900 2350 5900 2700

Commit message: Annotated Components
Parts:
- gave numbers to parts that had none: 12
Changed lines of the file:
@@
 $EndDescr
 $Comp
-L uSDCARD-H1.85 MSD?
+L uSDCARD-H1.85 MSD1
 U 1 1 56153956
 P 6350 4000
-F 0 "MSD?" H 6600 3300 60  0000 C CNN
+F 0 "MSD1" H 6600 3300 60  0000 C CNN
 F 1 "uSDCARD-H1.85" H 6450 4700 60  0000 C CNN
 F 2 "" H 6350 4000 60  0000 C CNN
@@
 SD1_WP
 $Comp
-L GND #PWR?
+L GND #PWR100
 U 1 1 5617363A
 P 5350 5050
-F 0 "#PWR?" H 5350 4800 50  0001 C CNN
+F 0 "#PWR100" H 5350 4800 50  0001 C CNN
 F 1 "GND" H 5350 4900 50  0000 C CNN
 F 2 "" H 5350 5050 60  0000 C CNN
@@
 $EndComp
 $Comp
-L GND #PWR?
+L GND #PWR101
 U 1 1 5617364F
 P 6100 5050
-F 0 "#PWR?" H 6100 4800 50  0001 C CNN
+F 0 "#PWR101" H 6100 4800 50  0001 C CNN
 F 1 "GND" H 6100 4900 50  0000 C CNN
 F 2 "" H 6100 5050 60  0000 C CNN
@@
 Connection ~ 5350 4550
 $Comp
-L R R?
+L R R67
 U 1 1 561736B3
 P 3950 3850
-F 0 "R?" V 4030 3850 50  0000 C CNN
+F 0 "R67" V 4030 3850 50  0000 C CNN
 F 1 "22" V 3950 3850 50  0000 C CNN
 F 2 "" V 3880 3850 30  0000 C CNN
@@
 	3800 3850 3450 3850
 $Comp
-L +3V3 #PWR?
+L +3V3 #PWR99
 U 1 1 561737FF
 P 5350 1550
-F 0 "#PWR?" H 5350 1400 50  0001 C CNN
+F 0 "#PWR99" H 5350 1400 50  0001 C CNN
 F 1 "+3V3" H 5350 1690 50  0000 C CNN
 F 2 "" H 5350 1550 60  0000 C CNN
@@
 	5350 3750 5500 3750
 $Comp
-L R R?
+L R R69
 U 1 1 56173C05
 P 4300 2200
-F 0 "R?" V 4350 2050 50  0000 C CNN
+F 0 "R69" V 4350 2050 50  0000 C CNN
 F 1 "10K" V 4300 2200 50  0000 C CNN
 F 2 "" V 4230 2200 30  0000 C CNN
@@
 $EndComp
 $Comp
-L R R?
+L R R70
 U 1 1 56173C21
 P 4400 2200
-F 0 "R?" V 4450 2050 50  0000 C CNN
+F 0 "R70" V 4450 2050 50  0000 C CNN
 F 1 "10K" V 4400 2200 50  0000 C CNN
 F 2 "" V 4330 2200 30  0000 C CNN
@@
 $EndComp
 $Comp
-L R R?
+L R R71
 U 1 1 56173C44
 P 4500 2200
-F 0 "R?" V 4550 2050 50  0000 C CNN
+F 0 "R71" V 4550 2050 50  0000 C CNN
 F 1 "10K" V 4500 2200 50  0000 C CNN
 F 2 "" V 4430 2200 30  0000 C CNN
@@
 $EndComp
 $Comp
-L R R?
+L R R72
 U 1 1 56173C66
 P 4600 2200
-F 0 "R?" V 4650 2050 50  0000 C CNN
+F 0 "R72" V 4650 2050 50  0000 C CNN
 F 1 "10K" V 4600 2200 50  0000 C CNN
 F 2 "" V 4530 2200 30  0000 C CNN
@@
 $EndComp
 $Comp
-L R R?
+L R R73
 U 1 1 56173C8B
 P 4700 2200
-F 0 "R?" V 4750 2050 50  0000 C CNN
+F 0 "R73" V 4750 2050 50  0000 C CNN
 F 1 "10K" V 4700 2200 50  0000 C CNN
 F 2 "" V 4630 2200 30  0000 C CNN
@@
 $EndComp
 $Comp
-L R R?
+L R R74
 U 1 1 56173CB3
 P 4800 2200
-F 0 "R?" V 4850 2050 50  0000 C CNN
+F 0 "R74" V 4850 2050 50  0000 C CNN
 F 1 "10K" V 4800 2200 50  0000 C CNN
 F 2 "" V 4730 2200 30  0000 C CNN
@@
 $EndComp
 $Comp
-L R R?
+L R R75
 U 1 1 56173CDE
 P 4900 2200
-F 0 "R?" V 4950 2050 50  0000 C CNN
+F 0 "R75" V 4950 2050 50  0000 C CNN
 F 1 "10K" V 4900 2200 50  0000 C CNN
 F 2 "" V 4830 2200 30  0000 C CNN
@@
 $EndComp
 $Comp
-L R R?
+L R R68
 U 1 1 56173D14
 P 4200 4750
-F 0 "R?" V 4250 4600 50  0000 C CNN
+F 0 "R68" V 4250 4600 50  0000 C CNN
 F 1 "10K" V 4200 4750 50  0000 C CNN
 F 2 "" V 4130 4750 30  0000 C CNN
@@
 	4200 4450 4200 4600
 $Comp
-L GND #PWR?
+L GND #PWR98
 U 1 1 56173E31
 P 4200 5050
-F 0 "#PWR?" H 4200 4800 50  0001 C CNN
+F 0 "#PWR98" H 4200 4800 50  0001 C CNN
 F 1 "GND" H 4200 4900 50  0000 C CNN
 F 2 "" H 4200 5050 60  0000 C CNN
@@
 Connection ~ 4900 1850
 $Comp
-L C C?
+L C C65
 U 1 1 5617422F
 P 5900 2200
-F 0 "C?" H 5925 2300 50  0000 L CNN
+F 0 "C65" H 5925 2300 50  0000 L CNN
 F 1 "10u/10V/X5R-C5" V 5800 1800 50  0000 L CNN
 F 2 "" H 5938 2050 30  0000 C CNN
@@
 $EndComp
 $Comp
-L C C?
+L C C66
 U 1 1 561742E8
 P 6500 2200
-F 0 "C?" H 6525 2300 50  0000 L CNN
+F 0 "C66" H 6525 2300 50  0000 L CNN
 F 1 "10u/16V/X7R-C2" V 6400 1800 50  0000 L CNN
 F 2 "" H 6538 2050 30  0000 C CNN
@@
 $EndComp
 $Comp
-L GND #PWR?
+L GND #PWR102
 U 1 1 5617463C
 P 6500 2850
-F 0 "#PWR?" H 6500 2600 50  0001 C CNN
+F 0 "#PWR102" H 6500 2600 50  0001 C CNN
 F 1 "GND" H 6500 2700 50  0000 C CNN
 F 2 "" H 6500 2850 60  0000 C CNN

Commit message: Work on hardware
Other:
- note added: "Do we need this?"
Changed lines of the file:
@@
 	5900 2700 6500 2700
 Connection ~ 6500 2700
+Text Notes 7400 4100 0    120  ~ 24
+Do we need this?
 $EndSCHEMATC

Commit message: Re-annotated schematic
Parts:
- renumbered C65 to C63, C66 to C64, R67 to R68, R68 to R69, R69 to R70, R70 to R71, R71 to R72, R72 to R73, R73 to R74, R74 to R75, R75 to R76
Changed lines of the file:
@@
 SD1_WP
 $Comp
-L GND #PWR0100
+L GND #PWR97
 U 1 1 5617363A
 P 5350 5050
-F 0 "#PWR0100" H 5350 4800 50  0001 C CNN
+F 0 "#PWR97" H 5350 4800 50  0001 C CNN
 F 1 "GND" H 5350 4900 50  0000 C CNN
 F 2 "" H 5350 5050 60  0000 C CNN
@@
 $EndComp
 $Comp
-L GND #PWR0101
+L GND #PWR98
 U 1 1 5617364F
 P 6100 5050
-F 0 "#PWR0101" H 6100 4800 50  0001 C CNN
+F 0 "#PWR98" H 6100 4800 50  0001 C CNN
 F 1 "GND" H 6100 4900 50  0000 C CNN
 F 2 "" H 6100 5050 60  0000 C CNN
@@
 Connection ~ 5350 4550
 $Comp
-L R R67
+L R R68
 U 1 1 561736B3
 P 3950 3850
-F 0 "R67" V 4030 3850 50  0000 C CNN
+F 0 "R68" V 4030 3850 50  0000 C CNN
 F 1 "22" V 3950 3850 50  0000 C CNN
 F 2 "" V 3880 3850 30  0000 C CNN
@@
 	3800 3850 3450 3850
 $Comp
-L +3V3 #PWR0102
+L +3V3 #PWR96
 U 1 1 561737FF
 P 5350 1550
-F 0 "#PWR0102" H 5350 1400 50  0001 C CNN
+F 0 "#PWR96" H 5350 1400 50  0001 C CNN
 F 1 "+3V3" H 5350 1690 50  0000 C CNN
 F 2 "" H 5350 1550 60  0000 C CNN
@@
 	5350 3750 5500 3750
 $Comp
-L R R69
+L R R70
 U 1 1 56173C05
 P 4300 2200
-F 0 "R69" V 4350 2050 50  0000 C CNN
+F 0 "R70" V 4350 2050 50  0000 C CNN
 F 1 "10K" V 4300 2200 50  0000 C CNN
 F 2 "" V 4230 2200 30  0000 C CNN
@@
 $EndComp
 $Comp
-L R R70
+L R R71
 U 1 1 56173C21
 P 4400 2200
-F 0 "R70" V 4450 2050 50  0000 C CNN
+F 0 "R71" V 4450 2050 50  0000 C CNN
 F 1 "10K" V 4400 2200 50  0000 C CNN
 F 2 "" V 4330 2200 30  0000 C CNN
@@
 $EndComp
 $Comp
-L R R71
+L R R72
 U 1 1 56173C44
 P 4500 2200
-F 0 "R71" V 4550 2050 50  0000 C CNN
+F 0 "R72" V 4550 2050 50  0000 C CNN
 F 1 "10K" V 4500 2200 50  0000 C CNN
 F 2 "" V 4430 2200 30  0000 C CNN
@@
 $EndComp
 $Comp
-L R R72
+L R R73
 U 1 1 56173C66
 P 4600 2200
-F 0 "R72" V 4650 2050 50  0000 C CNN
+F 0 "R73" V 4650 2050 50  0000 C CNN
 F 1 "10K" V 4600 2200 50  0000 C CNN
 F 2 "" V 4530 2200 30  0000 C CNN
@@
 $EndComp
 $Comp
-L R R73
+L R R74
 U 1 1 56173C8B
 P 4700 2200
-F 0 "R73" V 4750 2050 50  0000 C CNN
+F 0 "R74" V 4750 2050 50  0000 C CNN
 F 1 "10K" V 4700 2200 50  0000 C CNN
 F 2 "" V 4630 2200 30  0000 C CNN
@@
 $EndComp
 $Comp
-L R R74
+L R R75
 U 1 1 56173CB3
 P 4800 2200
-F 0 "R74" V 4850 2050 50  0000 C CNN
+F 0 "R75" V 4850 2050 50  0000 C CNN
 F 1 "10K" V 4800 2200 50  0000 C CNN
 F 2 "" V 4730 2200 30  0000 C CNN
@@
 $EndComp
 $Comp
-L R R75
+L R R76
 U 1 1 56173CDE
 P 4900 2200
-F 0 "R75" V 4950 2050 50  0000 C CNN
+F 0 "R76" V 4950 2050 50  0000 C CNN
 F 1 "10K" V 4900 2200 50  0000 C CNN
 F 2 "" V 4830 2200 30  0000 C CNN
@@
 $EndComp
 $Comp
-L R R68
+L R R69
 U 1 1 56173D14
 P 4200 4750
-F 0 "R68" V 4250 4600 50  0000 C CNN
+F 0 "R69" V 4250 4600 50  0000 C CNN
 F 1 "10K" V 4200 4750 50  0000 C CNN
 F 2 "" V 4130 4750 30  0000 C CNN
@@
 	4200 4450 4200 4600
 $Comp
-L GND #PWR0103
+L GND #PWR95
 U 1 1 56173E31
 P 4200 5050
-F 0 "#PWR0103" H 4200 4800 50  0001 C CNN
+F 0 "#PWR95" H 4200 4800 50  0001 C CNN
 F 1 "GND" H 4200 4900 50  0000 C CNN
 F 2 "" H 4200 5050 60  0000 C CNN
@@
 Connection ~ 4900 1850
 $Comp
-L C C65
+L C C63
 U 1 1 5617422F
 P 5900 2200
-F 0 "C65" H 5925 2300 50  0000 L CNN
+F 0 "C63" H 5925 2300 50  0000 L CNN
 F 1 "10u/10V/X5R-C5" V 5800 1800 50  0000 L CNN
 F 2 "" H 5938 2050 30  0000 C CNN
@@
 $EndComp
 $Comp
-L C C66
+L C C64
 U 1 1 561742E8
 P 6500 2200
-F 0 "C66" H 6525 2300 50  0000 L CNN
+F 0 "C64" H 6525 2300 50  0000 L CNN
 F 1 "10u/16V/X7R-C2" V 6400 1800 50  0000 L CNN
 F 2 "" H 6538 2050 30  0000 C CNN
@@
 $EndComp
 $Comp
-L GND #PWR0104
+L GND #PWR99
 U 1 1 5617463C
 P 6500 2850
-F 0 "#PWR0104" H 6500 2600 50  0001 C CNN
+F 0 "#PWR99" H 6500 2600 50  0001 C CNN
 F 1 "GND" H 6500 2700 50  0000 C CNN
 F 2 "" H 6500 2850 60  0000 C CNN

Commit message: Associated footprints for R and some of the C
Parts:
- R68, R69, R70, R71, R72, R73, R74, R75, R76: footprint (none) -> Resistors_SMD:R_0603
Changed lines of the file:
@@
 F 0 "MSD1" H 6600 3300 60  0000 C CNN
 F 1 "uSDCARD-H1.85" H 6450 4700 60  0000 C CNN
-F 2 "" H 6350 4000 60  0000 C CNN
+F 2 "" H 6350 4000 60  0001 C CNN
 F 3 "" H 6350 4000 60  0000 C CNN
 	1    6350 4000
@@
 SD1_WP
 $Comp
-L GND #PWR97
+L GND #PWR097
 U 1 1 5617363A
 P 5350 5050
-F 0 "#PWR97" H 5350 4800 50  0001 C CNN
+F 0 "#PWR097" H 5350 4800 50  0001 C CNN
 F 1 "GND" H 5350 4900 50  0000 C CNN
 F 2 "" H 5350 5050 60  0000 C CNN
@@
 $EndComp
 $Comp
-L GND #PWR98
+L GND #PWR098
 U 1 1 5617364F
 P 6100 5050
-F 0 "#PWR98" H 6100 4800 50  0001 C CNN
+F 0 "#PWR098" H 6100 4800 50  0001 C CNN
 F 1 "GND" H 6100 4900 50  0000 C CNN
 F 2 "" H 6100 5050 60  0000 C CNN
@@
 F 0 "R68" V 4030 3850 50  0000 C CNN
 F 1 "22" V 3950 3850 50  0000 C CNN
-F 2 "" V 3880 3850 30  0000 C CNN
+F 2 "Resistors_SMD:R_0603" V 3880 3850 30  0001 C CNN
 F 3 "" H 3950 3850 30  0000 C CNN
 	1    3950 3850
@@
 	3800 3850 3450 3850
 $Comp
-L +3V3 #PWR96
+L +3V3 #PWR099
 U 1 1 561737FF
 P 5350 1550
-F 0 "#PWR96" H 5350 1400 50  0001 C CNN
+F 0 "#PWR099" H 5350 1400 50  0001 C CNN
 F 1 "+3V3" H 5350 1690 50  0000 C CNN
 F 2 "" H 5350 1550 60  0000 C CNN
@@
 F 0 "R70" V 4350 2050 50  0000 C CNN
 F 1 "10K" V 4300 2200 50  0000 C CNN
-F 2 "" V 4230 2200 30  0000 C CNN
+F 2 "Resistors_SMD:R_0603" V 4230 2200 30  0001 C CNN
 F 3 "" H 4300 2200 30  0000 C CNN
 	1    4300 2200
@@
 F 0 "R71" V 4450 2050 50  0000 C CNN
 F 1 "10K" V 4400 2200 50  0000 C CNN
-F 2 "" V 4330 2200 30  0000 C CNN
+F 2 "Resistors_SMD:R_0603" V 4330 2200 30  0001 C CNN
 F 3 "" H 4400 2200 30  0000 C CNN
 	1    4400 2200
@@
 F 0 "R72" V 4550 2050 50  0000 C CNN
 F 1 "10K" V 4500 2200 50  0000 C CNN
-F 2 "" V 4430 2200 30  0000 C CNN
+F 2 "Resistors_SMD:R_0603" V 4430 2200 30  0001 C CNN
 F 3 "" H 4500 2200 30  0000 C CNN
 	1    4500 2200
@@
 F 0 "R73" V 4650 2050 50  0000 C CNN
 F 1 "10K" V 4600 2200 50  0000 C CNN
-F 2 "" V 4530 2200 30  0000 C CNN
+F 2 "Resistors_SMD:R_0603" V 4530 2200 30  0001 C CNN
 F 3 "" H 4600 2200 30  0000 C CNN
 	1    4600 2200
@@
 F 0 "R74" V 4750 2050 50  0000 C CNN
 F 1 "10K" V 4700 2200 50  0000 C CNN
-F 2 "" V 4630 2200 30  0000 C CNN
+F 2 "Resistors_SMD:R_0603" V 4630 2200 30  0001 C CNN
 F 3 "" H 4700 2200 30  0000 C CNN
 	1    4700 2200
@@
 F 0 "R75" V 4850 2050 50  0000 C CNN
 F 1 "10K" V 4800 2200 50  0000 C CNN
-F 2 "" V 4730 2200 30  0000 C CNN
+F 2 "Resistors_SMD:R_0603" V 4730 2200 30  0001 C CNN
 F 3 "" H 4800 2200 30  0000 C CNN
 	1    4800 2200
@@
 F 0 "R76" V 4950 2050 50  0000 C CNN
 F 1 "10K" V 4900 2200 50  0000 C CNN
-F 2 "" V 4830 2200 30  0000 C CNN
+F 2 "Resistors_SMD:R_0603" V 4830 2200 30  0001 C CNN
 F 3 "" H 4900 2200 30  0000 C CNN
 	1    4900 2200
@@
 F 0 "R69" V 4250 4600 50  0000 C CNN
 F 1 "10K" V 4200 4750 50  0000 C CNN
-F 2 "" V 4130 4750 30  0000 C CNN
+F 2 "Resistors_SMD:R_0603" V 4130 4750 30  0001 C CNN
 F 3 "" H 4200 4750 30  0000 C CNN
 	1    4200 4750
@@
 	4200 4450 4200 4600
 $Comp
-L GND #PWR95
+L GND #PWR0100
 U 1 1 56173E31
 P 4200 5050
-F 0 "#PWR95" H 4200 4800 50  0001 C CNN
+F 0 "#PWR0100" H 4200 4800 50  0001 C CNN
 F 1 "GND" H 4200 4900 50  0000 C CNN
 F 2 "" H 4200 5050 60  0000 C CNN
@@
 F 0 "C63" H 5925 2300 50  0000 L CNN
 F 1 "10u/10V/X5R-C5" V 5800 1800 50  0000 L CNN
-F 2 "" H 5938 2050 30  0000 C CNN
+F 2 "" H 5938 2050 30  0001 C CNN
 F 3 "" H 5900 2200 60  0000 C CNN
 	1    5900 2200
@@
 F 0 "C64" H 6525 2300 50  0000 L CNN
 F 1 "10u/16V/X7R-C2" V 6400 1800 50  0000 L CNN
-F 2 "" H 6538 2050 30  0000 C CNN
+F 2 "" H 6538 2050 30  0001 C CNN
 F 3 "" H 6500 2200 60  0000 C CNN
 	1    6500 2200
@@
 $EndComp
 $Comp
-L GND #PWR99
+L GND #PWR0101
 U 1 1 5617463C
 P 6500 2850
-F 0 "#PWR99" H 6500 2600 50  0001 C CNN
+F 0 "#PWR0101" H 6500 2600 50  0001 C CNN
 F 1 "GND" H 6500 2700 50  0000 C CNN
 F 2 "" H 6500 2850 60  0000 C CNN

Commit message: Work on cortex USB connection.
Parts:
- renumbered C63 to C?, C64 to C?, MSD1 to MSD?, R68 to R?, R70 to R?, R71 to R?, R72 to R?, R73 to R?, R74 to R?, R75 to R?, R76 to R?, R69 to R?
Changed lines of the file:
@@
 $EndDescr
 $Comp
-L uSDCARD-H1.85 MSD1
+L uSDCARD-H1.85 MSD?
 U 1 1 56153956
 P 6350 4000
-F 0 "MSD1" H 6600 3300 60  0000 C CNN
+F 0 "MSD?" H 6600 3300 60  0000 C CNN
 F 1 "uSDCARD-H1.85" H 6450 4700 60  0000 C CNN
 F 2 "" H 6350 4000 60  0001 C CNN
@@
 SD1_WP
 $Comp
-L GND #PWR097
+L GND #PWR?
 U 1 1 5617363A
 P 5350 5050
-F 0 "#PWR097" H 5350 4800 50  0001 C CNN
+F 0 "#PWR?" H 5350 4800 50  0001 C CNN
 F 1 "GND" H 5350 4900 50  0000 C CNN
 F 2 "" H 5350 5050 60  0000 C CNN
@@
 $EndComp
 $Comp
-L GND #PWR098
+L GND #PWR?
 U 1 1 5617364F
 P 6100 5050
-F 0 "#PWR098" H 6100 4800 50  0001 C CNN
+F 0 "#PWR?" H 6100 4800 50  0001 C CNN
 F 1 "GND" H 6100 4900 50  0000 C CNN
 F 2 "" H 6100 5050 60  0000 C CNN
@@
 Connection ~ 5350 4550
 $Comp
-L R R68
+L R R?
 U 1 1 561736B3
 P 3950 3850
-F 0 "R68" V 4030 3850 50  0000 C CNN
+F 0 "R?" V 4030 3850 50  0000 C CNN
 F 1 "22" V 3950 3850 50  0000 C CNN
 F 2 "Resistors_SMD:R_0603" V 3880 3850 30  0001 C CNN
@@
 	3800 3850 3450 3850
 $Comp
-L +3V3 #PWR099
+L +3V3 #PWR?
 U 1 1 561737FF
 P 5350 1550
-F 0 "#PWR099" H 5350 1400 50  0001 C CNN
+F 0 "#PWR?" H 5350 1400 50  0001 C CNN
 F 1 "+3V3" H 5350 1690 50  0000 C CNN
 F 2 "" H 5350 1550 60  0000 C CNN
@@
 	5350 3750 5500 3750
 $Comp
-L R R70
+L R R?
 U 1 1 56173C05
 P 4300 2200
-F 0 "R70" V 4350 2050 50  0000 C CNN
+F 0 "R?" V 4350 2050 50  0000 C CNN
 F 1 "10K" V 4300 2200 50  0000 C CNN
 F 2 "Resistors_SMD:R_0603" V 4230 2200 30  0001 C CNN
@@
 $EndComp
 $Comp
-L R R71
+L R R?
 U 1 1 56173C21
 P 4400 2200
-F 0 "R71" V 4450 2050 50  0000 C CNN
+F 0 "R?" V 4450 2050 50  0000 C CNN
 F 1 "10K" V 4400 2200 50  0000 C CNN
 F 2 "Resistors_SMD:R_0603" V 4330 2200 30  0001 C CNN
@@
 $EndComp
 $Comp
-L R R72
+L R R?
 U 1 1 56173C44
 P 4500 2200
-F 0 "R72" V 4550 2050 50  0000 C CNN
+F 0 "R?" V 4550 2050 50  0000 C CNN
 F 1 "10K" V 4500 2200 50  0000 C CNN
 F 2 "Resistors_SMD:R_0603" V 4430 2200 30  0001 C CNN
@@
 $EndComp
 $Comp
-L R R73
+L R R?
 U 1 1 56173C66
 P 4600 2200
-F 0 "R73" V 4650 2050 50  0000 C CNN
+F 0 "R?" V 4650 2050 50  0000 C CNN
 F 1 "10K" V 4600 2200 50  0000 C CNN
 F 2 "Resistors_SMD:R_0603" V 4530 2200 30  0001 C CNN
@@
 $EndComp
 $Comp
-L R R74
+L R R?
 U 1 1 56173C8B
 P 4700 2200
-F 0 "R74" V 4750 2050 50  0000 C CNN
+F 0 "R?" V 4750 2050 50  0000 C CNN
 F 1 "10K" V 4700 2200 50  0000 C CNN
 F 2 "Resistors_SMD:R_0603" V 4630 2200 30  0001 C CNN
@@
 $EndComp
 $Comp
-L R R75
+L R R?
 U 1 1 56173CB3
 P 4800 2200
-F 0 "R75" V 4850 2050 50  0000 C CNN
+F 0 "R?" V 4850 2050 50  0000 C CNN
 F 1 "10K" V 4800 2200 50  0000 C CNN
 F 2 "Resistors_SMD:R_0603" V 4730 2200 30  0001 C CNN
@@
 $EndComp
 $Comp
-L R R76
+L R R?
 U 1 1 56173CDE
 P 4900 2200
-F 0 "R76" V 4950 2050 50  0000 C CNN
+F 0 "R?" V 4950 2050 50  0000 C CNN
 F 1 "10K" V 4900 2200 50  0000 C CNN
 F 2 "Resistors_SMD:R_0603" V 4830 2200 30  0001 C CNN
@@
 $EndComp
 $Comp
-L R R69
+L R R?
 U 1 1 56173D14
 P 4200 4750
-F 0 "R69" V 4250 4600 50  0000 C CNN
+F 0 "R?" V 4250 4600 50  0000 C CNN
 F 1 "10K" V 4200 4750 50  0000 C CNN
 F 2 "Resistors_SMD:R_0603" V 4130 4750 30  0001 C CNN
@@
 	4200 4450 4200 4600
 $Comp
-L GND #PWR0100
+L GND #PWR?
 U 1 1 56173E31
 P 4200 5050
-F 0 "#PWR0100" H 4200 4800 50  0001 C CNN
+F 0 "#PWR?" H 4200 4800 50  0001 C CNN
 F 1 "GND" H 4200 4900 50  0000 C CNN
 F 2 "" H 4200 5050 60  0000 C CNN
@@
 Connection ~ 4900 1850
 $Comp
-L C C63
+L C C?
 U 1 1 5617422F
 P 5900 2200
-F 0 "C63" H 5925 2300 50  0000 L CNN
+F 0 "C?" H 5925 2300 50  0000 L CNN
 F 1 "10u/10V/X5R-C5" V 5800 1800 50  0000 L CNN
 F 2 "" H 5938 2050 30  0001 C CNN
@@
 $EndComp
 $Comp
-L C C64
+L C C?
 U 1 1 561742E8
 P 6500 2200
-F 0 "C64" H 6525 2300 50  0000 L CNN
+F 0 "C?" H 6525 2300 50  0000 L CNN
 F 1 "10u/16V/X7R-C2" V 6400 1800 50  0000 L CNN
 F 2 "" H 6538 2050 30  0001 C CNN
@@
 $EndComp
 $Comp
-L GND #PWR0101
+L GND #PWR?
 U 1 1 5617463C
 P 6500 2850
-F 0 "#PWR0101" H 6500 2600 50  0001 C CNN
+F 0 "#PWR?" H 6500 2600 50  0001 C CNN
 F 1 "GND" H 6500 2700 50  0000 C CNN
 F 2 "" H 6500 2850 60  0000 C CNN
