File: hardware/colibri-v2/gps.sch (KiCad schematic (older format))
At the start: 11 parts

Commit message: Annotated Components
Parts:
- gave numbers to parts that had none: 11
Changed lines of the file:
@@
 $EndDescr
 $Comp
-L R R?
+L R R115
 U 1 1 56139718
 P 4250 3650
-F 0 "R?" V 4200 3800 50  0000 C CNN
+F 0 "R115" V 4200 3800 50  0000 C CNN
 F 1 "22" V 4250 3650 50  0000 C CNN
 F 2 "" V 4180 3650 30  0000 C CNN
@@
 $EndComp
 $Comp
-L LEA-6S U?
+L LEA-6S U16
 U 1 1 56186F54
 P 6400 3950
-F 0 "U?" H 6900 4900 60  0000 C CNN
+F 0 "U16" H 6900 4900 60  0000 C CNN
 F 1 "LEA-6S" H 6800 3000 60  0000 C CNN
 F 2 "" H 6250 4050 60  0000 C CNN
@@
 $EndComp
 $Comp
-L R R?
+L R R116
 U 1 1 561870DD
 P 4250 3750
-F 0 "R?" V 4200 3900 50  0000 C CNN
+F 0 "R116" V 4200 3900 50  0000 C CNN
 F 1 "22" V 4250 3750 50  0000 C CNN
 F 2 "" V 4180 3750 30  0000 C CNN
@@
 	4400 3750 5600 3750
 $Comp
-L GND #PWR?
+L GND #PWR149
 U 1 1 56187100
 P 5350 5300
-F 0 "#PWR?" H 5350 5050 50  0001 C CNN
+F 0 "#PWR149" H 5350 5050 50  0001 C CNN
 F 1 "GND" H 5350 5150 50  0000 C CNN
 F 2 "" H 5350 5300 60  0000 C CNN
@@
 Connection ~ 5350 4750
 $Comp
-L GND #PWR?
+L GND #PWR150
 U 1 1 5618714A
 P 7450 5300
-F 0 "#PWR?" H 7450 5050 50  0001 C CNN
+F 0 "#PWR150" H 7450 5050 50  0001 C CNN
 F 1 "GND" H 7450 5150 50  0000 C CNN
 F 2 "" H 7450 5300 60  0000 C CNN
@@
 NoConn ~ 5600 4150
 $Comp
-L 1575AT43A0040E A?
+L 1575AT43A0040E A1
 U 1 1 561878D5
 P 9000 3050
-F 0 "A?" H 9300 3050 60  0000 C CNN
+F 0 "A1" H 9300 3050 60  0000 C CNN
 F 1 "1575AT43A0040E" H 9650 2950 60  0000 C CNN
 F 2 "" H 9000 3050 60  0000 C CNN
@@
 GPS_RXD(3V3)
 $Comp
-L Q_PMOS_GSD Q?
+L Q_PMOS_GSD Q8
 U 1 1 56187FA4
 P 3500 2000
-F 0 "Q?" H 3500 1850 50  0000 R CNN
+F 0 "Q8" H 3500 1850 50  0000 R CNN
 F 1 "IRLML6402TRPBF" V 3750 2300 50  0000 R CNN
 F 2 "" H 3700 2100 29  0000 C CNN
@@
 $EndComp
 $Comp
-L INDUCTOR L?
+L INDUCTOR L6
 U 1 1 561881F0
 P 4200 3150
-F 0 "L?" V 4150 3150 50  0000 C CNN
+F 0 "L6" V 4150 3150 50  0000 C CNN
 F 1 "60ohm/100MHz/300mA" V 4300 3150 50  0000 C CNN
 F 2 "" H 4200 3150 60  0000 C CNN
@@
 	4500 3150 5600 3150
 $Comp
-L +3V3 #PWR?
+L +3V3 #PWR147
 U 1 1 56188264
 P 3600 1300
-F 0 "#PWR?" H 3600 1150 50  0001 C CNN
+F 0 "#PWR147" H 3600 1150 50  0001 C CNN
 F 1 "+3V3" H 3600 1440 50  0000 C CNN
 F 2 "" H 3600 1300 60  0000 C CNN
@@
 	3600 1300 3600 1800
 $Comp
-L C C?
+L C C87
 U 1 1 561882A0
 P 4950 2000
-F 0 "C?" H 4975 2100 50  0000 L CNN
+F 0 "C87" H 4975 2100 50  0000 L CNN
 F 1 "10u/16V/X5R" V 5000 1400 50  0000 L CNN
 F 2 "" H 4988 1850 30  0000 C CNN
@@
 $EndComp
 $Comp
-L C C?
+L C C88
 U 1 1 561883B9
 P 5200 2000
-F 0 "C?" H 5225 2100 50  0000 L CNN
+F 0 "C88" H 5225 2100 50  0000 L CNN
 F 1 "100n/50V" V 5250 1550 50  0000 L CNN
 F 2 "" H 5238 1850 30  0000 C CNN
@@
 $EndComp
 $Comp
-L C C?
+L C C86
 U 1 1 561884B4
 P 4700 2000
-F 0 "C?" H 4725 2100 50  0000 L CNN
+F 0 "C86" H 4725 2100 50  0000 L CNN
 F 1 "1u/25V/X7R" V 4750 1450 50  0000 L CNN
 F 2 "" H 4738 1850 30  0000 C CNN
@@
 $EndComp
 $Comp
-L GND #PWR?
+L GND #PWR148
 U 1 1 561885FB
 P 4950 1300
-F 0 "#PWR?" H 4950 1050 50  0001 C CNN
+F 0 "#PWR148" H 4950 1050 50  0001 C CNN
 F 1 "GND" H 4950 1150 50  0000 C CNN
 F 2 "" H 4950 1300 60  0000 C CNN
@@
 GPS_PWR_CTRL(3V3)
 $Comp
-L R R?
+L R R113
 U 1 1 5618877E
 P 2650 2000
-F 0 "R?" V 2600 2150 50  0000 C CNN
+F 0 "R113" V 2600 2150 50  0000 C CNN
 F 1 "22" V 2650 2000 50  0000 C CNN
 F 2 "" V 2580 2000 30  0000 C CNN
@@
 $EndComp
 $Comp
-L R R?
+L R R114
 U 1 1 561887E6
 P 3100 1650
-F 0 "R?" V 3050 1800 50  0000 C CNN
+F 0 "R114" V 3050 1800 50  0000 C CNN
 F 1 "100K" V 3100 1650 50  0000 C CNN
 F 2 "" V 3030 1650 30  0000 C CNN
@@
 $EndComp
 $Comp
-L +3V3 #PWR?
+L +3V3 #PWR146
 U 1 1 5618885F
 P 3100 1300
-F 0 "#PWR?" H 3100 1150 50  0001 C CNN
+F 0 "#PWR146" H 3100 1150 50  0001 C CNN
 F 1 "+3V3" H 3100 1440 50  0000 C CNN
 F 2 "" H 3100 1300 60  0000 C CNN

Commit message: Re-annotated schematic
Parts:
- renumbered C86 to C84, C87 to C85, C88 to C86, R113 to R116, R114 to R117, R115 to R118, R116 to R119
Changed lines of the file:
@@
 $EndDescr
 $Comp
-L R R115
+L R R118
 U 1 1 56139718
 P 4250 3650
-F 0 "R115" V 4200 3800 50  0000 C CNN
+F 0 "R118" V 4200 3800 50  0000 C CNN
 F 1 "22" V 4250 3650 50  0000 C CNN
 F 2 "" V 4180 3650 30  0000 C CNN
@@
 $EndComp
 $Comp
-L R R116
+L R R119
 U 1 1 561870DD
 P 4250 3750
-F 0 "R116" V 4200 3900 50  0000 C CNN
+F 0 "R119" V 4200 3900 50  0000 C CNN
 F 1 "22" V 4250 3750 50  0000 C CNN
 F 2 "" V 4180 3750 30  0000 C CNN
@@
 	4400 3750 5600 3750
 $Comp
-L GND #PWR0148
+L GND #PWR147
 U 1 1 56187100
 P 5350 5300
-F 0 "#PWR0148" H 5350 5050 50  0001 C CNN
+F 0 "#PWR147" H 5350 5050 50  0001 C CNN
 F 1 "GND" H 5350 5150 50  0000 C CNN
 F 2 "" H 5350 5300 60  0000 C CNN
@@
 Connection ~ 5350 4750
 $Comp
-L GND #PWR0149
+L GND #PWR148
 U 1 1 5618714A
 P 7450 5300
-F 0 "#PWR0149" H 7450 5050 50  0001 C CNN
+F 0 "#PWR148" H 7450 5050 50  0001 C CNN
 F 1 "GND" H 7450 5150 50  0000 C CNN
 F 2 "" H 7450 5300 60  0000 C CNN
@@
 	4500 3150 5600 3150
 $Comp
-L +3V3 #PWR0150
+L +3V3 #PWR145
 U 1 1 56188264
 P 3600 1300
-F 0 "#PWR0150" H 3600 1150 50  0001 C CNN
+F 0 "#PWR145" H 3600 1150 50  0001 C CNN
 F 1 "+3V3" H 3600 1440 50  0000 C CNN
 F 2 "" H 3600 1300 60  0000 C CNN
@@
 	3600 1300 3600 1800
 $Comp
-L C C87
+L C C85
 U 1 1 561882A0
 P 4950 2000
-F 0 "C87" H 4975 2100 50  0000 L CNN
+F 0 "C85" H 4975 2100 50  0000 L CNN
 F 1 "10u/16V/X5R" V 5000 1400 50  0000 L CNN
 F 2 "" H 4988 1850 30  0000 C CNN
@@
 $EndComp
 $Comp
-L C C88
+L C C86
 U 1 1 561883B9
 P 5200 2000
-F 0 "C88" H 5225 2100 50  0000 L CNN
+F 0 "C86" H 5225 2100 50  0000 L CNN
 F 1 "100n/50V" V 5250 1550 50  0000 L CNN
 F 2 "" H 5238 1850 30  0000 C CNN
@@
 $EndComp
 $Comp
-L C C86
+L C C84
 U 1 1 561884B4
 P 4700 2000
-F 0 "C86" H 4725 2100 50  0000 L CNN
+F 0 "C84" H 4725 2100 50  0000 L CNN
 F 1 "1u/25V/X7R" V 4750 1450 50  0000 L CNN
 F 2 "" H 4738 1850 30  0000 C CNN
@@
 $EndComp
 $Comp
-L GND #PWR0151
+L GND #PWR146
 U 1 1 561885FB
 P 4950 1300
-F 0 "#PWR0151" H 4950 1050 50  0001 C CNN
+F 0 "#PWR146" H 4950 1050 50  0001 C CNN
 F 1 "GND" H 4950 1150 50  0000 C CNN
 F 2 "" H 4950 1300 60  0000 C CNN
@@
 GPS_PWR_CTRL(3V3)
 $Comp
-L R R113
+L R R116
 U 1 1 5618877E
 P 2650 2000
-F 0 "R113" V 2600 2150 50  0000 C CNN
+F 0 "R116" V 2600 2150 50  0000 C CNN
 F 1 "22" V 2650 2000 50  0000 C CNN
 F 2 "" V 2580 2000 30  0000 C CNN
@@
 $EndComp
 $Comp
-L R R114
+L R R117
 U 1 1 561887E6
 P 3100 1650
-F 0 "R114" V 3050 1800 50  0000 C CNN
+F 0 "R117" V 3050 1800 50  0000 C CNN
 F 1 "100K" V 3100 1650 50  0000 C CNN
 F 2 "" V 3030 1650 30  0000 C CNN
@@
 $EndComp
 $Comp
-L +3V3 #PWR0152
+L +3V3 #PWR144
 U 1 1 5618885F
 P 3100 1300
-F 0 "#PWR0152" H 3100 1150 50  0001 C CNN
+F 0 "#PWR144" H 3100 1150 50  0001 C CNN
 F 1 "+3V3" H 3100 1440 50  0000 C CNN
 F 2 "" H 3100 1300 60  0000 C CNN

Commit message: Associated footprints for R and some of the C
Parts:
- R116, R117, R118, R119: footprint (none) -> Resistors_SMD:R_0603
Changed lines of the file:
@@
 F 0 "R118" V 4200 3800 50  0000 C CNN
 F 1 "22" V 4250 3650 50  0000 C CNN
-F 2 "" V 4180 3650 30  0000 C CNN
+F 2 "Resistors_SMD:R_0603" V 4180 3650 30  0001 C CNN
 F 3 "" H 4250 3650 30  0000 C CNN
 	1    4250 3650
@@
 F 0 "U16" H 6900 4900 60  0000 C CNN
 F 1 "LEA-6S" H 6800 3000 60  0000 C CNN
-F 2 "" H 6250 4050 60  0000 C CNN
+F 2 "" H 6250 4050 60  0001 C CNN
 F 3 "" H 6250 4050 60  0000 C CNN
 	1    6400 3950
@@
 F 0 "R119" V 4200 3900 50  0000 C CNN
 F 1 "22" V 4250 3750 50  0000 C CNN
-F 2 "" V 4180 3750 30  0000 C CNN
+F 2 "Resistors_SMD:R_0603" V 4180 3750 30  0001 C CNN
 F 3 "" H 4250 3750 30  0000 C CNN
 	1    4250 3750
@@
 	4400 3750 5600 3750
 $Comp
-L GND #PWR147
+L GND #PWR0146
 U 1 1 56187100
 P 5350 5300
-F 0 "#PWR147" H 5350 5050 50  0001 C CNN
+F 0 "#PWR0146" H 5350 5050 50  0001 C CNN
 F 1 "GND" H 5350 5150 50  0000 C CNN
 F 2 "" H 5350 5300 60  0000 C CNN
@@
 Connection ~ 5350 4750
 $Comp
-L GND #PWR148
+L GND #PWR0147
 U 1 1 5618714A
 P 7450 5300
-F 0 "#PWR148" H 7450 5050 50  0001 C CNN
+F 0 "#PWR0147" H 7450 5050 50  0001 C CNN
 F 1 "GND" H 7450 5150 50  0000 C CNN
 F 2 "" H 7450 5300 60  0000 C CNN
@@
 F 0 "A1" H 9300 3050 60  0000 C CNN
 F 1 "1575AT43A0040E" H 9650 2950 60  0000 C CNN
-F 2 "" H 9000 3050 60  0000 C CNN
+F 2 "" H 9000 3050 60  0001 C CNN
 F 3 "" H 9000 3050 60  0000 C CNN
 	1    9000 3050
@@
 F 0 "Q8" H 3500 1850 50  0000 R CNN
 F 1 "IRLML6402TRPBF" V 3750 2300 50  0000 R CNN
-F 2 "" H 3700 2100 29  0000 C CNN
+F 2 "" H 3700 2100 29  0001 C CNN
 F 3 "" H 3500 2000 60  0000 C CNN
 	1    3500 2000
@@
 F 0 "L6" V 4150 3150 50  0000 C CNN
 F 1 "60ohm/100MHz/300mA" V 4300 3150 50  0000 C CNN
-F 2 "" H 4200 3150 60  0000 C CNN
+F 2 "" H 4200 3150 60  0001 C CNN
 F 3 "" H 4200 3150 60  0000 C CNN
 	1    4200 3150
@@
 	4500 3150 5600 3150
 $Comp
-L +3V3 #PWR145
+L +3V3 #PWR0148
 U 1 1 56188264
 P 3600 1300
-F 0 "#PWR145" H 3600 1150 50  0001 C CNN
+F 0 "#PWR0148" H 3600 1150 50  0001 C CNN
 F 1 "+3V3" H 3600 1440 50  0000 C CNN
 F 2 "" H 3600 1300 60  0000 C CNN
@@
 F 0 "C85" H 4975 2100 50  0000 L CNN
 F 1 "10u/16V/X5R" V 5000 1400 50  0000 L CNN
-F 2 "" H 4988 1850 30  0000 C CNN
+F 2 "" H 4988 1850 30  0001 C CNN
 F 3 "" H 4950 2000 60  0000 C CNN
 	1    4950 2000
@@
 F 0 "C86" H 5225 2100 50  0000 L CNN
 F 1 "100n/50V" V 5250 1550 50  0000 L CNN
-F 2 "" H 5238 1850 30  0000 C CNN
+F 2 "" H 5238 1850 30  0001 C CNN
 F 3 "" H 5200 2000 60  0000 C CNN
 	1    5200 2000
@@
 F 0 "C84" H 4725 2100 50  0000 L CNN
 F 1 "1u/25V/X7R" V 4750 1450 50  0000 L CNN
-F 2 "" H 4738 1850 30  0000 C CNN
+F 2 "" H 4738 1850 30  0001 C CNN
 F 3 "" H 4700 2000 60  0000 C CNN
 	1    4700 2000
@@
 $EndComp
 $Comp
-L GND #PWR146
+L GND #PWR0149
 U 1 1 561885FB
 P 4950 1300
-F 0 "#PWR146" H 4950 1050 50  0001 C CNN
+F 0 "#PWR0149" H 4950 1050 50  0001 C CNN
 F 1 "GND" H 4950 1150 50  0000 C CNN
 F 2 "" H 4950 1300 60  0000 C CNN
@@
 F 0 "R116" V 2600 2150 50  0000 C CNN
 F 1 "22" V 2650 2000 50  0000 C CNN
-F 2 "" V 2580 2000 30  0000 C CNN
+F 2 "Resistors_SMD:R_0603" V 2580 2000 30  0001 C CNN
 F 3 "" H 2650 2000 30  0000 C CNN
 	1    2650 2000
@@
 F 0 "R117" V 3050 1800 50  0000 C CNN
 F 1 "100K" V 3100 1650 50  0000 C CNN
-F 2 "" V 3030 1650 30  0000 C CNN
+F 2 "Resistors_SMD:R_0603" V 3030 1650 30  0001 C CNN
 F 3 "" H 3100 1650 30  0000 C CNN
 	1    3100 1650
@@
 $EndComp
 $Comp
-L +3V3 #PWR144
+L +3V3 #PWR0150
 U 1 1 5618885F
 P 3100 1300
-F 0 "#PWR144" H 3100 1150 50  0001 C CNN
+F 0 "#PWR0150" H 3100 1150 50  0001 C CNN
 F 1 "+3V3" H 3100 1440 50  0000 C CNN
 F 2 "" H 3100 1300 60  0000 C CNN

Commit message: Work on cortex USB connection.
Parts:
- renumbered A1 to A?, C85 to C?, C86 to C?, C84 to C?, L6 to L?, Q8 to Q?, R118 to R?, R119 to R?, R116 to R?, R117 to R?, U16 to U?
Changed lines of the file:
@@
 $EndDescr
 $Comp
-L R R118
+L R R?
 U 1 1 56139718
 P 4250 3650
-F 0 "R118" V 4200 3800 50  0000 C CNN
+F 0 "R?" V 4200 3800 50  0000 C CNN
 F 1 "22" V 4250 3650 50  0000 C CNN
 F 2 "Resistors_SMD:R_0603" V 4180 3650 30  0001 C CNN
@@
 $EndComp
 $Comp
-L LEA-6S U16
+L LEA-6S U?
 U 1 1 56186F54
 P 6400 3950
-F 0 "U16" H 6900 4900 60  0000 C CNN
+F 0 "U?" H 6900 4900 60  0000 C CNN
 F 1 "LEA-6S" H 6800 3000 60  0000 C CNN
 F 2 "" H 6250 4050 60  0001 C CNN
@@
 $EndComp
 $Comp
-L R R119
+L R R?
 U 1 1 561870DD
 P 4250 3750
-F 0 "R119" V 4200 3900 50  0000 C CNN
+F 0 "R?" V 4200 3900 50  0000 C CNN
 F 1 "22" V 4250 3750 50  0000 C CNN
 F 2 "Resistors_SMD:R_0603" V 4180 3750 30  0001 C CNN
@@
 	4400 3750 5600 3750
 $Comp
-L GND #PWR0146
+L GND #PWR?
 U 1 1 56187100
 P 5350 5300
-F 0 "#PWR0146" H 5350 5050 50  0001 C CNN
+F 0 "#PWR?" H 5350 5050 50  0001 C CNN
 F 1 "GND" H 5350 5150 50  0000 C CNN
 F 2 "" H 5350 5300 60  0000 C CNN
@@
 Connection ~ 5350 4750
 $Comp
-L GND #PWR0147
+L GND #PWR?
 U 1 1 5618714A
 P 7450 5300
-F 0 "#PWR0147" H 7450 5050 50  0001 C CNN
+F 0 "#PWR?" H 7450 5050 50  0001 C CNN
 F 1 "GND" H 7450 5150 50  0000 C CNN
 F 2 "" H 7450 5300 60  0000 C CNN
@@
 NoConn ~ 5600 4150
 $Comp
-L 1575AT43A0040E A1
+L 1575AT43A0040E A?
 U 1 1 561878D5
 P 9000 3050
-F 0 "A1" H 9300 3050 60  0000 C CNN
+F 0 "A?" H 9300 3050 60  0000 C CNN
 F 1 "1575AT43A0040E" H 9650 2950 60  0000 C CNN
 F 2 "" H 9000 3050 60  0001 C CNN
@@
 GPS_RXD(3V3)
 $Comp
-L Q_PMOS_GSD Q8
+L Q_PMOS_GSD Q?
 U 1 1 56187FA4
 P 3500 2000
-F 0 "Q8" H 3500 1850 50  0000 R CNN
+F 0 "Q?" H 3500 1850 50  0000 R CNN
 F 1 "IRLML6402TRPBF" V 3750 2300 50  0000 R CNN
 F 2 "" H 3700 2100 29  0001 C CNN
@@
 $EndComp
 $Comp
-L INDUCTOR L6
+L INDUCTOR L?
 U 1 1 561881F0
 P 4200 3150
-F 0 "L6" V 4150 3150 50  0000 C CNN
+F 0 "L?" V 4150 3150 50  0000 C CNN
 F 1 "60ohm/100MHz/300mA" V 4300 3150 50  0000 C CNN
 F 2 "" H 4200 3150 60  0001 C CNN
@@
 	4500 3150 5600 3150
 $Comp
-L +3V3 #PWR0148
+L +3V3 #PWR?
 U 1 1 56188264
 P 3600 1300
-F 0 "#PWR0148" H 3600 1150 50  0001 C CNN
+F 0 "#PWR?" H 3600 1150 50  0001 C CNN
 F 1 "+3V3" H 3600 1440 50  0000 C CNN
 F 2 "" H 3600 1300 60  0000 C CNN
@@
 	3600 1300 3600 1800
 $Comp
-L C C85
+L C C?
 U 1 1 561882A0
 P 4950 2000
-F 0 "C85" H 4975 2100 50  0000 L CNN
+F 0 "C?" H 4975 2100 50  0000 L CNN
 F 1 "10u/16V/X5R" V 5000 1400 50  0000 L CNN
 F 2 "" H 4988 1850 30  0001 C CNN
@@
 $EndComp
 $Comp
-L C C86
+L C C?
 U 1 1 561883B9
 P 5200 2000
-F 0 "C86" H 5225 2100 50  0000 L CNN
+F 0 "C?" H 5225 2100 50  0000 L CNN
 F 1 "100n/50V" V 5250 1550 50  0000 L CNN
 F 2 "" H 5238 1850 30  0001 C CNN
@@
 $EndComp
 $Comp
-L C C84
+L C C?
 U 1 1 561884B4
 P 4700 2000
-F 0 "C84" H 4725 2100 50  0000 L CNN
+F 0 "C?" H 4725 2100 50  0000 L CNN
 F 1 "1u/25V/X7R" V 4750 1450 50  0000 L CNN
 F 2 "" H 4738 1850 30  0001 C CNN
@@
 $EndComp
 $Comp
-L GND #PWR0149
+L GND #PWR?
 U 1 1 561885FB
 P 4950 1300
-F 0 "#PWR0149" H 4950 1050 50  0001 C CNN
+F 0 "#PWR?" H 4950 1050 50  0001 C CNN
 F 1 "GND" H 4950 1150 50  0000 C CNN
 F 2 "" H 4950 1300 60  0000 C CNN
@@
 GPS_PWR_CTRL(3V3)
 $Comp
-L R R116
+L R R?
 U 1 1 5618877E
 P 2650 2000
-F 0 "R116" V 2600 2150 50  0000 C CNN
+F 0 "R?" V 2600 2150 50  0000 C CNN
 F 1 "22" V 2650 2000 50  0000 C CNN
 F 2 "Resistors_SMD:R_0603" V 2580 2000 30  0001 C CNN
@@
 $EndComp
 $Comp
-L R R117
+L R R?
 U 1 1 561887E6
 P 3100 1650
-F 0 "R117" V 3050 1800 50  0000 C CNN
+F 0 "R?" V 3050 1800 50  0000 C CNN
 F 1 "100K" V 3100 1650 50  0000 C CNN
 F 2 "Resistors_SMD:R_0603" V 3030 1650 30  0001 C CNN
@@
 $EndComp
 $Comp
-L +3V3 #PWR0150
+L +3V3 #PWR?
 U 1 1 5618885F
 P 3100 1300
-F 0 "#PWR0150" H 3100 1150 50  0001 C CNN
+F 0 "#PWR?" H 3100 1150 50  0001 C CNN
 F 1 "+3V3" H 3100 1440 50  0000 C CNN
 F 2 "" H 3100 1300 60  0000 C CNN
