File: hardware/colibri-v2/stm32f4_sdram.sch (KiCad schematic (older format))
At the start: 8 parts

Commit message: added wnd_lcd.sch
Changed lines of the file:
@@
 $Descr A4 11693 8268
 encoding utf-8
-Sheet 6 22
+Sheet 6 23
 Title ""
 Date ""
@@
 	5800 3250 6600 3250
 Wire Wire Line
-	5800 4400 6000 4400
-Wire Wire Line
-	6000 4400 6600 4400
+	5800 4400 6600 4400
 Wire Wire Line
 	5800 3800 6000 3800
 Wire Wire Line
-	6000 3800 6000 3900
-Wire Wire Line
-	6000 3900 6000 4000
-Wire Wire Line
-	6000 4000 6000 4100
-Wire Wire Line
-	6000 4100 6000 4200
-Wire Wire Line
-	6000 4200 6000 4300
-Wire Wire Line
-	6000 4300 6000 4400
+	6000 3800 6000 4400
 Connection ~ 6000 4400
 Wire Wire Line
@@
 	5800 4300 6000 4300
 Wire Wire Line
-	3500 4400 3950 4400
-Wire Wire Line
-	3950 4400 4200 4400
+	3500 4400 4200 4400
 Wire Wire Line
 	4200 3800 3950 3800
 Wire Wire Line
-	3950 3800 3950 3900
-Wire Wire Line
-	3950 3900 3950 4000
-Wire Wire Line
-	3950 4000 3950 4100
-Wire Wire Line
-	3950 4100 3950 4200
-Wire Wire Line
-	3950 4200 3950 4300
-Wire Wire Line
-	3950 4300 3950 4400
+	3950 3800 3950 4400
 Connection ~ 3950 4400
 Wire Wire Line
@@
 $EndComp
 Wire Wire Line
-	3400 5250 3400 5350
-Wire Wire Line
-	3400 5350 3400 5600
-Wire Wire Line
-	3400 5350 3700 5350
-Wire Wire Line
-	3700 5350 4000 5350
-Wire Wire Line
-	4000 5350 4300 5350
-Wire Wire Line
-	4300 5350 4600 5350
-Wire Wire Line
-	4600 5350 4900 5350
-Wire Wire Line
-	4900 5350 5200 5350
+	3400 5250 3400 5600
+Wire Wire Line
+	3400 5350 5200 5350
 Wire Wire Line
 	5200 5350 5200 5600
 Connection ~ 3400 5350
 Wire Wire Line
-	3400 5900 3400 6200
-Wire Wire Line
-	3400 6200 3400 6250
-Wire Wire Line
-	3400 6200 3700 6200
-Wire Wire Line
-	3700 6200 4000 6200
-Wire Wire Line
-	4000 6200 4300 6200
-Wire Wire Line
-	4300 6200 4600 6200
-Wire Wire Line
-	4600 6200 4900 6200
-Wire Wire Line
-	4900 6200 5200 6200
+	3400 5900 3400 6250
+Wire Wire Line
+	3400 6200 5200 6200
 Wire Wire Line
 	5200 6200 5200 5900

Commit message: Annotated Components
Parts:
- gave numbers to parts that had none: 8
Changed lines of the file:
@@
 $EndDescr
 $Comp
-L IS42S16400J U?
+L IS42S16400J U4
 U 1 1 55895059
 P 5000 2900
-F 0 "U?" H 5450 4550 60  0000 C CNN
+F 0 "U4" H 5450 4550 60  0000 C CNN
 F 1 "IS42S16400J" H 4800 4550 60  0000 C CNN
 F 2 "" H 5000 3400 60  0000 C CNN
@@
 FMC_SDCKE1
 $Comp
-L GND #PWR?
+L GND #PWR45
 U 1 1 55895A0D
 P 6600 4400
-F 0 "#PWR?" H 6600 4150 50  0001 C CNN
+F 0 "#PWR45" H 6600 4150 50  0001 C CNN
 F 1 "GND" H 6600 4250 50  0000 C CNN
 F 2 "" H 6600 4400 60  0000 C CNN
@@
 $EndComp
 $Comp
-L +3V3 #PWR?
+L +3V3 #PWR44
 U 1 1 55895AE5
 P 3500 4400
-F 0 "#PWR?" H 3500 4250 50  0001 C CNN
+F 0 "#PWR44" H 3500 4250 50  0001 C CNN
 F 1 "+3V3" H 3500 4540 50  0000 C CNN
 F 2 "" H 3500 4400 60  0000 C CNN
@@
 	3950 4300 4200 4300
 $Comp
-L C C?
+L C C42
 U 1 1 55895E59
 P 3400 5750
-F 0 "C?" H 3425 5850 50  0000 L CNN
+F 0 "C42" H 3425 5850 50  0000 L CNN
 F 1 "100nF" H 3425 5650 50  0000 L CNN
 F 2 "" H 3438 5600 30  0000 C CNN
@@
 $EndComp
 $Comp
-L C C?
+L C C43
 U 1 1 55895F29
 P 3700 5750
-F 0 "C?" H 3725 5850 50  0000 L CNN
+F 0 "C43" H 3725 5850 50  0000 L CNN
 F 1 "100nF" H 3725 5650 50  0000 L CNN
 F 2 "" H 3738 5600 30  0000 C CNN
@@
 $EndComp
 $Comp
-L C C?
+L C C44
 U 1 1 55895F4B
 P 4000 5750
-F 0 "C?" H 4025 5850 50  0000 L CNN
+F 0 "C44" H 4025 5850 50  0000 L CNN
 F 1 "100nF" H 4025 5650 50  0000 L CNN
 F 2 "" H 4038 5600 30  0000 C CNN
@@
 $EndComp
 $Comp
-L C C?
+L C C45
 U 1 1 55895F6D
 P 4300 5750
-F 0 "C?" H 4325 5850 50  0000 L CNN
+F 0 "C45" H 4325 5850 50  0000 L CNN
 F 1 "100nF" H 4325 5650 50  0000 L CNN
 F 2 "" H 4338 5600 30  0000 C CNN
@@
 $EndComp
 $Comp
-L C C?
+L C C46
 U 1 1 55895F97
 P 4600 5750
-F 0 "C?" H 4625 5850 50  0000 L CNN
+F 0 "C46" H 4625 5850 50  0000 L CNN
 F 1 "100nF" H 4625 5650 50  0000 L CNN
 F 2 "" H 4638 5600 30  0000 C CNN
@@
 $EndComp
 $Comp
-L C C?
+L C C47
 U 1 1 55895FE3
 P 4900 5750
-F 0 "C?" H 4925 5850 50  0000 L CNN
+F 0 "C47" H 4925 5850 50  0000 L CNN
 F 1 "100nF" H 4925 5650 50  0000 L CNN
 F 2 "" H 4938 5600 30  0000 C CNN
@@
 $EndComp
 $Comp
-L C C?
+L C C48
 U 1 1 5589600B
 P 5200 5750
-F 0 "C?" H 5225 5850 50  0000 L CNN
+F 0 "C48" H 5225 5850 50  0000 L CNN
 F 1 "100nF" H 5225 5650 50  0000 L CNN
 F 2 "" H 5238 5600 30  0000 C CNN
@@
 $EndComp
 $Comp
-L +3V3 #PWR?
+L +3V3 #PWR42
 U 1 1 5589603F
 P 3400 5250
-F 0 "#PWR?" H 3400 5100 50  0001 C CNN
+F 0 "#PWR42" H 3400 5100 50  0001 C CNN
 F 1 "+3V3" H 3400 5390 50  0000 C CNN
 F 2 "" H 3400 5250 60  0000 C CNN
@@
 $EndComp
 $Comp
-L GND #PWR?
+L GND #PWR43
 U 1 1 5589605A
 P 3400 6250
-F 0 "#PWR?" H 3400 6000 50  0001 C CNN
+F 0 "#PWR43" H 3400 6000 50  0001 C CNN
 F 1 "GND" H 3400 6100 50  0000 C CNN
 F 2 "" H 3400 6250 60  0000 C CNN

Commit message: Re-annotated schematic
Parts:
- renumbered C42 to C40, C43 to C41, C44 to C42, C45 to C43, C46 to C44, C47 to C45, C48 to C46
Changed lines of the file:
@@
 FMC_SDCKE1
 $Comp
-L GND #PWR043
+L GND #PWR41
 U 1 1 55895A0D
 P 6600 4400
-F 0 "#PWR043" H 6600 4150 50  0001 C CNN
+F 0 "#PWR41" H 6600 4150 50  0001 C CNN
 F 1 "GND" H 6600 4250 50  0000 C CNN
 F 2 "" H 6600 4400 60  0000 C CNN
@@
 $EndComp
 $Comp
-L +3V3 #PWR044
+L +3V3 #PWR40
 U 1 1 55895AE5
 P 3500 4400
-F 0 "#PWR044" H 3500 4250 50  0001 C CNN
+F 0 "#PWR40" H 3500 4250 50  0001 C CNN
 F 1 "+3V3" H 3500 4540 50  0000 C CNN
 F 2 "" H 3500 4400 60  0000 C CNN
@@
 	3950 4300 4200 4300
 $Comp
-L C C42
+L C C40
 U 1 1 55895E59
 P 3400 5750
-F 0 "C42" H 3425 5850 50  0000 L CNN
+F 0 "C40" H 3425 5850 50  0000 L CNN
 F 1 "100nF" H 3425 5650 50  0000 L CNN
 F 2 "" H 3438 5600 30  0000 C CNN
@@
 $EndComp
 $Comp
-L C C43
+L C C41
 U 1 1 55895F29
 P 3700 5750
-F 0 "C43" H 3725 5850 50  0000 L CNN
+F 0 "C41" H 3725 5850 50  0000 L CNN
 F 1 "100nF" H 3725 5650 50  0000 L CNN
 F 2 "" H 3738 5600 30  0000 C CNN
@@
 $EndComp
 $Comp
-L C C44
+L C C42
 U 1 1 55895F4B
 P 4000 5750
-F 0 "C44" H 4025 5850 50  0000 L CNN
+F 0 "C42" H 4025 5850 50  0000 L CNN
 F 1 "100nF" H 4025 5650 50  0000 L CNN
 F 2 "" H 4038 5600 30  0000 C CNN
@@
 $EndComp
 $Comp
-L C C45
+L C C43
 U 1 1 55895F6D
 P 4300 5750
-F 0 "C45" H 4325 5850 50  0000 L CNN
+F 0 "C43" H 4325 5850 50  0000 L CNN
 F 1 "100nF" H 4325 5650 50  0000 L CNN
 F 2 "" H 4338 5600 30  0000 C CNN
@@
 $EndComp
 $Comp
-L C C46
+L C C44
 U 1 1 55895F97
 P 4600 5750
-F 0 "C46" H 4625 5850 50  0000 L CNN
+F 0 "C44" H 4625 5850 50  0000 L CNN
 F 1 "100nF" H 4625 5650 50  0000 L CNN
 F 2 "" H 4638 5600 30  0000 C CNN
@@
 $EndComp
 $Comp
-L C C47
+L C C45
 U 1 1 55895FE3
 P 4900 5750
-F 0 "C47" H 4925 5850 50  0000 L CNN
+F 0 "C45" H 4925 5850 50  0000 L CNN
 F 1 "100nF" H 4925 5650 50  0000 L CNN
 F 2 "" H 4938 5600 30  0000 C CNN
@@
 $EndComp
 $Comp
-L C C48
+L C C46
 U 1 1 5589600B
 P 5200 5750
-F 0 "C48" H 5225 5850 50  0000 L CNN
+F 0 "C46" H 5225 5850 50  0000 L CNN
 F 1 "100nF" H 5225 5650 50  0000 L CNN
 F 2 "" H 5238 5600 30  0000 C CNN
@@
 $EndComp
 $Comp
-L +3V3 #PWR045
+L +3V3 #PWR38
 U 1 1 5589603F
 P 3400 5250
-F 0 "#PWR045" H 3400 5100 50  0001 C CNN
+F 0 "#PWR38" H 3400 5100 50  0001 C CNN
 F 1 "+3V3" H 3400 5390 50  0000 C CNN
 F 2 "" H 3400 5250 60  0000 C CNN
@@
 $EndComp
 $Comp
-L GND #PWR046
+L GND #PWR39
 U 1 1 5589605A
 P 3400 6250
-F 0 "#PWR046" H 3400 6000 50  0001 C CNN
+F 0 "#PWR39" H 3400 6000 50  0001 C CNN
 F 1 "GND" H 3400 6100 50  0000 C CNN
 F 2 "" H 3400 6250 60  0000 C CNN

Commit message: Associated footprints for R and some of the C
Parts:
- C40, C41, C42, C43, C44, C45, C46: footprint (none) -> Capacitors_SMD:C_0805
Changed lines of the file:
@@
 F 0 "U4" H 5450 4550 60  0000 C CNN
 F 1 "IS42S16400J" H 4800 4550 60  0000 C CNN
-F 2 "" H 5000 3400 60  0000 C CNN
+F 2 "" H 5000 3400 60  0001 C CNN
 F 3 "" H 5000 3400 60  0000 C CNN
 	1    5000 2900
@@
 FMC_SDCKE1
 $Comp
-L GND #PWR41
+L GND #PWR039
 U 1 1 55895A0D
 P 6600 4400
-F 0 "#PWR41" H 6600 4150 50  0001 C CNN
+F 0 "#PWR039" H 6600 4150 50  0001 C CNN
 F 1 "GND" H 6600 4250 50  0000 C CNN
 F 2 "" H 6600 4400 60  0000 C CNN
@@
 $EndComp
 $Comp
-L +3V3 #PWR40
+L +3V3 #PWR040
 U 1 1 55895AE5
 P 3500 4400
-F 0 "#PWR40" H 3500 4250 50  0001 C CNN
+F 0 "#PWR040" H 3500 4250 50  0001 C CNN
 F 1 "+3V3" H 3500 4540 50  0000 C CNN
 F 2 "" H 3500 4400 60  0000 C CNN
@@
 F 0 "C40" H 3425 5850 50  0000 L CNN
 F 1 "100nF" H 3425 5650 50  0000 L CNN
-F 2 "" H 3438 5600 30  0000 C CNN
+F 2 "Capacitors_SMD:C_0805" H 3438 5600 30  0001 C CNN
 F 3 "" H 3400 5750 60  0000 C CNN
 	1    3400 5750
@@
 F 0 "C41" H 3725 5850 50  0000 L CNN
 F 1 "100nF" H 3725 5650 50  0000 L CNN
-F 2 "" H 3738 5600 30  0000 C CNN
+F 2 "Capacitors_SMD:C_0805" H 3738 5600 30  0001 C CNN
 F 3 "" H 3700 5750 60  0000 C CNN
 	1    3700 5750
@@
 F 0 "C42" H 4025 5850 50  0000 L CNN
 F 1 "100nF" H 4025 5650 50  0000 L CNN
-F 2 "" H 4038 5600 30  0000 C CNN
+F 2 "Capacitors_SMD:C_0805" H 4038 5600 30  0001 C CNN
 F 3 "" H 4000 5750 60  0000 C CNN
 	1    4000 5750
@@
 F 0 "C43" H 4325 5850 50  0000 L CNN
 F 1 "100nF" H 4325 5650 50  0000 L CNN
-F 2 "" H 4338 5600 30  0000 C CNN
+F 2 "Capacitors_SMD:C_0805" H 4338 5600 30  0001 C CNN
 F 3 "" H 4300 5750 60  0000 C CNN
 	1    4300 5750
@@
 F 0 "C44" H 4625 5850 50  0000 L CNN
 F 1 "100nF" H 4625 5650 50  0000 L CNN
-F 2 "" H 4638 5600 30  0000 C CNN
+F 2 "Capacitors_SMD:C_0805" H 4638 5600 30  0001 C CNN
 F 3 "" H 4600 5750 60  0000 C CNN
 	1    4600 5750
@@
 F 0 "C45" H 4925 5850 50  0000 L CNN
 F 1 "100nF" H 4925 5650 50  0000 L CNN
-F 2 "" H 4938 5600 30  0000 C CNN
+F 2 "Capacitors_SMD:C_0805" H 4938 5600 30  0001 C CNN
 F 3 "" H 4900 5750 60  0000 C CNN
 	1    4900 5750
@@
 F 0 "C46" H 5225 5850 50  0000 L CNN
 F 1 "100nF" H 5225 5650 50  0000 L CNN
-F 2 "" H 5238 5600 30  0000 C CNN
+F 2 "Capacitors_SMD:C_0805" H 5238 5600 30  0001 C CNN
 F 3 "" H 5200 5750 60  0000 C CNN
 	1    5200 5750
@@
 $EndComp
 $Comp
-L +3V3 #PWR38
+L +3V3 #PWR041
 U 1 1 5589603F
 P 3400 5250
-F 0 "#PWR38" H 3400 5100 50  0001 C CNN
+F 0 "#PWR041" H 3400 5100 50  0001 C CNN
 F 1 "+3V3" H 3400 5390 50  0000 C CNN
 F 2 "" H 3400 5250 60  0000 C CNN
@@
 $EndComp
 $Comp
-L GND #PWR39
+L GND #PWR042
 U 1 1 5589605A
 P 3400 6250
-F 0 "#PWR39" H 3400 6000 50  0001 C CNN
+F 0 "#PWR042" H 3400 6000 50  0001 C CNN
 F 1 "GND" H 3400 6100 50  0000 C CNN
 F 2 "" H 3400 6250 60  0000 C CNN

Commit message: Work on cortex USB connection.
Parts:
- removed C40, C41, C42, C43, C44, C45, C46: 100nF, Capacitors_SMD:C_0805, symbol C
- added C? (x7): 100nF/50V/X7R, Capacitors_SMD:C_0603, symbol C_SMT
- renumbered U4 to U?
Connections:
- net +3V3: now also C?.1, C?.1, C?.1, C?.1, C?.1, C?.1, C?.1
- net GND: now also C?.2, C?.2, C?.2, C?.2, C?.2, C?.2, C?.2

Commit message: Work on wandboard lcd and usb
Changed lines of the file:
@@
 	5800 3250 6600 3250
 Wire Wire Line
-	5800 4400 6000 4400
-Wire Wire Line
-	6000 4400 6600 4400
+	5800 4400 6600 4400
 Wire Wire Line
 	5800 3800 6000 3800
 Wire Wire Line
-	6000 3800 6000 3900
-Wire Wire Line
-	6000 3900 6000 4000
-Wire Wire Line
-	6000 4000 6000 4100
-Wire Wire Line
-	6000 4100 6000 4200
-Wire Wire Line
-	6000 4200 6000 4300
-Wire Wire Line
-	6000 4300 6000 4400
+	6000 3800 6000 4400
 Connection ~ 6000 4400
 Wire Wire Line
@@
 	5800 4300 6000 4300
 Wire Wire Line
-	3500 4400 3950 4400
-Wire Wire Line
-	3950 4400 4200 4400
+	3500 4400 4200 4400
 Wire Wire Line
 	4200 3800 3950 3800
 Wire Wire Line
-	3950 3800 3950 3900
-Wire Wire Line
-	3950 3900 3950 4000
-Wire Wire Line
-	3950 4000 3950 4100
-Wire Wire Line
-	3950 4100 3950 4200
-Wire Wire Line
-	3950 4200 3950 4300
-Wire Wire Line
-	3950 4300 3950 4400
+	3950 3800 3950 4400
 Connection ~ 3950 4400
 Wire Wire Line
@@
 $EndComp
 Wire Wire Line
-	2400 5250 2400 5350
+	2400 5250 2400 5600
 Wire Wire Line
-	2400 5350 2400 5600
-Wire Wire Line
-	2400 5350 3200 5350
-Wire Wire Line
-	3200 5350 4000 5350
-Wire Wire Line
-	4000 5350 4800 5350
-Wire Wire Line
-	4800 5350 5600 5350
-Wire Wire Line
-	5600 5350 6400 5350
-Wire Wire Line
-	6400 5350 7200 5350
+	2400 5350 7200 5350
 Wire Wire Line
 	7200 5350 7200 5600
 Connection ~ 2400 5350
 Wire Wire Line
-	2400 5900 2400 6200
+	2400 5900 2400 6250
 Wire Wire Line
-	2400 6200 2400 6250
-Wire Wire Line
-	2400 6200 3200 6200
-Wire Wire Line
-	3200 6200 4000 6200
-Wire Wire Line
-	4000 6200 4800 6200
-Wire Wire Line
-	4800 6200 5600 6200
-Wire Wire Line
-	5600 6200 6400 6200
-Wire Wire Line
-	6400 6200 7200 6200
+	2400 6200 7200 6200
 Wire Wire Line
 	7200 6200 7200 5900
