File: hardware/colibri-v2/wb_ftdi_interface.sch (KiCad schematic (older format))
At the start: 12 parts

Commit message: Annotated Components
Parts:
- gave numbers to parts that had none: 12
Changed lines of the file:
@@
 $EndDescr
 $Comp
-L FT232RL U?
+L FT232RL U8
 U 1 1 560A13A8
 P 7000 4150
-F 0 "U?" H 7350 5200 60  0000 C CNN
+F 0 "U8" H 7350 5200 60  0000 C CNN
 F 1 "FT232RL" H 6750 3100 60  0000 C CNN
 F 2 "" H 7000 4150 60  0000 C CNN
@@
 $EndComp
 $Comp
-L USB_B P?
+L USB_B P7
 U 1 1 560A13AF
 P 1750 3550
-F 0 "P?" H 1950 3350 50  0000 C CNN
+F 0 "P7" H 1950 3350 50  0000 C CNN
 F 1 "USB_B" H 1700 3750 50  0000 C CNN
 F 2 "" V 1700 3450 60  0000 C CNN
@@
 $EndComp
 $Comp
-L INDUCTOR L?
+L INDUCTOR L3
 U 1 1 560A13B6
 P 3600 3350
-F 0 "L?" V 3550 3350 50  0000 C CNN
+F 0 "L3" V 3550 3350 50  0000 C CNN
 F 1 "INDUCTOR" V 3700 3350 50  0000 C CNN
 F 2 "" H 3600 3350 60  0000 C CNN
@@
 	2050 3550 6300 3550
 $Comp
-L GND #PWR?
+L GND #PWR85
 U 1 1 560A13C1
 P 6100 5350
-F 0 "#PWR?" H 6100 5100 50  0001 C CNN
+F 0 "#PWR85" H 6100 5100 50  0001 C CNN
 F 1 "GND" H 6100 5200 50  0000 C CNN
 F 2 "" H 6100 5350 60  0000 C CNN
@@
 Connection ~ 6100 5050
 $Comp
-L C C?
+L C C63
 U 1 1 560A13D1
 P 5700 4950
-F 0 "C?" H 5725 5050 50  0000 L CNN
+F 0 "C63" H 5725 5050 50  0000 L CNN
 F 1 "100nF" H 5725 4850 50  0000 L CNN
 F 2 "" H 5738 4800 30  0000 C CNN
@@
 	5700 4550 5700 4800
 $Comp
-L GND #PWR?
+L GND #PWR83
 U 1 1 560A13DA
 P 5700 5350
-F 0 "#PWR?" H 5700 5100 50  0001 C CNN
+F 0 "#PWR83" H 5700 5100 50  0001 C CNN
 F 1 "GND" H 5700 5200 50  0000 C CNN
 F 2 "" H 5700 5350 60  0000 C CNN
@@
 	5700 5100 5700 5350
 $Comp
-L +3V3 #PWR?
+L +3V3 #PWR84
 U 1 1 560A13E1
 P 6100 2350
-F 0 "#PWR?" H 6100 2200 50  0001 C CNN
+F 0 "#PWR84" H 6100 2200 50  0001 C CNN
 F 1 "+3V3" H 6100 2490 50  0000 C CNN
 F 2 "" H 6100 2350 60  0000 C CNN
@@
 $EndComp
 $Comp
-L C C?
+L C C62
 U 1 1 560A13E7
 P 5700 2750
-F 0 "C?" H 5725 2850 50  0000 L CNN
+F 0 "C62" H 5725 2850 50  0000 L CNN
 F 1 "100nF" H 5725 2650 50  0000 L CNN
 F 2 "" H 5738 2600 30  0000 C CNN
@@
 $EndComp
 $Comp
-L GND #PWR?
+L GND #PWR82
 U 1 1 560A13EE
 P 5700 2350
-F 0 "#PWR?" H 5700 2100 50  0001 C CNN
+F 0 "#PWR82" H 5700 2100 50  0001 C CNN
 F 1 "GND" H 5700 2200 50  0000 C CNN
 F 2 "" H 5700 2350 60  0000 C CNN
@@
 	5700 2900 5700 3250
 $Comp
-L C C?
+L C C61
 U 1 1 560A13F6
 P 5300 2750
-F 0 "C?" H 5325 2850 50  0000 L CNN
+F 0 "C61" H 5325 2850 50  0000 L CNN
 F 1 "10uF" H 5325 2650 50  0000 L CNN
 F 2 "" H 5338 2600 30  0000 C CNN
@@
 $EndComp
 $Comp
-L GND #PWR?
+L GND #PWR81
 U 1 1 560A13FD
 P 5300 2350
-F 0 "#PWR?" H 5300 2100 50  0001 C CNN
+F 0 "#PWR81" H 5300 2100 50  0001 C CNN
 F 1 "GND" H 5300 2200 50  0000 C CNN
 F 2 "" H 5300 2350 60  0000 C CNN
@@
 Connection ~ 5700 3250
 $Comp
-L C C?
+L C C59
 U 1 1 560A1406
 P 2400 2750
-F 0 "C?" H 2425 2850 50  0000 L CNN
+F 0 "C59" H 2425 2850 50  0000 L CNN
 F 1 "10uF" H 2425 2650 50  0000 L CNN
 F 2 "" H 2438 2600 30  0000 C CNN
@@
 $EndComp
 $Comp
-L C C?
+L C C60
 U 1 1 560A140D
 P 4900 2750
-F 0 "C?" H 4925 2850 50  0000 L CNN
+F 0 "C60" H 4925 2850 50  0000 L CNN
 F 1 "100nF" H 4925 2650 50  0000 L CNN
 F 2 "" H 4938 2600 30  0000 C CNN
@@
 $EndComp
 $Comp
-L GND #PWR?
+L GND #PWR80
 U 1 1 560A1414
 P 4900 2350
-F 0 "#PWR?" H 4900 2100 50  0001 C CNN
+F 0 "#PWR80" H 4900 2100 50  0001 C CNN
 F 1 "GND" H 4900 2200 50  0000 C CNN
 F 2 "" H 4900 2350 60  0000 C CNN
@@
 $EndComp
 $Comp
-L GND #PWR?
+L GND #PWR78
 U 1 1 560A141A
 P 2400 2350
-F 0 "#PWR?" H 2400 2100 50  0001 C CNN
+F 0 "#PWR78" H 2400 2100 50  0001 C CNN
 F 1 "GND" H 2400 2200 50  0000 C CNN
 F 2 "" H 2400 2350 60  0000 C CNN
@@
 Connection ~ 2400 3350
 $Comp
-L GND #PWR?
+L GND #PWR79
 U 1 1 560A1426
 P 2400 5350
-F 0 "#PWR?" H 2400 5100 50  0001 C CNN
+F 0 "#PWR79" H 2400 5100 50  0001 C CNN
 F 1 "GND" H 2400 5200 50  0000 C CNN
 F 2 "" H 2400 5350 60  0000 C CNN
@@
 	2400 3650 2400 5350
 $Comp
-L GND #PWR?
+L GND #PWR77
 U 1 1 560A142E
 P 1650 5350
-F 0 "#PWR?" H 1650 5100 50  0001 C CNN
+F 0 "#PWR77" H 1650 5100 50  0001 C CNN
 F 1 "GND" H 1650 5200 50  0000 C CNN
 F 2 "" H 1650 5350 60  0000 C CNN
@@
 	7700 3950 9250 3950
 $Comp
-L LED D?
+L LED D11
 U 1 1 560A1448
 P 9000 4250
-F 0 "D?" H 9000 4350 50  0000 C CNN
+F 0 "D11" H 9000 4350 50  0000 C CNN
 F 1 "GREEN" H 9000 4150 50  0000 C CNN
 F 2 "" H 9000 4250 60  0000 C CNN
@@
 $EndComp
 $Comp
-L R R?
+L R R57
 U 1 1 560A144F
 P 8450 4250
-F 0 "R?" V 8400 4450 50  0000 C CNN
+F 0 "R57" V 8400 4450 50  0000 C CNN
 F 1 "270" V 8450 4250 50  0000 C CNN
 F 2 "" V 8380 4250 30  0000 C CNN
@@
 $EndComp
 $Comp
-L +3V3 #PWR?
+L +3V3 #PWR86
 U 1 1 560A1456
 P 9400 4250
-F 0 "#PWR?" H 9400 4100 50  0001 C CNN
+F 0 "#PWR86" H 9400 4100 50  0001 C CNN
 F 1 "+3V3" H 9400 4390 50  0000 C CNN
 F 2 "" H 9400 4250 60  0000 C CNN
@@
 	9200 4250 9400 4250
 $Comp
-L LED D?
+L LED D12
 U 1 1 560A145E
 P 9000 4600
-F 0 "D?" H 9000 4700 50  0000 C CNN
+F 0 "D12" H 9000 4700 50  0000 C CNN
 F 1 "RED" H 9000 4500 50  0000 C CNN
 F 2 "" H 9000 4600 60  0000 C CNN
@@
 $EndComp
 $Comp
-L R R?
+L R R58
 U 1 1 560A1465
 P 8450 4600
-F 0 "R?" V 8400 4800 50  0000 C CNN
+F 0 "R58" V 8400 4800 50  0000 C CNN
 F 1 "270" V 8450 4600 50  0000 C CNN
 F 2 "" V 8380 4600 30  0000 C CNN
@@
 $EndComp
 $Comp
-L +3V3 #PWR?
+L +3V3 #PWR87
 U 1 1 560A146C
 P 9400 4600
-F 0 "#PWR?" H 9400 4450 50  0001 C CNN
+F 0 "#PWR87" H 9400 4450 50  0001 C CNN
 F 1 "+3V3" H 9400 4740 50  0000 C CNN
 F 2 "" H 9400 4600 60  0000 C CNN

Commit message: Re-annotated schematic
Parts:
- renumbered C59 to C57, C60 to C58, C61 to C59, C62 to C60, C63 to C61, R57 to R58, R58 to R59
Changed lines of the file:
@@
 	2050 3550 6300 3550
 $Comp
-L GND #PWR079
+L GND #PWR82
 U 1 1 560A13C1
 P 6100 5350
-F 0 "#PWR079" H 6100 5100 50  0001 C CNN
+F 0 "#PWR82" H 6100 5100 50  0001 C CNN
 F 1 "GND" H 6100 5200 50  0000 C CNN
 F 2 "" H 6100 5350 60  0000 C CNN
@@
 Connection ~ 6100 5050
 $Comp
-L C C63
+L C C61
 U 1 1 560A13D1
 P 5700 4950
-F 0 "C63" H 5725 5050 50  0000 L CNN
+F 0 "C61" H 5725 5050 50  0000 L CNN
 F 1 "100nF" H 5725 4850 50  0000 L CNN
 F 2 "" H 5738 4800 30  0000 C CNN
@@
 	5700 4550 5700 4800
 $Comp
-L GND #PWR080
+L GND #PWR80
 U 1 1 560A13DA
 P 5700 5350
-F 0 "#PWR080" H 5700 5100 50  0001 C CNN
+F 0 "#PWR80" H 5700 5100 50  0001 C CNN
 F 1 "GND" H 5700 5200 50  0000 C CNN
 F 2 "" H 5700 5350 60  0000 C CNN
@@
 	5700 5100 5700 5350
 $Comp
-L +3V3 #PWR081
+L +3V3 #PWR81
 U 1 1 560A13E1
 P 6100 2350
-F 0 "#PWR081" H 6100 2200 50  0001 C CNN
+F 0 "#PWR81" H 6100 2200 50  0001 C CNN
 F 1 "+3V3" H 6100 2490 50  0000 C CNN
 F 2 "" H 6100 2350 60  0000 C CNN
@@
 $EndComp
 $Comp
-L C C62
+L C C60
 U 1 1 560A13E7
 P 5700 2750
-F 0 "C62" H 5725 2850 50  0000 L CNN
+F 0 "C60" H 5725 2850 50  0000 L CNN
 F 1 "100nF" H 5725 2650 50  0000 L CNN
 F 2 "" H 5738 2600 30  0000 C CNN
@@
 $EndComp
 $Comp
-L GND #PWR082
+L GND #PWR79
 U 1 1 560A13EE
 P 5700 2350
-F 0 "#PWR082" H 5700 2100 50  0001 C CNN
+F 0 "#PWR79" H 5700 2100 50  0001 C CNN
 F 1 "GND" H 5700 2200 50  0000 C CNN
 F 2 "" H 5700 2350 60  0000 C CNN
@@
 	5700 2900 5700 3250
 $Comp
-L C C61
+L C C59
 U 1 1 560A13F6
 P 5300 2750
-F 0 "C61" H 5325 2850 50  0000 L CNN
+F 0 "C59" H 5325 2850 50  0000 L CNN
 F 1 "10uF" H 5325 2650 50  0000 L CNN
 F 2 "" H 5338 2600 30  0000 C CNN
@@
 $EndComp
 $Comp
-L GND #PWR083
+L GND #PWR78
 U 1 1 560A13FD
 P 5300 2350
-F 0 "#PWR083" H 5300 2100 50  0001 C CNN
+F 0 "#PWR78" H 5300 2100 50  0001 C CNN
 F 1 "GND" H 5300 2200 50  0000 C CNN
 F 2 "" H 5300 2350 60  0000 C CNN
@@
 Connection ~ 5700 3250
 $Comp
-L C C59
+L C C57
 U 1 1 560A1406
 P 2400 2750
-F 0 "C59" H 2425 2850 50  0000 L CNN
+F 0 "C57" H 2425 2850 50  0000 L CNN
 F 1 "10uF" H 2425 2650 50  0000 L CNN
 F 2 "" H 2438 2600 30  0000 C CNN
@@
 $EndComp
 $Comp
-L C C60
+L C C58
 U 1 1 560A140D
 P 4900 2750
-F 0 "C60" H 4925 2850 50  0000 L CNN
+F 0 "C58" H 4925 2850 50  0000 L CNN
 F 1 "100nF" H 4925 2650 50  0000 L CNN
 F 2 "" H 4938 2600 30  0000 C CNN
@@
 $EndComp
 $Comp
-L GND #PWR084
+L GND #PWR77
 U 1 1 560A1414
 P 4900 2350
-F 0 "#PWR084" H 4900 2100 50  0001 C CNN
+F 0 "#PWR77" H 4900 2100 50  0001 C CNN
 F 1 "GND" H 4900 2200 50  0000 C CNN
 F 2 "" H 4900 2350 60  0000 C CNN
@@
 $EndComp
 $Comp
-L GND #PWR085
+L GND #PWR75
 U 1 1 560A141A
 P 2400 2350
-F 0 "#PWR085" H 2400 2100 50  0001 C CNN
+F 0 "#PWR75" H 2400 2100 50  0001 C CNN
 F 1 "GND" H 2400 2200 50  0000 C CNN
 F 2 "" H 2400 2350 60  0000 C CNN
@@
 Connection ~ 2400 3350
 $Comp
-L GND #PWR086
+L GND #PWR76
 U 1 1 560A1426
 P 2400 5350
-F 0 "#PWR086" H 2400 5100 50  0001 C CNN
+F 0 "#PWR76" H 2400 5100 50  0001 C CNN
 F 1 "GND" H 2400 5200 50  0000 C CNN
 F 2 "" H 2400 5350 60  0000 C CNN
@@
 	2400 3650 2400 5350
 $Comp
-L GND #PWR087
+L GND #PWR74
 U 1 1 560A142E
 P 1650 5350
-F 0 "#PWR087" H 1650 5100 50  0001 C CNN
+F 0 "#PWR74" H 1650 5100 50  0001 C CNN
 F 1 "GND" H 1650 5200 50  0000 C CNN
 F 2 "" H 1650 5350 60  0000 C CNN
@@
 $EndComp
 $Comp
-L R R57
+L R R58
 U 1 1 560A144F
 P 8450 4250
-F 0 "R57" V 8400 4450 50  0000 C CNN
+F 0 "R58" V 8400 4450 50  0000 C CNN
 F 1 "270" V 8450 4250 50  0000 C CNN
 F 2 "" V 8380 4250 30  0000 C CNN
@@
 $EndComp
 $Comp
-L +3V3 #PWR088
+L +3V3 #PWR83
 U 1 1 560A1456
 P 9400 4250
-F 0 "#PWR088" H 9400 4100 50  0001 C CNN
+F 0 "#PWR83" H 9400 4100 50  0001 C CNN
 F 1 "+3V3" H 9400 4390 50  0000 C CNN
 F 2 "" H 9400 4250 60  0000 C CNN
@@
 $EndComp
 $Comp
-L R R58
+L R R59
 U 1 1 560A1465
 P 8450 4600
-F 0 "R58" V 8400 4800 50  0000 C CNN
+F 0 "R59" V 8400 4800 50  0000 C CNN
 F 1 "270" V 8450 4600 50  0000 C CNN
 F 2 "" V 8380 4600 30  0000 C CNN
@@
 $EndComp
 $Comp
-L +3V3 #PWR089
+L +3V3 #PWR84
 U 1 1 560A146C
 P 9400 4600
-F 0 "#PWR089" H 9400 4450 50  0001 C CNN
+F 0 "#PWR84" H 9400 4450 50  0001 C CNN
 F 1 "+3V3" H 9400 4740 50  0000 C CNN
 F 2 "" H 9400 4600 60  0000 C CNN

Commit message: Associated footprints for R and some of the C
Parts:
- C57, C58, C59, C60, C61: footprint (none) -> Capacitors_SMD:C_0805
- R58, R59: footprint (none) -> Resistors_SMD:R_0603
Changed lines of the file:
@@
 F 0 "U8" H 7350 5200 60  0000 C CNN
 F 1 "FT232RL" H 6750 3100 60  0000 C CNN
-F 2 "" H 7000 4150 60  0000 C CNN
+F 2 "" H 7000 4150 60  0001 C CNN
 F 3 "" H 7000 4150 60  0000 C CNN
 	1    7000 4150
@@
 F 0 "P7" H 1950 3350 50  0000 C CNN
 F 1 "USB_B" H 1700 3750 50  0000 C CNN
-F 2 "" V 1700 3450 60  0000 C CNN
+F 2 "" V 1700 3450 60  0001 C CNN
 F 3 "" V 1700 3450 60  0000 C CNN
 	1    1750 3550
@@
 F 0 "L3" V 3550 3350 50  0000 C CNN
 F 1 "INDUCTOR" V 3700 3350 50  0000 C CNN
-F 2 "" H 3600 3350 60  0000 C CNN
+F 2 "" H 3600 3350 60  0001 C CNN
 F 3 "" H 3600 3350 60  0000 C CNN
 	1    3600 3350
@@
 	2050 3550 6300 3550
 $Comp
-L GND #PWR82
+L GND #PWR076
 U 1 1 560A13C1
 P 6100 5350
-F 0 "#PWR82" H 6100 5100 50  0001 C CNN
+F 0 "#PWR076" H 6100 5100 50  0001 C CNN
 F 1 "GND" H 6100 5200 50  0000 C CNN
 F 2 "" H 6100 5350 60  0000 C CNN
@@
 F 0 "C61" H 5725 5050 50  0000 L CNN
 F 1 "100nF" H 5725 4850 50  0000 L CNN
-F 2 "" H 5738 4800 30  0000 C CNN
+F 2 "Capacitors_SMD:C_0805" H 5738 4800 30  0001 C CNN
 F 3 "" H 5700 4950 60  0000 C CNN
 	1    5700 4950
@@
 	5700 4550 5700 4800
 $Comp
-L GND #PWR80
+L GND #PWR077
 U 1 1 560A13DA
 P 5700 5350
-F 0 "#PWR80" H 5700 5100 50  0001 C CNN
+F 0 "#PWR077" H 5700 5100 50  0001 C CNN
 F 1 "GND" H 5700 5200 50  0000 C CNN
 F 2 "" H 5700 5350 60  0000 C CNN
@@
 	5700 5100 5700 5350
 $Comp
-L +3V3 #PWR81
+L +3V3 #PWR078
 U 1 1 560A13E1
 P 6100 2350
-F 0 "#PWR81" H 6100 2200 50  0001 C CNN
+F 0 "#PWR078" H 6100 2200 50  0001 C CNN
 F 1 "+3V3" H 6100 2490 50  0000 C CNN
 F 2 "" H 6100 2350 60  0000 C CNN
@@
 F 0 "C60" H 5725 2850 50  0000 L CNN
 F 1 "100nF" H 5725 2650 50  0000 L CNN
-F 2 "" H 5738 2600 30  0000 C CNN
+F 2 "Capacitors_SMD:C_0805" H 5738 2600 30  0001 C CNN
 F 3 "" H 5700 2750 60  0000 C CNN
 	1    5700 2750
@@
 $EndComp
 $Comp
-L GND #PWR79
+L GND #PWR079
 U 1 1 560A13EE
 P 5700 2350
-F 0 "#PWR79" H 5700 2100 50  0001 C CNN
+F 0 "#PWR079" H 5700 2100 50  0001 C CNN
 F 1 "GND" H 5700 2200 50  0000 C CNN
 F 2 "" H 5700 2350 60  0000 C CNN
@@
 F 0 "C59" H 5325 2850 50  0000 L CNN
 F 1 "10uF" H 5325 2650 50  0000 L CNN
-F 2 "" H 5338 2600 30  0000 C CNN
+F 2 "Capacitors_SMD:C_0805" H 5338 2600 30  0001 C CNN
 F 3 "" H 5300 2750 60  0000 C CNN
 	1    5300 2750
@@
 $EndComp
 $Comp
-L GND #PWR78
+L GND #PWR080
 U 1 1 560A13FD
 P 5300 2350
-F 0 "#PWR78" H 5300 2100 50  0001 C CNN
+F 0 "#PWR080" H 5300 2100 50  0001 C CNN
 F 1 "GND" H 5300 2200 50  0000 C CNN
 F 2 "" H 5300 2350 60  0000 C CNN
@@
 F 0 "C57" H 2425 2850 50  0000 L CNN
 F 1 "10uF" H 2425 2650 50  0000 L CNN
-F 2 "" H 2438 2600 30  0000 C CNN
+F 2 "Capacitors_SMD:C_0805" H 2438 2600 30  0001 C CNN
 F 3 "" H 2400 2750 60  0000 C CNN
 	1    2400 2750
@@
 F 0 "C58" H 4925 2850 50  0000 L CNN
 F 1 "100nF" H 4925 2650 50  0000 L CNN
-F 2 "" H 4938 2600 30  0000 C CNN
+F 2 "Capacitors_SMD:C_0805" H 4938 2600 30  0001 C CNN
 F 3 "" H 4900 2750 60  0000 C CNN
 	1    4900 2750
@@
 $EndComp
 $Comp
-L GND #PWR77
+L GND #PWR081
 U 1 1 560A1414
 P 4900 2350
-F 0 "#PWR77" H 4900 2100 50  0001 C CNN
+F 0 "#PWR081" H 4900 2100 50  0001 C CNN
 F 1 "GND" H 4900 2200 50  0000 C CNN
 F 2 "" H 4900 2350 60  0000 C CNN
@@
 $EndComp
 $Comp
-L GND #PWR75
+L GND #PWR082
 U 1 1 560A141A
 P 2400 2350
-F 0 "#PWR75" H 2400 2100 50  0001 C CNN
+F 0 "#PWR082" H 2400 2100 50  0001 C CNN
 F 1 "GND" H 2400 2200 50  0000 C CNN
 F 2 "" H 2400 2350 60  0000 C CNN
@@
 Connection ~ 2400 3350
 $Comp
-L GND #PWR76
+L GND #PWR083
 U 1 1 560A1426
 P 2400 5350
-F 0 "#PWR76" H 2400 5100 50  0001 C CNN
+F 0 "#PWR083" H 2400 5100 50  0001 C CNN
 F 1 "GND" H 2400 5200 50  0000 C CNN
 F 2 "" H 2400 5350 60  0000 C CNN
@@
 	2400 3650 2400 5350
 $Comp
-L GND #PWR74
+L GND #PWR084
 U 1 1 560A142E
 P 1650 5350
-F 0 "#PWR74" H 1650 5100 50  0001 C CNN
+F 0 "#PWR084" H 1650 5100 50  0001 C CNN
 F 1 "GND" H 1650 5200 50  0000 C CNN
 F 2 "" H 1650 5350 60  0000 C CNN
@@
 F 0 "D11" H 9000 4350 50  0000 C CNN
 F 1 "GREEN" H 9000 4150 50  0000 C CNN
-F 2 "" H 9000 4250 60  0000 C CNN
+F 2 "" H 9000 4250 60  0001 C CNN
 F 3 "" H 9000 4250 60  0000 C CNN
 	1    9000 4250
@@
 F 0 "R58" V 8400 4450 50  0000 C CNN
 F 1 "270" V 8450 4250 50  0000 C CNN
-F 2 "" V 8380 4250 30  0000 C CNN
+F 2 "Resistors_SMD:R_0603" V 8380 4250 30  0001 C CNN
 F 3 "" H 8450 4250 30  0000 C CNN
 	1    8450 4250
@@
 $EndComp
 $Comp
-L +3V3 #PWR83
+L +3V3 #PWR085
 U 1 1 560A1456
 P 9400 4250
-F 0 "#PWR83" H 9400 4100 50  0001 C CNN
+F 0 "#PWR085" H 9400 4100 50  0001 C CNN
 F 1 "+3V3" H 9400 4390 50  0000 C CNN
 F 2 "" H 9400 4250 60  0000 C CNN
@@
 F 0 "D12" H 9000 4700 50  0000 C CNN
 F 1 "RED" H 9000 4500 50  0000 C CNN
-F 2 "" H 9000 4600 60  0000 C CNN
+F 2 "" H 9000 4600 60  0001 C CNN
 F 3 "" H 9000 4600 60  0000 C CNN
 	1    9000 4600
@@
 F 0 "R59" V 8400 4800 50  0000 C CNN
 F 1 "270" V 8450 4600 50  0000 C CNN
-F 2 "" V 8380 4600 30  0000 C CNN
+F 2 "Resistors_SMD:R_0603" V 8380 4600 30  0001 C CNN
 F 3 "" H 8450 4600 30  0000 C CNN
 	1    8450 4600
@@
 $EndComp
 $Comp
-L +3V3 #PWR84
+L +3V3 #PWR086
 U 1 1 560A146C
 P 9400 4600
-F 0 "#PWR84" H 9400 4450 50  0001 C CNN
+F 0 "#PWR086" H 9400 4450 50  0001 C CNN
 F 1 "+3V3" H 9400 4740 50  0000 C CNN
 F 2 "" H 9400 4600 60  0000 C CNN

Commit message: Work on cortex USB connection.
Parts:
- renumbered C61 to C?, C60 to C?, C59 to C?, C57 to C?, C58 to C?, D11 to D?, D12 to D?, L3 to L?, P7 to P?, R58 to R?, R59 to R?, U8 to U?
Changed lines of the file:
@@
 $EndDescr
 $Comp
-L FT232RL U8
+L FT232RL U?
 U 1 1 560A13A8
 P 7000 4150
-F 0 "U8" H 7350 5200 60  0000 C CNN
+F 0 "U?" H 7350 5200 60  0000 C CNN
 F 1 "FT232RL" H 6750 3100 60  0000 C CNN
 F 2 "" H 7000 4150 60  0001 C CNN
@@
 $EndComp
 $Comp
-L USB_B P7
+L USB_B P?
 U 1 1 560A13AF
 P 1750 3550
-F 0 "P7" H 1950 3350 50  0000 C CNN
+F 0 "P?" H 1950 3350 50  0000 C CNN
 F 1 "USB_B" H 1700 3750 50  0000 C CNN
 F 2 "" V 1700 3450 60  0001 C CNN
@@
 $EndComp
 $Comp
-L INDUCTOR L3
+L INDUCTOR L?
 U 1 1 560A13B6
 P 3600 3350
-F 0 "L3" V 3550 3350 50  0000 C CNN
+F 0 "L?" V 3550 3350 50  0000 C CNN
 F 1 "INDUCTOR" V 3700 3350 50  0000 C CNN
 F 2 "" H 3600 3350 60  0001 C CNN
@@
 	2050 3550 6300 3550
 $Comp
-L GND #PWR076
+L GND #PWR?
 U 1 1 560A13C1
 P 6100 5350
-F 0 "#PWR076" H 6100 5100 50  0001 C CNN
+F 0 "#PWR?" H 6100 5100 50  0001 C CNN
 F 1 "GND" H 6100 5200 50  0000 C CNN
 F 2 "" H 6100 5350 60  0000 C CNN
@@
 Connection ~ 6100 5050
 $Comp
-L C C61
+L C C?
 U 1 1 560A13D1
 P 5700 4950
-F 0 "C61" H 5725 5050 50  0000 L CNN
+F 0 "C?" H 5725 5050 50  0000 L CNN
 F 1 "100nF" H 5725 4850 50  0000 L CNN
 F 2 "Capacitors_SMD:C_0805" H 5738 4800 30  0001 C CNN
@@
 	5700 4550 5700 4800
 $Comp
-L GND #PWR077
+L GND #PWR?
 U 1 1 560A13DA
 P 5700 5350
-F 0 "#PWR077" H 5700 5100 50  0001 C CNN
+F 0 "#PWR?" H 5700 5100 50  0001 C CNN
 F 1 "GND" H 5700 5200 50  0000 C CNN
 F 2 "" H 5700 5350 60  0000 C CNN
@@
 	5700 5100 5700 5350
 $Comp
-L +3V3 #PWR078
+L +3V3 #PWR?
 U 1 1 560A13E1
 P 6100 2350
-F 0 "#PWR078" H 6100 2200 50  0001 C CNN
+F 0 "#PWR?" H 6100 2200 50  0001 C CNN
 F 1 "+3V3" H 6100 2490 50  0000 C CNN
 F 2 "" H 6100 2350 60  0000 C CNN
@@
 $EndComp
 $Comp
-L C C60
+L C C?
 U 1 1 560A13E7
 P 5700 2750
-F 0 "C60" H 5725 2850 50  0000 L CNN
+F 0 "C?" H 5725 2850 50  0000 L CNN
 F 1 "100nF" H 5725 2650 50  0000 L CNN
 F 2 "Capacitors_SMD:C_0805" H 5738 2600 30  0001 C CNN
@@
 $EndComp
 $Comp
-L GND #PWR079
+L GND #PWR?
 U 1 1 560A13EE
 P 5700 2350
-F 0 "#PWR079" H 5700 2100 50  0001 C CNN
+F 0 "#PWR?" H 5700 2100 50  0001 C CNN
 F 1 "GND" H 5700 2200 50  0000 C CNN
 F 2 "" H 5700 2350 60  0000 C CNN
@@
 	5700 2900 5700 3250
 $Comp
-L C C59
+L C C?
 U 1 1 560A13F6
 P 5300 2750
-F 0 "C59" H 5325 2850 50  0000 L CNN
+F 0 "C?" H 5325 2850 50  0000 L CNN
 F 1 "10uF" H 5325 2650 50  0000 L CNN
 F 2 "Capacitors_SMD:C_0805" H 5338 2600 30  0001 C CNN
@@
 $EndComp
 $Comp
-L GND #PWR080
+L GND #PWR?
 U 1 1 560A13FD
 P 5300 2350
-F 0 "#PWR080" H 5300 2100 50  0001 C CNN
+F 0 "#PWR?" H 5300 2100 50  0001 C CNN
 F 1 "GND" H 5300 2200 50  0000 C CNN
 F 2 "" H 5300 2350 60  0000 C CNN
@@
 Connection ~ 5700 3250
 $Comp
-L C C57
+L C C?
 U 1 1 560A1406
 P 2400 2750
-F 0 "C57" H 2425 2850 50  0000 L CNN
+F 0 "C?" H 2425 2850 50  0000 L CNN
 F 1 "10uF" H 2425 2650 50  0000 L CNN
 F 2 "Capacitors_SMD:C_0805" H 2438 2600 30  0001 C CNN
@@
 $EndComp
 $Comp
-L C C58
+L C C?
 U 1 1 560A140D
 P 4900 2750
-F 0 "C58" H 4925 2850 50  0000 L CNN
+F 0 "C?" H 4925 2850 50  0000 L CNN
 F 1 "100nF" H 4925 2650 50  0000 L CNN
 F 2 "Capacitors_SMD:C_0805" H 4938 2600 30  0001 C CNN
@@
 $EndComp
 $Comp
-L GND #PWR081
+L GND #PWR?
 U 1 1 560A1414
 P 4900 2350
-F 0 "#PWR081" H 4900 2100 50  0001 C CNN
+F 0 "#PWR?" H 4900 2100 50  0001 C CNN
 F 1 "GND" H 4900 2200 50  0000 C CNN
 F 2 "" H 4900 2350 60  0000 C CNN
@@
 $EndComp
 $Comp
-L GND #PWR082
+L GND #PWR?
 U 1 1 560A141A
 P 2400 2350
-F 0 "#PWR082" H 2400 2100 50  0001 C CNN
+F 0 "#PWR?" H 2400 2100 50  0001 C CNN
 F 1 "GND" H 2400 2200 50  0000 C CNN
 F 2 "" H 2400 2350 60  0000 C CNN
@@
 Connection ~ 2400 3350
 $Comp
-L GND #PWR083
+L GND #PWR?
 U 1 1 560A1426
 P 2400 5350
-F 0 "#PWR083" H 2400 5100 50  0001 C CNN
+F 0 "#PWR?" H 2400 5100 50  0001 C CNN
 F 1 "GND" H 2400 5200 50  0000 C CNN
 F 2 "" H 2400 5350 60  0000 C CNN
@@
 	2400 3650 2400 5350
 $Comp
-L GND #PWR084
+L GND #PWR?
 U 1 1 560A142E
 P 1650 5350
-F 0 "#PWR084" H 1650 5100 50  0001 C CNN
+F 0 "#PWR?" H 1650 5100 50  0001 C CNN
 F 1 "GND" H 1650 5200 50  0000 C CNN
 F 2 "" H 1650 5350 60  0000 C CNN
@@
 	7700 3950 9250 3950
 $Comp
-L LED D11
+L LED D?
 U 1 1 560A1448
 P 9000 4250
-F 0 "D11" H 9000 4350 50  0000 C CNN
+F 0 "D?" H 9000 4350 50  0000 C CNN
 F 1 "GREEN" H 9000 4150 50  0000 C CNN
 F 2 "" H 9000 4250 60  0001 C CNN
@@
 $EndComp
 $Comp
-L R R58
+L R R?
 U 1 1 560A144F
 P 8450 4250
-F 0 "R58" V 8400 4450 50  0000 C CNN
+F 0 "R?" V 8400 4450 50  0000 C CNN
 F 1 "270" V 8450 4250 50  0000 C CNN
 F 2 "Resistors_SMD:R_0603" V 8380 4250 30  0001 C CNN
@@
 $EndComp
 $Comp
-L +3V3 #PWR085
+L +3V3 #PWR?
 U 1 1 560A1456
 P 9400 4250
-F 0 "#PWR085" H 9400 4100 50  0001 C CNN
+F 0 "#PWR?" H 9400 4100 50  0001 C CNN
 F 1 "+3V3" H 9400 4390 50  0000 C CNN
 F 2 "" H 9400 4250 60  0000 C CNN
@@
 	9200 4250 9400 4250
 $Comp
-L LED D12
+L LED D?
 U 1 1 560A145E
 P 9000 4600
-F 0 "D12" H 9000 4700 50  0000 C CNN
+F 0 "D?" H 9000 4700 50  0000 C CNN
 F 1 "RED" H 9000 4500 50  0000 C CNN
 F 2 "" H 9000 4600 60  0001 C CNN
@@
 $EndComp
 $Comp
-L R R59
+L R R?
 U 1 1 560A1465
 P 8450 4600
-F 0 "R59" V 8400 4800 50  0000 C CNN
+F 0 "R?" V 8400 4800 50  0000 C CNN
 F 1 "270" V 8450 4600 50  0000 C CNN
 F 2 "Resistors_SMD:R_0603" V 8380 4600 30  0001 C CNN
@@
 $EndComp
 $Comp
-L +3V3 #PWR086
+L +3V3 #PWR?
 U 1 1 560A146C
 P 9400 4600
-F 0 "#PWR086" H 9400 4450 50  0001 C CNN
+F 0 "#PWR?" H 9400 4450 50  0001 C CNN
 F 1 "+3V3" H 9400 4740 50  0000 C CNN
 F 2 "" H 9400 4600 60  0000 C CNN
