File: hardware/colibri-v2/wb_ftdi_interface.sch (KiCad schematic (older format))
At the start: 13 parts, among them P5 USB_B, U7 FT232RL

Commit message: Added and assigned footprints.
Parts:
- removed D10: RED, symbol LED
- added DL18: RED, LEDs:LED-0603, symbol LED_SMT
Changed lines of the file:
@@
-$EndComp
-$Comp
-L LED D10
-U 1 1 56335832
-P 9000 4600
-F 0 "D10" H 9000 4700 50  0000 C CNN
-F 1 "RED" H 9000 4500 50  0000 C CNN
-F 2 "" H 9000 4600 60  0001 C CNN
-F 3 "" H 9000 4600 60  0000 C CNN
-	1    9000 4600
-	1    0    0    -1
 $EndComp
 $Comp
@@
 	4200 2350 4200 3350
 Connection ~ 4200 3350
+$Comp
+L LED_SMT DL18
+U 1 1 56CFF954
+P 9000 4600
+F 0 "DL18" H 9000 4700 50  0000 C CNN
+F 1 "RED" H 9000 4500 50  0000 C CNN
+F 2 "LEDs:LED-0603" H 9000 4450 30  0001 C CNN
+F 3 "" H 9000 4600 60  0000 C CNN
+F 4 "0603" H 8885 4580 30  0000 C CNN "SMT"
+F 5 "2322071" H 9000 4400 30  0001 C CNN "Part"
+F 6 "Farnell" H 9000 4350 30  0001 C CNN "Provider"
+	1    9000 4600
+	1    0    0    -1
+$EndComp
 $EndSCHEMATC

Commit message: Added footprints
Parts:
- removed P5: USB_B, symbol USB_B
- added CN11: 629_105_150_921, Sigmadrone:WURTH_629105150921, symbol 629_105_150_921
Connections:
- wire segments 49 -> 54
- no-connect marks 8 -> 9
Changed lines of the file:
@@
 	1    0    0    -1
-$EndComp
-$Comp
-L USB_B P5
-U 1 1 560A13AF
-P 1750 3550
-F 0 "P5" H 1950 3350 50  0000 C CNN
-F 1 "USB_B" H 1700 3750 50  0000 C CNN
-F 2 "" V 1700 3450 60  0001 C CNN
-F 3 "" V 1700 3450 60  0000 C CNN
-	1    1750 3550
-	0    -1   1    0
 $EndComp
 Wire Wire Line
@@
 	2050 3550 6300 3550
 $Comp
-L GND #PWR0101
+L GND #PWR0103
 U 1 1 560A13C1
 P 6100 5350
-F 0 "#PWR0101" H 6100 5100 50  0001 C CNN
+F 0 "#PWR0103" H 6100 5100 50  0001 C CNN
 F 1 "GND" H 6100 5200 50  0000 C CNN
 F 2 "" H 6100 5350 60  0000 C CNN
@@
 	5700 4550 5700 4800
 $Comp
-L GND #PWR0102
+L GND #PWR0104
 U 1 1 560A13DA
 P 5700 5350
-F 0 "#PWR0102" H 5700 5100 50  0001 C CNN
+F 0 "#PWR0104" H 5700 5100 50  0001 C CNN
 F 1 "GND" H 5700 5200 50  0000 C CNN
 F 2 "" H 5700 5350 60  0000 C CNN
@@
 	5700 5100 5700 5350
 $Comp
-L +3V3 #PWR0103
+L +3V3 #PWR0105
 U 1 1 560A13E1
 P 6100 2350
-F 0 "#PWR0103" H 6100 2200 50  0001 C CNN
+F 0 "#PWR0105" H 6100 2200 50  0001 C CNN
 F 1 "+3V3" H 6100 2490 50  0000 C CNN
 F 2 "" H 6100 2350 60  0000 C CNN
@@
 $EndComp
 $Comp
-L GND #PWR0104
+L GND #PWR0106
 U 1 1 560A13EE
 P 5700 2350
-F 0 "#PWR0104" H 5700 2100 50  0001 C CNN
+F 0 "#PWR0106" H 5700 2100 50  0001 C CNN
 F 1 "GND" H 5700 2200 50  0000 C CNN
 F 2 "" H 5700 2350 60  0000 C CNN
@@
 	5700 2900 5700 3250
 $Comp
-L GND #PWR0105
+L GND #PWR0107
 U 1 1 560A13FD
 P 5300 2350
-F 0 "#PWR0105" H 5300 2100 50  0001 C CNN
+F 0 "#PWR0107" H 5300 2100 50  0001 C CNN
 F 1 "GND" H 5300 2200 50  0000 C CNN
 F 2 "" H 5300 2350 60  0000 C CNN
@@
 Connection ~ 5700 3250
 $Comp
-L GND #PWR0106
+L GND #PWR0108
 U 1 1 560A1414
 P 4900 2350
-F 0 "#PWR0106" H 4900 2100 50  0001 C CNN
+F 0 "#PWR0108" H 4900 2100 50  0001 C CNN
 F 1 "GND" H 4900 2200 50  0000 C CNN
 F 2 "" H 4900 2350 60  0000 C CNN
@@
 $EndComp
 $Comp
-L GND #PWR0107
+L GND #PWR0109
 U 1 1 560A141A
 P 2400 2350
-F 0 "#PWR0107" H 2400 2100 50  0001 C CNN
+F 0 "#PWR0109" H 2400 2100 50  0001 C CNN
 F 1 "GND" H 2400 2200 50  0000 C CNN
 F 2 "" H 2400 2350 60  0000 C CNN
@@
 	2400 2900 2400 3350
 Connection ~ 2400 3350
-$Comp
-L GND #PWR0108
-U 1 1 560A1426
-P 2400 5350
-F 0 "#PWR0108" H 2400 5100 50  0001 C CNN
-F 1 "GND" H 2400 5200 50  0000 C CNN
-F 2 "" H 2400 5350 60  0000 C CNN
-F 3 "" H 2400 5350 60  0000 C CNN
-	1    2400 5350
-	1    0    0    -1
-$EndComp
-Wire Wire Line
-	2050 3650 2400 3650
-Wire Wire Line
-	2400 3650 2400 5350
-$Comp
-L GND #PWR0109
-U 1 1 560A142E
-P 1650 5350
-F 0 "#PWR0109" H 1650 5100 50  0001 C CNN
-F 1 "GND" H 1650 5200 50  0000 C CNN
-F 2 "" H 1650 5350 60  0000 C CNN
-F 3 "" H 1650 5350 60  0000 C CNN
-	1    1650 5350
-	1    0    0    -1
-$EndComp
-Wire Wire Line
-	1650 3850 1650 5350
 NoConn ~ 6300 3750
 NoConn ~ 6300 4350
@@
 	1    0    0    -1
 $EndComp
+$Comp
+L GND #PWR0113
+U 1 1 56D2F36C
+P 2250 5350
+F 0 "#PWR0113" H 2250 5100 50  0001 C CNN
+F 1 "GND" H 2250 5200 50  0000 C CNN
+F 2 "" H 2250 5350 60  0000 C CNN
+F 3 "" H 2250 5350 60  0000 C CNN
+	1    2250 5350
+	1    0    0    -1
+$EndComp
+Wire Wire Line
+	2250 3750 2250 5350
+$Comp
+L 629_105_150_921 CN11
+U 1 1 56D2F379
+P 1650 3850
+F 0 "CN11" H 1800 4500 60  0000 C CNN
+F 1 "629_105_150_921" V 1900 3700 60  0000 C CNN
+F 2 "Sigmadrone:WURTH_629105150921" H 3200 5150 60  0001 C CNN
+F 3 "" H 3200 5150 60  0000 C CNN
+	1    1650 3850
+	-1   0    0    -1
+$EndComp
+NoConn ~ 2050 3650
+Wire Wire Line
+	2050 3850 2250 3850
+Wire Wire Line
+	2050 3950 2250 3950
+Wire Wire Line
+	2050 4050 2250 4050
+Wire Wire Line
+	2050 4150 2250 4150
+Wire Wire Line
+	2050 4250 2250 4250
+Wire Wire Line
+	2050 4350 2250 4350
+Connection ~ 2250 3950
+Connection ~ 2250 4050
+Connection ~ 2250 4150
+Connection ~ 2250 4250
+Connection ~ 2250 4350
+Connection ~ 2250 3850
+Wire Wire Line
+	2050 3750 2250 3750
 $EndSCHEMATC

Commit message: Added footprints
Parts:
- U7: footprint (none) -> Housings_SSOP:SSOP-28_5.3x10.2mm_Pitch0.65mm
Changed lines of the file:
@@
 F 0 "U7" H 7350 5200 60  0000 C CNN
 F 1 "FT232RL" H 6750 3100 60  0000 C CNN
-F 2 "" H 7000 4150 60  0001 C CNN
+F 2 "Housings_SSOP:SSOP-28_5.3x10.2mm_Pitch0.65mm" H 7000 4150 60  0001 C CNN
 F 3 "" H 7000 4150 60  0000 C CNN
 	1    7000 4150

Commit message: Added AP6681GMT-HF-3.kicad_mod. Fixed netlist errors
Parts:
- DL18, DL7: footprint LEDs:LED-0603 -> LEDs:LED_0603
Changed lines of the file:
@@
 F 0 "DL7" H 9000 4350 50  0000 C CNN
 F 1 "GREEN" H 9000 4150 50  0000 C CNN
-F 2 "LEDs:LED-0603" H 9000 4100 30  0001 C CNN
+F 2 "LEDs:LED_0603" H 9000 4100 30  0001 C CNN
 F 3 "" H 9000 4250 60  0000 C CNN
 F 4 "0603" H 8885 4230 30  0000 C CNN "SMT"
@@
 F 0 "DL18" H 9000 4700 50  0000 C CNN
 F 1 "RED" H 9000 4500 50  0000 C CNN
-F 2 "LEDs:LED-0603" H 9000 4450 30  0001 C CNN
+F 2 "LEDs:LED_0603" H 9000 4450 30  0001 C CNN
 F 3 "" H 9000 4600 60  0000 C CNN
 F 4 "0603" H 8885 4580 30  0000 C CNN "SMT"
