File: hardware/colibri-v2/wnd_usb_otg.sch (KiCad schematic (older format))
At the start: 17 parts

Commit message: Work on the Cortex sheet
Parts:
- removed C?: 220u/6V3_T, symbol C
- removed C?: 100n/50V, symbol C
- removed D?: RED, symbol LED
- removed D?: GREEN, symbol LED
- removed L?: BLM18EG101TN1D, symbol INDUCTOR
- removed P?: USB_OTG, symbol USB_OTG
- removed Q?: BSS138PW, symbol Q_NMOS_GSD
- removed R? (x2): 22, Resistors_SMD:R_0603, symbol R
- removed R? (x2): 10K, Resistors_SMD:R_0603, symbol R
- removed R? (x2): 47K, Resistors_SMD:R_0603, symbol R
- removed R? (x2): 620, Resistors_SMD:R_0603, symbol R
- removed U?: VBUS053CZ-HAF-G-08, symbol VBUS053CZ-HAF-G-08
- removed U?: TPS2061CDBVT, symbol TPS2061CDBVT
- added C?: 100nF/50V/X7R, Capacitors_SMD:C_0603, symbol C_SMT
- added C?: 220uF/10%/6V3, Capacitors_Tantalum_SMD:TantalC_SizeC_EIA-6032_Reflow, symbol CP_SMT
- added D?: RED, symbol LED
- added DL?: GREEN, LEDs:LED-0603, symbol LED_SMT
- added FB?: BEAD/0.045OHM/2A, Resistors_SMD:R_0603, symbol FB_SMT
- added P?: USB_OTG, symbol USB_OTG
- added Q?: BSS138PW, symbol Q_NMOS_GSD
- added R? (x3): 10K/5%, Resistors_SMD:R_0603, symbol R_SMT
- added R? (x2): 620R/5%, Resistors_SMD:R_0603, symbol R_SMT
- added R? (x2): 22R/5%, Resistors_SMD:R_0603, symbol R_SMT
- added R?: 47K/5%, Resistors_SMD:R_0603, symbol R_SMT
- added U?: VBUS053CZ-HAF-G-08, symbol VBUS053CZ-HAF-G-08
- added U?: TPS2061CDBVT, symbol TPS2061CDBVT
Connections:
- net +3V3: now also R?.1, R?.1, R?.1, R?.2
- net +5V: now also U?.5 (IN)
- net GND: now also C?.2, C?.2, P?.5 (GND), P?.6 (shield), Q?.2 (S), R?.1, U?.2 (GND), U?.7 (GND)
- net OTG_FS_DM: now also R?.2
- net OTG_FS_DP: now also R?.2
- net OTG_FS_ID: now also P?.4 (ID), U?.3 (ID)
- net OTG_FS_OC: now also D?.1 (K), R?.2, U?.3 (~FLT)
- net OTG_FS_PSO: now also R?.2, U?.4 (~EN)
- net VBUS_FS: now also C?.1, C?.1, FB?.2, P?.1 (VCC), R?.2, U?.6 (VBUUS)
- new net: P?.2 (D-), R?.1, U?.1 (D-)
- new net: P?.3 (D+), R?.1, U?.2 (D+)
- new net: D?.2 (A), R?.2
- new net: Q?.1 (G), R?.1, R?.2
- new net: DL?.1 (K), Q?.3 (D)
- new net: FB?.1, U?.1 (OUT)
- new net: DL?.2 (A), R?.1
- no-connect marks 0 -> 2
Other:
- note added: "Should this be +5V"
- note added: "or use TPS2041CDBVT ???"

Commit message: Work on voltage regulators sheet.
Parts:
- removed D?: RED, symbol LED
- added DL?: RED, LEDs:LED-0603, symbol LED_SMT
Connections:
- net OTG_FS_OC: now also DL?.1 (K)
- net at R?.2: now also DL?.2 (A)
Changed lines of the file:
@@
-$EndComp
-$Comp
-L LED D?
-U 1 1 563427D7
-P 2800 2100
-F 0 "D?" H 2800 2200 50  0000 C CNN
-F 1 "RED" H 2800 2000 50  0000 C CNN
-F 2 "" H 2800 2100 60  0001 C CNN
-F 3 "" H 2800 2100 60  0000 C CNN
-	1    2800 2100
-	0    -1   -1   0
 $EndComp
 $Comp
@@
 	1    0    0    -1
 $EndComp
+$Comp
+L LED_SMT DL?
+U 1 1 563753E7
+P 2800 2100
+F 0 "DL?" H 2800 2200 50  0000 C CNN
+F 1 "RED" H 2800 2000 50  0000 C CNN
+F 2 "LEDs:LED-0603" H 2800 1950 30  0001 C CNN
+F 3 "" H 2800 2100 60  0000 C CNN
+F 4 "0603" H 2685 2080 30  0000 C CNN "SMT"
+F 5 "2322071" H 2800 1900 30  0001 C CNN "Part"
+F 6 "Farnell" H 2800 1850 30  0001 C CNN "Provider"
+	1    2800 2100
+	0    -1   -1   0
+$EndComp
 $EndSCHEMATC

Commit message: Work on PWM, USB, MEMS, Power
Parts:
- removed C?: 100nF/50V/X7R, Capacitors_SMD:C_0603, symbol C_SMT
- removed C?: 220uF/10%/6V3, Capacitors_Tantalum_SMD:TantalC_SizeC_EIA-6032_Reflow, symbol CP_SMT
- removed DL?: GREEN, LEDs:LED-0603, symbol LED_SMT
- removed DL?: RED, LEDs:LED-0603, symbol LED_SMT
- removed FB?: BEAD/0.045OHM/2A, Resistors_SMD:R_0603, symbol FB_SMT
- removed P?: USB_OTG, symbol USB_OTG
- removed Q?: BSS138PW, symbol Q_NMOS_GSD
- removed R? (x3): 10K/5%, Resistors_SMD:R_0603, symbol R_SMT
- removed R? (x2): 620R/5%, Resistors_SMD:R_0603, symbol R_SMT
- removed R? (x2): 22R/5%, Resistors_SMD:R_0603, symbol R_SMT
- removed R?: 47K/5%, Resistors_SMD:R_0603, symbol R_SMT
- removed U?: VBUS053CZ-HAF-G-08, symbol VBUS053CZ-HAF-G-08
- removed U?: TPS2061CDBVT, symbol TPS2061CDBVT
- added C?: 10uF/16V/X5R, Capacitors_SMD:C_0603, symbol C_SMT
- added C?: 100nF/50V/X7R, Capacitors_SMD:C_0603, symbol C_SMT
- added C? (x2): 47pF/100V/C0G, Capacitors_SMD:C_0603, symbol C_SMT
- added CN?: 629_105_150_921, symbol 629_105_150_921
- added DL?: GREEN, LEDs:LED-0603, symbol LED_SMT
- added FB?: BEAD/0.045OHM/2A, Resistors_SMD:R_0603, symbol FB_SMT
- added R? (x2): 10K/5%, Resistors_SMD:R_0603, symbol R_SMT
- added R? (x2): 22R/5%, Resistors_SMD:R_0603, symbol R_SMT
- added R?: 1k2/5%, Resistors_SMD:R_0603, symbol R_SMT
- added R?: NA, Resistors_SMD:R_0603, symbol R_SMT
- added U?: VBUS053CZ-HAF-G-08, symbol VBUS053CZ-HAF-G-08
- added U?: TPS2061CDBVT, symbol TPS2061CDBVT
Connections:
- net +3V3: now also R?.1, R?.1
- net +5V: now also U?.5 (IN)
- net GND: now also C?.2, C?.2, C?.2, C?.2, CN?.10 (FN), CN?.11 (FN), CN?.5 (GND), CN?.6 (FN), CN?.7 (FN), CN?.8 (FN), CN?.9 (FN), DL?.1 (K), R?.2, U?.2 (GND), U?.7 (GND)
- new net: CN?.2 (DM), R?.1, U?.1 (D-)
- new net: CN?.3 (DP), R?.1, U?.2 (D+)
- new net: FB?.1, U?.1 (OUT)
- new net: DL?.2 (A), R?.1
- new net USB_OGT_DM: C?.1, R?.2
- new net USB_OTG_DP: C?.1, R?.2
- new net USB_OTG_ID: CN?.4 (ID), R?.1, U?.3 (ID)
- new net USB_OTG_OC: R?.2, U?.3 (~FLT)
- new net USB_OTG_PWR_EN: R?.2, U?.4 (~EN)
- new net USG_OTG_VBUS: C?.1, C?.1, CN?.1 (Vbus), FB?.2, R?.2, U?.6 (VBUUS)
Other:
- note removed: "Should this be +5V"
- note removed: "or use TPS2041CDBVT ???"
