File: hardware/colibri-v2/cortex.sch (KiCad schematic (older format))
At the start: 50 parts

Commit message: Annotated Components
Parts:
- gave numbers to parts that had none: 39

Commit message: Re-annotated schematic
Parts:
- renumbered R4 to R1, R13 to R10, R5 to R2, R6 to R3, R7 to R4, R8 to R5, R9 to R6, R10 to R7, R11 to R8, R12 to R9
Changed lines of the file:
@@
 $EndComp
 $Comp
-L GND #PWR01
+L GND #PWR10
 U 1 1 557C9331
 P 15650 3500
-F 0 "#PWR01" H 15650 3250 50  0001 C CNN
+F 0 "#PWR10" H 15650 3250 50  0001 C CNN
 F 1 "GND" H 15650 3350 50  0000 C CNN
 F 2 "" H 15650 3500 60  0000 C CNN
@@
 $EndComp
 $Comp
-L VDD #PWR02
+L VDD #PWR6
 U 1 1 557C9AC8
 P 12050 1100
-F 0 "#PWR02" H 12050 950 50  0001 C CNN
+F 0 "#PWR6" H 12050 950 50  0001 C CNN
 F 1 "VDD" H 12050 1250 50  0000 C CNN
 F 2 "" H 12050 1100 60  0000 C CNN
@@
 $EndComp
 $Comp
-L GND #PWR03
+L GND #PWR5
 U 1 1 557CC861
 P 11250 1100
-F 0 "#PWR03" H 11250 850 50  0001 C CNN
+F 0 "#PWR5" H 11250 850 50  0001 C CNN
 F 1 "GND" H 11250 950 50  0000 C CNN
 F 2 "" H 11250 1100 60  0000 C CNN
@@
 $EndComp
 $Comp
-L GND #PWR04
+L GND #PWR7
 U 1 1 557CE751
 P 12700 3650
-F 0 "#PWR04" H 12700 3400 50  0001 C CNN
+F 0 "#PWR7" H 12700 3400 50  0001 C CNN
 F 1 "GND" H 12700 3500 50  0000 C CNN
 F 2 "" H 12700 3650 60  0000 C CNN
@@
 $EndComp
 $Comp
-L GND #PWR05
+L GND #PWR8
 U 1 1 557CEC5D
 P 12700 4550
-F 0 "#PWR05" H 12700 4300 50  0001 C CNN
+F 0 "#PWR8" H 12700 4300 50  0001 C CNN
 F 1 "GND" H 12700 4400 50  0000 C CNN
 F 2 "" H 12700 4550 60  0000 C CNN
@@
 $EndComp
 $Comp
-L R R8
+L R R5
 U 1 1 557CF0B9
 P 12400 3500
-F 0 "R8" V 12480 3500 50  0000 C CNN
+F 0 "R5" V 12480 3500 50  0000 C CNN
 F 1 "0R" V 12400 3500 50  0000 C CNN
 F 2 "" V 12330 3500 30  0000 C CNN
@@
 $EndComp
 $Comp
-L VDD #PWR06
+L VDD #PWR9
 U 1 1 557CFB16
 P 15100 1100
-F 0 "#PWR06" H 15100 950 50  0001 C CNN
+F 0 "#PWR9" H 15100 950 50  0001 C CNN
 F 1 "VDD" H 15100 1250 50  0000 C CNN
 F 2 "" H 15100 1100 60  0000 C CNN
@@
 $EndComp
 $Comp
-L R R13
+L R R10
 U 1 1 557CC883
 P 14850 1450
-F 0 "R13" V 14930 1450 50  0000 C CNN
+F 0 "R10" V 14930 1450 50  0000 C CNN
 F 1 "0R" V 14850 1450 50  0000 C CNN
 F 2 "" V 14780 1450 30  0000 C CNN
@@
 $EndComp
 $Comp
-L GND #PWR07
+L GND #PWR1
 U 1 1 557CECF9
 P 7500 8450
-F 0 "#PWR07" H 7500 8200 50  0001 C CNN
+F 0 "#PWR1" H 7500 8200 50  0001 C CNN
 F 1 "GND" H 7500 8300 50  0000 C CNN
 F 2 "" H 7500 8450 60  0000 C CNN
@@
 BOOT0
 $Comp
-L R R4
+L R R1
 U 1 1 557CF5E6
 P 7850 7400
-F 0 "R4" V 7900 7250 50  0000 C CNN
+F 0 "R1" V 7900 7250 50  0000 C CNN
 F 1 "NA" V 7850 7400 50  0000 C CNN
 F 2 "" V 7780 7400 30  0000 C CNN
@@
 $EndComp
 $Comp
-L R R5
+L R R2
 U 1 1 557CF6A2
 P 7850 7600
-F 0 "R5" V 7900 7450 50  0000 C CNN
+F 0 "R2" V 7900 7450 50  0000 C CNN
 F 1 "510" V 7850 7600 50  0000 C CNN
 F 2 "" V 7780 7600 30  0000 C CNN
@@
 $EndComp
 $Comp
-L GND #PWR08
+L GND #PWR4
 U 1 1 557CF83B
 P 7600 7600
-F 0 "#PWR08" H 7600 7350 50  0001 C CNN
+F 0 "#PWR4" H 7600 7350 50  0001 C CNN
 F 1 "GND" V 7600 7400 50  0000 C CNN
 F 2 "" H 7600 7600 60  0000 C CNN
@@
 $EndComp
 $Comp
-L VDD #PWR09
+L VDD #PWR3
 U 1 1 557CF94E
 P 7600 7400
-F 0 "#PWR09" H 7600 7250 50  0001 C CNN
+F 0 "#PWR3" H 7600 7250 50  0001 C CNN
 F 1 "VDD" V 7600 7600 50  0000 C CNN
 F 2 "" H 7600 7400 60  0000 C CNN
@@
 $EndComp
 $Comp
-L GND #PWR010
+L GND #PWR2
 U 1 1 557D1DFA
 P 7500 9550
-F 0 "#PWR010" H 7500 9300 50  0001 C CNN
+F 0 "#PWR2" H 7500 9300 50  0001 C CNN
 F 1 "GND" V 7500 9350 50  0000 C CNN
 F 2 "" H 7500 9550 60  0000 C CNN
@@
 PD7
 $Comp
-L R R9
+L R R6
 U 1 1 55801FDE
 P 14150 9400
-F 0 "R9" V 14100 9250 50  0000 C CNN
+F 0 "R6" V 14100 9250 50  0000 C CNN
 F 1 "0R" V 14150 9400 50  0000 C CNN
 F 2 "" V 14080 9400 30  0000 C CNN
@@
 $EndComp
 $Comp
-L R R10
+L R R7
 U 1 1 5580218A
 P 14150 9500
-F 0 "R10" V 14100 9350 50  0000 C CNN
+F 0 "R7" V 14100 9350 50  0000 C CNN
 F 1 "0R" V 14150 9500 50  0000 C CNN
 F 2 "" V 14080 9500 30  0000 C CNN
@@
 $EndComp
 $Comp
-L R R11
+L R R8
 U 1 1 5580222A
 P 14150 9600
-F 0 "R11" V 14100 9450 50  0000 C CNN
+F 0 "R8" V 14100 9450 50  0000 C CNN
 F 1 "0R" V 14150 9600 50  0000 C CNN
 F 2 "" V 14080 9600 30  0000 C CNN
@@
 $EndComp
 $Comp
-L R R12
+L R R9
 U 1 1 55802327
 P 14150 9700
-F 0 "R12" V 14100 9550 50  0000 C CNN
+F 0 "R9" V 14100 9550 50  0000 C CNN
 F 1 "0R" V 14150 9700 50  0000 C CNN
 F 2 "" V 14080 9700 30  0000 C CNN
@@
 PH1
 $Comp
-L R R6
+L R R3
 U 1 1 55825BF2
 P 8650 8950
-F 0 "R6" V 8730 8950 50  0000 C CNN
+F 0 "R3" V 8730 8950 50  0000 C CNN
 F 1 "0" V 8650 8950 50  0000 C CNN
 F 2 "" V 8580 8950 30  0000 C CNN
@@
 $EndComp
 $Comp
-L R R7
+L R R4
 U 1 1 55825D09
 P 8650 9350
-F 0 "R7" V 8730 9350 50  0000 C CNN
+F 0 "R4" V 8730 9350 50  0000 C CNN
 F 1 "220" V 8650 9350 50  0000 C CNN
 F 2 "" V 8580 9350 30  0000 C CNN

Commit message: Associated footprints for R and some of the C
Parts:
- C1, C10, C11, C12, C13, C14, C15, C16, C17, C18, C19, C2, C20, C21, C22, C23, C24, C25, C26, C3, C4, C5, C6, C7, C8, C9: footprint (none) -> Capacitors_SMD:C_0603
- R1, R10, R2, R3, R4, R5, R6, R7, R8, R9: footprint (none) -> Resistors_SMD:R_0603

Commit message: Work on cortex USB connection.
Parts:
- renumbered C5 to C?, C6 to C?, C7 to C?, C8 to C?, C9 to C?, C10 to C?, C11 to C?, C12 to C?, C13 to C?, C14 to C?, C15 to C?, C16 to C?, C17 to C?, C18 to C?, C19 to C?, C20 to C?, C21 to C?, C23 to C?, C25 to C?, C22 to C?, C24 to C?, C1 to C?, C2 to C?, C26 to C?, C3 to C?, C4 to C?, L1 to L?, R10 to R?, R5 to R?, R1 to R?, R2 to R?, R6 to R?, R7 to R?, R8 to R?, R9 to R?, R3 to R?, R4 to R?, U1 to U?, Y1 to Y?

Commit message: Work on the Cortex sheet
Parts:
- removed C? (x19): 100nF, Capacitors_SMD:C_0603, symbol C
- removed C? (x3): 1uF, Capacitors_SMD:C_0603, symbol C
- removed C? (x2): 2.2uF, Capacitors_SMD:C_0603, symbol C
- removed C? (x2): 20pF, Capacitors_SMD:C_0603, symbol C
- removed L?: BEAD, symbol INDUCTOR
- removed R? (x2): 0R, Resistors_SMD:R_0603, symbol R
- removed R?: NA, Resistors_SMD:R_0603, symbol R
- removed R?: 510, Resistors_SMD:R_0603, symbol R
- removed R?: 0, Resistors_SMD:R_0603, symbol R
- removed R?: 220, Resistors_SMD:R_0603, symbol R
- added C? (x19): 100nF/50V/X7R, Capacitors_SMD:C_0603, symbol C_SMT
- added C? (x3): 1u/25V/X7R, Capacitors_SMD:C_0603, symbol C_SMT
- added C? (x2): 2u2/10V/X5R, Capacitors_SMD:C_0603, symbol C_SMT
- added C? (x2): 10pF/50V/NPO, Capacitors_SMD:C_0603, symbol C_SMT
- added C? (x2): 15pF/50V/NPO, Capacitors_SMD:C_0603, symbol C_SMT
- added FB?: BEAD/0.045OHM/2A, Resistors_SMD:R_0603, symbol FB_SMT
- added R? (x2): 0R/1%, Resistors_SMD:R_0805, symbol R_SMT
- added R?: 10K/5%, Resistors_SMD:R_0603, symbol R_SMT
- added R? (x3): 0R/5%, Resistors_SMD:R_0603, symbol R_SMT
- added R?: 220R/1%, Resistors_SMD:R_0603, symbol R_SMT
- added Y?: 32.768KHZ, symbol Crystal
- Y?: Part (none) -> 1611803; Provider (none) -> Farnell; SMT (none) -> 6mm X 3.6mm
Connections:
- net BOOT0: now also R?.1
- net GND: now also C?.1, C?.1, C?.1, C?.1, C?.1, C?.1, C?.1, C?.1, C?.1, C?.1, C?.1, C?.1, C?.1, C?.1, C?.1, C?.1, C?.1, C?.1, C?.1, C?.1, C?.1, C?.1, C?.1, C?.2, C?.2, C?.2, C?.2, C?.2, R?.2
- net PH0: now also U?.32 (PH0-OSC_IN), R?.1
- net PH1: now also U?.33 (PH1-OSC_OUT), R?.1
- net VCAP1: now also C?.2
- net VCAP2: now also C?.2
- net VREF: now reaches U?.41 (VREF+)
- net VREF: now also C?.1, C?.1, R?.1
- net VDDA: now reaches U?.42 (VDDA)
- net VDDA: now also C?.1, C?.1, FB?.2, R?.2
- net at U?.6 (VBAT): now also R?.2
- net at Y?.1: now also C?.2, R?.2
- net at Y?.2: now also C?.2, R?.2
- net PC14 renamed OSC-IN
- net OSC-IN: now also R?.1
- net PC15 renamed OSC-OUT
- net OSC-OUT: now also R?.1
- net VDD renamed +3V3
- net +3V3: now also C?.1, C?.2, C?.2, C?.2, C?.2, C?.2, C?.2, C?.2, C?.2, C?.2, C?.2, C?.2, C?.2, C?.2, C?.2, C?.2, C?.2, C?.2, FB?.1, R?.1
- new net: C?.2, R?.2, Y?.1
- new net: C?.2, R?.2, Y?.2
Other:
- note added: "Do we need this to be 220R"
- moved on the sheet: U?L, Y?
