File: hardware/colibri-v2/wnd_hdmi.sch (KiCad schematic (older format))
At the start: 13 parts

Commit message: Annotated Components
Parts:
- gave numbers to parts that had none: 13
Changed lines of the file:
@@
 $EndDescr
 $Comp
-L TPD12S521DBTR U?
+L TPD12S521DBTR U11
 U 1 1 56184875
 P 5750 3500
-F 0 "U?" H 6450 4550 60  0000 C CNN
+F 0 "U11" H 6450 4550 60  0000 C CNN
 F 1 "TPD12S521DBTR" H 6250 2450 60  0000 C CNN
 F 2 "" H 5750 3000 60  0000 C CNN
@@
 $EndComp
 $Comp
-L GND #PWR?
+L GND #PWR117
 U 1 1 56186A61
 P 9350 5550
-F 0 "#PWR?" H 9350 5300 50  0001 C CNN
+F 0 "#PWR117" H 9350 5300 50  0001 C CNN
 F 1 "GND" H 9350 5400 50  0000 C CNN
 F 2 "" H 9350 5550 60  0000 C CNN
@@
 $EndComp
 $Comp
-L C C?
+L C C71
 U 1 1 56186B32
 P 7300 2300
-F 0 "C?" H 7325 2400 50  0000 L CNN
+F 0 "C71" H 7325 2400 50  0000 L CNN
 F 1 "100n" H 7325 2200 50  0000 L CNN
 F 2 "" H 7338 2150 30  0000 C CNN
@@
 $EndComp
 $Comp
-L C C?
+L C C70
 U 1 1 56186CEA
 P 7000 2300
-F 0 "C?" H 7025 2400 50  0000 L CNN
+F 0 "C70" H 7025 2400 50  0000 L CNN
 F 1 "100n" H 7025 2200 50  0000 L CNN
 F 2 "" H 7038 2150 30  0000 C CNN
@@
 $EndComp
 $Comp
-L GND #PWR?
+L GND #PWR113
 U 1 1 56186DD2
 P 7300 1800
-F 0 "#PWR?" H 7300 1550 50  0001 C CNN
+F 0 "#PWR113" H 7300 1550 50  0001 C CNN
 F 1 "GND" H 7300 1650 50  0000 C CNN
 F 2 "" H 7300 1800 60  0000 C CNN
@@
 $EndComp
 $Comp
-L GND #PWR?
+L GND #PWR112
 U 1 1 5618793A
 P 7000 5550
-F 0 "#PWR?" H 7000 5300 50  0001 C CNN
+F 0 "#PWR112" H 7000 5300 50  0001 C CNN
 F 1 "GND" H 7000 5400 50  0000 C CNN
 F 2 "" H 7000 5550 60  0000 C CNN
@@
 $EndComp
 $Comp
-L R R?
+L R R82
 U 1 1 5618799C
 P 8250 2300
-F 0 "R?" V 8330 2300 50  0000 C CNN
+F 0 "R82" V 8330 2300 50  0000 C CNN
 F 1 "1.7K" V 8250 2300 50  0000 C CNN
 F 2 "" V 8180 2300 30  0000 C CNN
@@
 $EndComp
 $Comp
-L R R?
+L R R83
 U 1 1 56187A24
 P 8550 2300
-F 0 "R?" V 8630 2300 50  0000 C CNN
+F 0 "R83" V 8630 2300 50  0000 C CNN
 F 1 "1.7K" V 8550 2300 50  0000 C CNN
 F 2 "" V 8480 2300 30  0000 C CNN
@@
 $EndComp
 $Comp
-L R R?
+L R R84
 U 1 1 56187A50
 P 8850 2300
-F 0 "R?" V 8930 2300 50  0000 C CNN
+F 0 "R84" V 8930 2300 50  0000 C CNN
 F 1 "27K" V 8850 2300 50  0000 C CNN
 F 2 "" V 8780 2300 30  0000 C CNN
@@
 $EndComp
 $Comp
-L +5V #PWR?
+L +5V #PWR114
 U 1 1 56187AA3
 P 8250 1800
-F 0 "#PWR?" H 8250 1650 50  0001 C CNN
+F 0 "#PWR114" H 8250 1650 50  0001 C CNN
 F 1 "+5V" H 8250 1940 50  0000 C CNN
 F 2 "" H 8250 1800 60  0000 C CNN
@@
 $EndComp
 $Comp
-L +5V #PWR?
+L +5V #PWR115
 U 1 1 56187ACA
 P 8550 1800
-F 0 "#PWR?" H 8550 1650 50  0001 C CNN
+F 0 "#PWR115" H 8550 1650 50  0001 C CNN
 F 1 "+5V" H 8550 1940 50  0000 C CNN
 F 2 "" H 8550 1800 60  0000 C CNN
@@
 $EndComp
 $Comp
-L +3V3 #PWR?
+L +3V3 #PWR116
 U 1 1 56187AE5
 P 8850 1800
-F 0 "#PWR?" H 8850 1650 50  0001 C CNN
+F 0 "#PWR116" H 8850 1650 50  0001 C CNN
 F 1 "+3V3" H 8850 1940 50  0000 C CNN
 F 2 "" H 8850 1800 60  0000 C CNN
@@
 $EndComp
 $Comp
-L 685_119_136_923 CN?
+L 685_119_136_923 CN2
 U 1 1 56188483
 P 10150 4000
-F 0 "CN?" H 10450 5550 60  0000 C CNN
+F 0 "CN2" H 10450 5550 60  0000 C CNN
 F 1 "685_119_136_923" H 10150 2650 60  0000 C CNN
 F 2 "" H 10000 4200 60  0000 C CNN
@@
 $EndComp
 $Comp
-L +5V #PWR?
+L +5V #PWR109
 U 1 1 561892D1
 P 3950 1750
-F 0 "#PWR?" H 3950 1600 50  0001 C CNN
+F 0 "#PWR109" H 3950 1600 50  0001 C CNN
 F 1 "+5V" H 3950 1890 50  0000 C CNN
 F 2 "" H 3950 1750 60  0000 C CNN
@@
 $EndComp
 $Comp
-L R R?
+L R R81
 U 1 1 56189381
 P 3650 2250
-F 0 "R?" V 3730 2250 50  0000 C CNN
+F 0 "R81" V 3730 2250 50  0000 C CNN
 F 1 "10K" V 3650 2250 50  0000 C CNN
 F 2 "" V 3580 2250 30  0000 C CNN
@@
 $EndComp
 $Comp
-L +3V3 #PWR?
+L +3V3 #PWR108
 U 1 1 56189387
 P 3650 1750
-F 0 "#PWR?" H 3650 1600 50  0001 C CNN
+F 0 "#PWR108" H 3650 1600 50  0001 C CNN
 F 1 "+3V3" H 3650 1890 50  0000 C CNN
 F 2 "" H 3650 1750 60  0000 C CNN
@@
 $EndComp
 $Comp
-L C C?
+L C C69
 U 1 1 5618957F
 P 4500 2250
-F 0 "C?" H 4525 2350 50  0000 L CNN
+F 0 "C69" H 4525 2350 50  0000 L CNN
 F 1 "100n" H 4525 2150 50  0000 L CNN
 F 2 "" H 4538 2100 30  0000 C CNN
@@
 $EndComp
 $Comp
-L C C?
+L C C68
 U 1 1 56189585
 P 4200 2250
-F 0 "C?" H 4225 2350 50  0000 L CNN
+F 0 "C68" H 4225 2350 50  0000 L CNN
 F 1 "100n" H 4225 2150 50  0000 L CNN
 F 2 "" H 4238 2100 30  0000 C CNN
@@
 $EndComp
 $Comp
-L GND #PWR?
+L GND #PWR110
 U 1 1 5618958B
 P 4500 1750
-F 0 "#PWR?" H 4500 1500 50  0001 C CNN
+F 0 "#PWR110" H 4500 1500 50  0001 C CNN
 F 1 "GND" H 4500 1600 50  0000 C CNN
 F 2 "" H 4500 1750 60  0000 C CNN
@@
 HDMI1_HPD
 $Comp
-L R R?
+L R R80
 U 1 1 56189F9C
 P 3350 2250
-F 0 "R?" V 3430 2250 50  0000 C CNN
+F 0 "R80" V 3430 2250 50  0000 C CNN
 F 1 "2.2K" V 3350 2250 50  0000 C CNN
 F 2 "" V 3280 2250 30  0000 C CNN
@@
 $EndComp
 $Comp
-L +5V #PWR?
+L +5V #PWR107
 U 1 1 56189FA2
 P 3350 1750
-F 0 "#PWR?" H 3350 1600 50  0001 C CNN
+F 0 "#PWR107" H 3350 1600 50  0001 C CNN
 F 1 "+5V" H 3350 1890 50  0000 C CNN
 F 2 "" H 3350 1750 60  0000 C CNN
@@
 $EndComp
 $Comp
-L R R?
+L R R79
 U 1 1 56189FFD
 P 3050 2250
-F 0 "R?" V 3130 2250 50  0000 C CNN
+F 0 "R79" V 3130 2250 50  0000 C CNN
 F 1 "2.2K" V 3050 2250 50  0000 C CNN
 F 2 "" V 2980 2250 30  0000 C CNN
@@
 $EndComp
 $Comp
-L +5V #PWR?
+L +5V #PWR106
 U 1 1 5618A003
 P 3050 1750
-F 0 "#PWR?" H 3050 1600 50  0001 C CNN
+F 0 "#PWR106" H 3050 1600 50  0001 C CNN
 F 1 "+5V" H 3050 1890 50  0000 C CNN
 F 2 "" H 3050 1750 60  0000 C CNN
@@
 $EndComp
 $Comp
-L R R?
+L R R78
 U 1 1 5618A152
 P 2750 2250
-F 0 "R?" V 2830 2250 50  0000 C CNN
+F 0 "R78" V 2830 2250 50  0000 C CNN
 F 1 "51K" V 2750 2250 50  0000 C CNN
 F 2 "" V 2680 2250 30  0000 C CNN
@@
 $EndComp
 $Comp
-L +3V3 #PWR?
+L +3V3 #PWR105
 U 1 1 5618A158
 P 2750 1750
-F 0 "#PWR?" H 2750 1600 50  0001 C CNN
+F 0 "#PWR105" H 2750 1600 50  0001 C CNN
 F 1 "+3V3" H 2750 1890 50  0000 C CNN
 F 2 "" H 2750 1750 60  0000 C CNN
@@
 Connection ~ 3350 4300
 $Comp
-L GND #PWR?
+L GND #PWR111
 U 1 1 5618AE70
 P 4500 5550
-F 0 "#PWR?" H 4500 5300 50  0001 C CNN
+F 0 "#PWR111" H 4500 5300 50  0001 C CNN
 F 1 "GND" H 4500 5400 50  0000 C CNN
 F 2 "" H 4500 5550 60  0000 C CNN

Commit message: Re-annotated schematic
Parts:
- renumbered C68 to C66, C69 to C67, C70 to C68, C71 to C69, R78 to R79, R79 to R80, R80 to R81, R81 to R82, R82 to R83, R83 to R84, R84 to R85
Changed lines of the file:
@@
 $EndComp
 $Comp
-L GND #PWR0107
+L GND #PWR114
 U 1 1 56186A61
 P 9350 5550
-F 0 "#PWR0107" H 9350 5300 50  0001 C CNN
+F 0 "#PWR114" H 9350 5300 50  0001 C CNN
 F 1 "GND" H 9350 5400 50  0000 C CNN
 F 2 "" H 9350 5550 60  0000 C CNN
@@
 $EndComp
 $Comp
-L C C71
+L C C69
 U 1 1 56186B32
 P 7300 2300
-F 0 "C71" H 7325 2400 50  0000 L CNN
+F 0 "C69" H 7325 2400 50  0000 L CNN
 F 1 "100n" H 7325 2200 50  0000 L CNN
 F 2 "" H 7338 2150 30  0000 C CNN
@@
 $EndComp
 $Comp
-L C C70
+L C C68
 U 1 1 56186CEA
 P 7000 2300
-F 0 "C70" H 7025 2400 50  0000 L CNN
+F 0 "C68" H 7025 2400 50  0000 L CNN
 F 1 "100n" H 7025 2200 50  0000 L CNN
 F 2 "" H 7038 2150 30  0000 C CNN
@@
 $EndComp
 $Comp
-L GND #PWR0108
+L GND #PWR110
 U 1 1 56186DD2
 P 7300 1800
-F 0 "#PWR0108" H 7300 1550 50  0001 C CNN
+F 0 "#PWR110" H 7300 1550 50  0001 C CNN
 F 1 "GND" H 7300 1650 50  0000 C CNN
 F 2 "" H 7300 1800 60  0000 C CNN
@@
 $EndComp
 $Comp
-L GND #PWR0109
+L GND #PWR109
 U 1 1 5618793A
 P 7000 5550
-F 0 "#PWR0109" H 7000 5300 50  0001 C CNN
+F 0 "#PWR109" H 7000 5300 50  0001 C CNN
 F 1 "GND" H 7000 5400 50  0000 C CNN
 F 2 "" H 7000 5550 60  0000 C CNN
@@
 $EndComp
 $Comp
-L R R82
+L R R83
 U 1 1 5618799C
 P 8250 2300
-F 0 "R82" V 8330 2300 50  0000 C CNN
+F 0 "R83" V 8330 2300 50  0000 C CNN
 F 1 "1.7K" V 8250 2300 50  0000 C CNN
 F 2 "" V 8180 2300 30  0000 C CNN
@@
 $EndComp
 $Comp
-L R R83
+L R R84
 U 1 1 56187A24
 P 8550 2300
-F 0 "R83" V 8630 2300 50  0000 C CNN
+F 0 "R84" V 8630 2300 50  0000 C CNN
 F 1 "1.7K" V 8550 2300 50  0000 C CNN
 F 2 "" V 8480 2300 30  0000 C CNN
@@
 $EndComp
 $Comp
-L R R84
+L R R85
 U 1 1 56187A50
 P 8850 2300
-F 0 "R84" V 8930 2300 50  0000 C CNN
+F 0 "R85" V 8930 2300 50  0000 C CNN
 F 1 "27K" V 8850 2300 50  0000 C CNN
 F 2 "" V 8780 2300 30  0000 C CNN
@@
 $EndComp
 $Comp
-L +5V #PWR0110
+L +5V #PWR111
 U 1 1 56187AA3
 P 8250 1800
-F 0 "#PWR0110" H 8250 1650 50  0001 C CNN
+F 0 "#PWR111" H 8250 1650 50  0001 C CNN
 F 1 "+5V" H 8250 1940 50  0000 C CNN
 F 2 "" H 8250 1800 60  0000 C CNN
@@
 $EndComp
 $Comp
-L +5V #PWR0111
+L +5V #PWR112
 U 1 1 56187ACA
 P 8550 1800
-F 0 "#PWR0111" H 8550 1650 50  0001 C CNN
+F 0 "#PWR112" H 8550 1650 50  0001 C CNN
 F 1 "+5V" H 8550 1940 50  0000 C CNN
 F 2 "" H 8550 1800 60  0000 C CNN
@@
 $EndComp
 $Comp
-L +3V3 #PWR0112
+L +3V3 #PWR113
 U 1 1 56187AE5
 P 8850 1800
-F 0 "#PWR0112" H 8850 1650 50  0001 C CNN
+F 0 "#PWR113" H 8850 1650 50  0001 C CNN
 F 1 "+3V3" H 8850 1940 50  0000 C CNN
 F 2 "" H 8850 1800 60  0000 C CNN
@@
 $EndComp
 $Comp
-L +5V #PWR0113
+L +5V #PWR106
 U 1 1 561892D1
 P 3950 1750
-F 0 "#PWR0113" H 3950 1600 50  0001 C CNN
+F 0 "#PWR106" H 3950 1600 50  0001 C CNN
 F 1 "+5V" H 3950 1890 50  0000 C CNN
 F 2 "" H 3950 1750 60  0000 C CNN
@@
 $EndComp
 $Comp
-L R R81
+L R R82
 U 1 1 56189381
 P 3650 2250
-F 0 "R81" V 3730 2250 50  0000 C CNN
+F 0 "R82" V 3730 2250 50  0000 C CNN
 F 1 "10K" V 3650 2250 50  0000 C CNN
 F 2 "" V 3580 2250 30  0000 C CNN
@@
 $EndComp
 $Comp
-L +3V3 #PWR0114
+L +3V3 #PWR105
 U 1 1 56189387
 P 3650 1750
-F 0 "#PWR0114" H 3650 1600 50  0001 C CNN
+F 0 "#PWR105" H 3650 1600 50  0001 C CNN
 F 1 "+3V3" H 3650 1890 50  0000 C CNN
 F 2 "" H 3650 1750 60  0000 C CNN
@@
 $EndComp
 $Comp
-L C C69
+L C C67
 U 1 1 5618957F
 P 4500 2250
-F 0 "C69" H 4525 2350 50  0000 L CNN
+F 0 "C67" H 4525 2350 50  0000 L CNN
 F 1 "100n" H 4525 2150 50  0000 L CNN
 F 2 "" H 4538 2100 30  0000 C CNN
@@
 $EndComp
 $Comp
-L C C68
+L C C66
 U 1 1 56189585
 P 4200 2250
-F 0 "C68" H 4225 2350 50  0000 L CNN
+F 0 "C66" H 4225 2350 50  0000 L CNN
 F 1 "100n" H 4225 2150 50  0000 L CNN
 F 2 "" H 4238 2100 30  0000 C CNN
@@
 $EndComp
 $Comp
-L GND #PWR0115
+L GND #PWR107
 U 1 1 5618958B
 P 4500 1750
-F 0 "#PWR0115" H 4500 1500 50  0001 C CNN
+F 0 "#PWR107" H 4500 1500 50  0001 C CNN
 F 1 "GND" H 4500 1600 50  0000 C CNN
 F 2 "" H 4500 1750 60  0000 C CNN
@@
 HDMI1_HPD
 $Comp
-L R R80
+L R R81
 U 1 1 56189F9C
 P 3350 2250
-F 0 "R80" V 3430 2250 50  0000 C CNN
+F 0 "R81" V 3430 2250 50  0000 C CNN
 F 1 "2.2K" V 3350 2250 50  0000 C CNN
 F 2 "" V 3280 2250 30  0000 C CNN
@@
 $EndComp
 $Comp
-L +5V #PWR0116
+L +5V #PWR104
 U 1 1 56189FA2
 P 3350 1750
-F 0 "#PWR0116" H 3350 1600 50  0001 C CNN
+F 0 "#PWR104" H 3350 1600 50  0001 C CNN
 F 1 "+5V" H 3350 1890 50  0000 C CNN
 F 2 "" H 3350 1750 60  0000 C CNN
@@
 $EndComp
 $Comp
-L R R79
+L R R80
 U 1 1 56189FFD
 P 3050 2250
-F 0 "R79" V 3130 2250 50  0000 C CNN
+F 0 "R80" V 3130 2250 50  0000 C CNN
 F 1 "2.2K" V 3050 2250 50  0000 C CNN
 F 2 "" V 2980 2250 30  0000 C CNN
@@
 $EndComp
 $Comp
-L +5V #PWR0117
+L +5V #PWR103
 U 1 1 5618A003
 P 3050 1750
-F 0 "#PWR0117" H 3050 1600 50  0001 C CNN
+F 0 "#PWR103" H 3050 1600 50  0001 C CNN
 F 1 "+5V" H 3050 1890 50  0000 C CNN
 F 2 "" H 3050 1750 60  0000 C CNN
@@
 $EndComp
 $Comp
-L R R78
+L R R79
 U 1 1 5618A152
 P 2750 2250
-F 0 "R78" V 2830 2250 50  0000 C CNN
+F 0 "R79" V 2830 2250 50  0000 C CNN
 F 1 "51K" V 2750 2250 50  0000 C CNN
 F 2 "" V 2680 2250 30  0000 C CNN
@@
 $EndComp
 $Comp
-L +3V3 #PWR0118
+L +3V3 #PWR102
 U 1 1 5618A158
 P 2750 1750
-F 0 "#PWR0118" H 2750 1600 50  0001 C CNN
+F 0 "#PWR102" H 2750 1600 50  0001 C CNN
 F 1 "+3V3" H 2750 1890 50  0000 C CNN
 F 2 "" H 2750 1750 60  0000 C CNN
@@
 Connection ~ 3350 4300
 $Comp
-L GND #PWR0119
+L GND #PWR108
 U 1 1 5618AE70
 P 4500 5550
-F 0 "#PWR0119" H 4500 5300 50  0001 C CNN
+F 0 "#PWR108" H 4500 5300 50  0001 C CNN
 F 1 "GND" H 4500 5400 50  0000 C CNN
 F 2 "" H 4500 5550 60  0000 C CNN

Commit message: Associated footprints for R and some of the C
Parts:
- R79, R80, R81, R82, R83, R84, R85: footprint (none) -> Resistors_SMD:R_0603
Changed lines of the file:
@@
 F 0 "U11" H 6450 4550 60  0000 C CNN
 F 1 "TPD12S521DBTR" H 6250 2450 60  0000 C CNN
-F 2 "" H 5750 3000 60  0000 C CNN
+F 2 "" H 5750 3000 60  0001 C CNN
 F 3 "" H 5750 3000 60  0000 C CNN
 	1    5750 3500
@@
 $EndComp
 $Comp
-L GND #PWR114
+L GND #PWR0104
 U 1 1 56186A61
 P 9350 5550
-F 0 "#PWR114" H 9350 5300 50  0001 C CNN
+F 0 "#PWR0104" H 9350 5300 50  0001 C CNN
 F 1 "GND" H 9350 5400 50  0000 C CNN
 F 2 "" H 9350 5550 60  0000 C CNN
@@
 F 0 "C69" H 7325 2400 50  0000 L CNN
 F 1 "100n" H 7325 2200 50  0000 L CNN
-F 2 "" H 7338 2150 30  0000 C CNN
+F 2 "" H 7338 2150 30  0001 C CNN
 F 3 "" H 7300 2300 60  0000 C CNN
 	1    7300 2300
@@
 F 0 "C68" H 7025 2400 50  0000 L CNN
 F 1 "100n" H 7025 2200 50  0000 L CNN
-F 2 "" H 7038 2150 30  0000 C CNN
+F 2 "" H 7038 2150 30  0001 C CNN
 F 3 "" H 7000 2300 60  0000 C CNN
 	1    7000 2300
@@
 $EndComp
 $Comp
-L GND #PWR110
+L GND #PWR0105
 U 1 1 56186DD2
 P 7300 1800
-F 0 "#PWR110" H 7300 1550 50  0001 C CNN
+F 0 "#PWR0105" H 7300 1550 50  0001 C CNN
 F 1 "GND" H 7300 1650 50  0000 C CNN
 F 2 "" H 7300 1800 60  0000 C CNN
@@
 $EndComp
 $Comp
-L GND #PWR109
+L GND #PWR0106
 U 1 1 5618793A
 P 7000 5550
-F 0 "#PWR109" H 7000 5300 50  0001 C CNN
+F 0 "#PWR0106" H 7000 5300 50  0001 C CNN
 F 1 "GND" H 7000 5400 50  0000 C CNN
 F 2 "" H 7000 5550 60  0000 C CNN
@@
 F 0 "R83" V 8330 2300 50  0000 C CNN
 F 1 "1.7K" V 8250 2300 50  0000 C CNN
-F 2 "" V 8180 2300 30  0000 C CNN
+F 2 "Resistors_SMD:R_0603" V 8180 2300 30  0001 C CNN
 F 3 "" H 8250 2300 30  0000 C CNN
 	1    8250 2300
@@
 F 0 "R84" V 8630 2300 50  0000 C CNN
 F 1 "1.7K" V 8550 2300 50  0000 C CNN
-F 2 "" V 8480 2300 30  0000 C CNN
+F 2 "Resistors_SMD:R_0603" V 8480 2300 30  0001 C CNN
 F 3 "" H 8550 2300 30  0000 C CNN
 	1    8550 2300
@@
 F 0 "R85" V 8930 2300 50  0000 C CNN
 F 1 "27K" V 8850 2300 50  0000 C CNN
-F 2 "" V 8780 2300 30  0000 C CNN
+F 2 "Resistors_SMD:R_0603" V 8780 2300 30  0001 C CNN
 F 3 "" H 8850 2300 30  0000 C CNN
 	1    8850 2300
@@
 $EndComp
 $Comp
-L +5V #PWR111
+L +5V #PWR0107
 U 1 1 56187AA3
 P 8250 1800
-F 0 "#PWR111" H 8250 1650 50  0001 C CNN
+F 0 "#PWR0107" H 8250 1650 50  0001 C CNN
 F 1 "+5V" H 8250 1940 50  0000 C CNN
 F 2 "" H 8250 1800 60  0000 C CNN
@@
 $EndComp
 $Comp
-L +5V #PWR112
+L +5V #PWR0108
 U 1 1 56187ACA
 P 8550 1800
-F 0 "#PWR112" H 8550 1650 50  0001 C CNN
+F 0 "#PWR0108" H 8550 1650 50  0001 C CNN
 F 1 "+5V" H 8550 1940 50  0000 C CNN
 F 2 "" H 8550 1800 60  0000 C CNN
@@
 $EndComp
 $Comp
-L +3V3 #PWR113
+L +3V3 #PWR0109
 U 1 1 56187AE5
 P 8850 1800
-F 0 "#PWR113" H 8850 1650 50  0001 C CNN
+F 0 "#PWR0109" H 8850 1650 50  0001 C CNN
 F 1 "+3V3" H 8850 1940 50  0000 C CNN
 F 2 "" H 8850 1800 60  0000 C CNN
@@
 F 0 "CN2" H 10450 5550 60  0000 C CNN
 F 1 "685_119_136_923" H 10150 2650 60  0000 C CNN
-F 2 "" H 10000 4200 60  0000 C CNN
+F 2 "" H 10000 4200 60  0001 C CNN
 F 3 "" H 10000 4200 60  0000 C CNN
 	1    10150 4000
@@
 $EndComp
 $Comp
-L +5V #PWR106
+L +5V #PWR0110
 U 1 1 561892D1
 P 3950 1750
-F 0 "#PWR106" H 3950 1600 50  0001 C CNN
+F 0 "#PWR0110" H 3950 1600 50  0001 C CNN
 F 1 "+5V" H 3950 1890 50  0000 C CNN
 F 2 "" H 3950 1750 60  0000 C CNN
@@
 F 0 "R82" V 3730 2250 50  0000 C CNN
 F 1 "10K" V 3650 2250 50  0000 C CNN
-F 2 "" V 3580 2250 30  0000 C CNN
+F 2 "Resistors_SMD:R_0603" V 3580 2250 30  0001 C CNN
 F 3 "" H 3650 2250 30  0000 C CNN
 	1    3650 2250
@@
 $EndComp
 $Comp
-L +3V3 #PWR105
+L +3V3 #PWR0111
 U 1 1 56189387
 P 3650 1750
-F 0 "#PWR105" H 3650 1600 50  0001 C CNN
+F 0 "#PWR0111" H 3650 1600 50  0001 C CNN
 F 1 "+3V3" H 3650 1890 50  0000 C CNN
 F 2 "" H 3650 1750 60  0000 C CNN
@@
 F 0 "C67" H 4525 2350 50  0000 L CNN
 F 1 "100n" H 4525 2150 50  0000 L CNN
-F 2 "" H 4538 2100 30  0000 C CNN
+F 2 "" H 4538 2100 30  0001 C CNN
 F 3 "" H 4500 2250 60  0000 C CNN
 	1    4500 2250
@@
 F 0 "C66" H 4225 2350 50  0000 L CNN
 F 1 "100n" H 4225 2150 50  0000 L CNN
-F 2 "" H 4238 2100 30  0000 C CNN
+F 2 "" H 4238 2100 30  0001 C CNN
 F 3 "" H 4200 2250 60  0000 C CNN
 	1    4200 2250
@@
 $EndComp
 $Comp
-L GND #PWR107
+L GND #PWR0112
 U 1 1 5618958B
 P 4500 1750
-F 0 "#PWR107" H 4500 1500 50  0001 C CNN
+F 0 "#PWR0112" H 4500 1500 50  0001 C CNN
 F 1 "GND" H 4500 1600 50  0000 C CNN
 F 2 "" H 4500 1750 60  0000 C CNN
@@
 F 0 "R81" V 3430 2250 50  0000 C CNN
 F 1 "2.2K" V 3350 2250 50  0000 C CNN
-F 2 "" V 3280 2250 30  0000 C CNN
+F 2 "Resistors_SMD:R_0603" V 3280 2250 30  0001 C CNN
 F 3 "" H 3350 2250 30  0000 C CNN
 	1    3350 2250
@@
 $EndComp
 $Comp
-L +5V #PWR104
+L +5V #PWR0113
 U 1 1 56189FA2
 P 3350 1750
-F 0 "#PWR104" H 3350 1600 50  0001 C CNN
+F 0 "#PWR0113" H 3350 1600 50  0001 C CNN
 F 1 "+5V" H 3350 1890 50  0000 C CNN
 F 2 "" H 3350 1750 60  0000 C CNN
@@
 F 0 "R80" V 3130 2250 50  0000 C CNN
 F 1 "2.2K" V 3050 2250 50  0000 C CNN
-F 2 "" V 2980 2250 30  0000 C CNN
+F 2 "Resistors_SMD:R_0603" V 2980 2250 30  0001 C CNN
 F 3 "" H 3050 2250 30  0000 C CNN
 	1    3050 2250
@@
 $EndComp
 $Comp
-L +5V #PWR103
+L +5V #PWR0114
 U 1 1 5618A003
 P 3050 1750
-F 0 "#PWR103" H 3050 1600 50  0001 C CNN
+F 0 "#PWR0114" H 3050 1600 50  0001 C CNN
 F 1 "+5V" H 3050 1890 50  0000 C CNN
 F 2 "" H 3050 1750 60  0000 C CNN
@@
 F 0 "R79" V 2830 2250 50  0000 C CNN
 F 1 "51K" V 2750 2250 50  0000 C CNN
-F 2 "" V 2680 2250 30  0000 C CNN
+F 2 "Resistors_SMD:R_0603" V 2680 2250 30  0001 C CNN
 F 3 "" H 2750 2250 30  0000 C CNN
 	1    2750 2250
@@
 $EndComp
 $Comp
-L +3V3 #PWR102
+L +3V3 #PWR0115
 U 1 1 5618A158
 P 2750 1750
-F 0 "#PWR102" H 2750 1600 50  0001 C CNN
+F 0 "#PWR0115" H 2750 1600 50  0001 C CNN
 F 1 "+3V3" H 2750 1890 50  0000 C CNN
 F 2 "" H 2750 1750 60  0000 C CNN
@@
 Connection ~ 3350 4300
 $Comp
-L GND #PWR108
+L GND #PWR0116
 U 1 1 5618AE70
 P 4500 5550
-F 0 "#PWR108" H 4500 5300 50  0001 C CNN
+F 0 "#PWR0116" H 4500 5300 50  0001 C CNN
 F 1 "GND" H 4500 5400 50  0000 C CNN
 F 2 "" H 4500 5550 60  0000 C CNN
