File: hardware/colibri-v2/wnd_hdmi.sch (KiCad schematic (older format))
At the start: 13 parts, among them CN2 685_119_136_923, U11 TPD12S521DBTR

Commit message: Work on cortex USB connection.
Parts:
- renumbered C69 to C?, C68 to C?, C67 to C?, C66 to C?, CN2 to CN?, R83 to R?, R84 to R?, R85 to R?, R82 to R?, R81 to R?, R80 to R?, R79 to R?, U11 to U?
Changed lines of the file:
@@
 $EndDescr
 $Comp
-L TPD12S521DBTR U11
+L TPD12S521DBTR U?
 U 1 1 56184875
 P 5750 3500
-F 0 "U11" H 6450 4550 60  0000 C CNN
+F 0 "U?" H 6450 4550 60  0000 C CNN
 F 1 "TPD12S521DBTR" H 6250 2450 60  0000 C CNN
 F 2 "" H 5750 3000 60  0001 C CNN
@@
 $EndComp
 $Comp
-L GND #PWR0104
+L GND #PWR?
 U 1 1 56186A61
 P 9350 5550
-F 0 "#PWR0104" H 9350 5300 50  0001 C CNN
+F 0 "#PWR?" H 9350 5300 50  0001 C CNN
 F 1 "GND" H 9350 5400 50  0000 C CNN
 F 2 "" H 9350 5550 60  0000 C CNN
@@
 $EndComp
 $Comp
-L C C69
+L C C?
 U 1 1 56186B32
 P 7300 2300
-F 0 "C69" H 7325 2400 50  0000 L CNN
+F 0 "C?" H 7325 2400 50  0000 L CNN
 F 1 "100n" H 7325 2200 50  0000 L CNN
 F 2 "" H 7338 2150 30  0001 C CNN
@@
 $EndComp
 $Comp
-L C C68
+L C C?
 U 1 1 56186CEA
 P 7000 2300
-F 0 "C68" H 7025 2400 50  0000 L CNN
+F 0 "C?" H 7025 2400 50  0000 L CNN
 F 1 "100n" H 7025 2200 50  0000 L CNN
 F 2 "" H 7038 2150 30  0001 C CNN
@@
 $EndComp
 $Comp
-L GND #PWR0105
+L GND #PWR?
 U 1 1 56186DD2
 P 7300 1800
-F 0 "#PWR0105" H 7300 1550 50  0001 C CNN
+F 0 "#PWR?" H 7300 1550 50  0001 C CNN
 F 1 "GND" H 7300 1650 50  0000 C CNN
 F 2 "" H 7300 1800 60  0000 C CNN
@@
 $EndComp
 $Comp
-L GND #PWR0106
+L GND #PWR?
 U 1 1 5618793A
 P 7000 5550
-F 0 "#PWR0106" H 7000 5300 50  0001 C CNN
+F 0 "#PWR?" H 7000 5300 50  0001 C CNN
 F 1 "GND" H 7000 5400 50  0000 C CNN
 F 2 "" H 7000 5550 60  0000 C CNN
@@
 $EndComp
 $Comp
-L R R83
+L R R?
 U 1 1 5618799C
 P 8250 2300
-F 0 "R83" V 8330 2300 50  0000 C CNN
+F 0 "R?" V 8330 2300 50  0000 C CNN
 F 1 "1.7K" V 8250 2300 50  0000 C CNN
 F 2 "Resistors_SMD:R_0603" V 8180 2300 30  0001 C CNN
@@
 $EndComp
 $Comp
-L R R84
+L R R?
 U 1 1 56187A24
 P 8550 2300
-F 0 "R84" V 8630 2300 50  0000 C CNN
+F 0 "R?" V 8630 2300 50  0000 C CNN
 F 1 "1.7K" V 8550 2300 50  0000 C CNN
 F 2 "Resistors_SMD:R_0603" V 8480 2300 30  0001 C CNN
@@
 $EndComp
 $Comp
-L R R85
+L R R?
 U 1 1 56187A50
 P 8850 2300
-F 0 "R85" V 8930 2300 50  0000 C CNN
+F 0 "R?" V 8930 2300 50  0000 C CNN
 F 1 "27K" V 8850 2300 50  0000 C CNN
 F 2 "Resistors_SMD:R_0603" V 8780 2300 30  0001 C CNN
@@
 $EndComp
 $Comp
-L +5V #PWR0107
+L +5V #PWR?
 U 1 1 56187AA3
 P 8250 1800
-F 0 "#PWR0107" H 8250 1650 50  0001 C CNN
+F 0 "#PWR?" H 8250 1650 50  0001 C CNN
 F 1 "+5V" H 8250 1940 50  0000 C CNN
 F 2 "" H 8250 1800 60  0000 C CNN
@@
 $EndComp
 $Comp
-L +5V #PWR0108
+L +5V #PWR?
 U 1 1 56187ACA
 P 8550 1800
-F 0 "#PWR0108" H 8550 1650 50  0001 C CNN
+F 0 "#PWR?" H 8550 1650 50  0001 C CNN
 F 1 "+5V" H 8550 1940 50  0000 C CNN
 F 2 "" H 8550 1800 60  0000 C CNN
@@
 $EndComp
 $Comp
-L +3V3 #PWR0109
+L +3V3 #PWR?
 U 1 1 56187AE5
 P 8850 1800
-F 0 "#PWR0109" H 8850 1650 50  0001 C CNN
+F 0 "#PWR?" H 8850 1650 50  0001 C CNN
 F 1 "+3V3" H 8850 1940 50  0000 C CNN
 F 2 "" H 8850 1800 60  0000 C CNN
@@
 $EndComp
 $Comp
-L 685_119_136_923 CN2
+L 685_119_136_923 CN?
 U 1 1 56188483
 P 10150 4000
-F 0 "CN2" H 10450 5550 60  0000 C CNN
+F 0 "CN?" H 10450 5550 60  0000 C CNN
 F 1 "685_119_136_923" H 10150 2650 60  0000 C CNN
 F 2 "" H 10000 4200 60  0001 C CNN
@@
 $EndComp
 $Comp
-L +5V #PWR0110
+L +5V #PWR?
 U 1 1 561892D1
 P 3950 1750
-F 0 "#PWR0110" H 3950 1600 50  0001 C CNN
+F 0 "#PWR?" H 3950 1600 50  0001 C CNN
 F 1 "+5V" H 3950 1890 50  0000 C CNN
 F 2 "" H 3950 1750 60  0000 C CNN
@@
 $EndComp
 $Comp
-L R R82
+L R R?
 U 1 1 56189381
 P 3650 2250
-F 0 "R82" V 3730 2250 50  0000 C CNN
+F 0 "R?" V 3730 2250 50  0000 C CNN
 F 1 "10K" V 3650 2250 50  0000 C CNN
 F 2 "Resistors_SMD:R_0603" V 3580 2250 30  0001 C CNN
@@
 $EndComp
 $Comp
-L +3V3 #PWR0111
+L +3V3 #PWR?
 U 1 1 56189387
 P 3650 1750
-F 0 "#PWR0111" H 3650 1600 50  0001 C CNN
+F 0 "#PWR?" H 3650 1600 50  0001 C CNN
 F 1 "+3V3" H 3650 1890 50  0000 C CNN
 F 2 "" H 3650 1750 60  0000 C CNN
@@
 $EndComp
 $Comp
-L C C67
+L C C?
 U 1 1 5618957F
 P 4500 2250
-F 0 "C67" H 4525 2350 50  0000 L CNN
+F 0 "C?" H 4525 2350 50  0000 L CNN
 F 1 "100n" H 4525 2150 50  0000 L CNN
 F 2 "" H 4538 2100 30  0001 C CNN
@@
 $EndComp
 $Comp
-L C C66
+L C C?
 U 1 1 56189585
 P 4200 2250
-F 0 "C66" H 4225 2350 50  0000 L CNN
+F 0 "C?" H 4225 2350 50  0000 L CNN
 F 1 "100n" H 4225 2150 50  0000 L CNN
 F 2 "" H 4238 2100 30  0001 C CNN
@@
 $EndComp
 $Comp
-L GND #PWR0112
+L GND #PWR?
 U 1 1 5618958B
 P 4500 1750
-F 0 "#PWR0112" H 4500 1500 50  0001 C CNN
+F 0 "#PWR?" H 4500 1500 50  0001 C CNN
 F 1 "GND" H 4500 1600 50  0000 C CNN
 F 2 "" H 4500 1750 60  0000 C CNN
@@
 HDMI1_HPD
 $Comp
-L R R81
+L R R?
 U 1 1 56189F9C
 P 3350 2250
-F 0 "R81" V 3430 2250 50  0000 C CNN
+F 0 "R?" V 3430 2250 50  0000 C CNN
 F 1 "2.2K" V 3350 2250 50  0000 C CNN
 F 2 "Resistors_SMD:R_0603" V 3280 2250 30  0001 C CNN
@@
 $EndComp
 $Comp
-L +5V #PWR0113
+L +5V #PWR?
 U 1 1 56189FA2
 P 3350 1750
-F 0 "#PWR0113" H 3350 1600 50  0001 C CNN
+F 0 "#PWR?" H 3350 1600 50  0001 C CNN
 F 1 "+5V" H 3350 1890 50  0000 C CNN
 F 2 "" H 3350 1750 60  0000 C CNN
@@
 $EndComp
 $Comp
-L R R80
+L R R?
 U 1 1 56189FFD
 P 3050 2250
-F 0 "R80" V 3130 2250 50  0000 C CNN
+F 0 "R?" V 3130 2250 50  0000 C CNN
 F 1 "2.2K" V 3050 2250 50  0000 C CNN
 F 2 "Resistors_SMD:R_0603" V 2980 2250 30  0001 C CNN
@@
 $EndComp
 $Comp
-L +5V #PWR0114
+L +5V #PWR?
 U 1 1 5618A003
 P 3050 1750
-F 0 "#PWR0114" H 3050 1600 50  0001 C CNN
+F 0 "#PWR?" H 3050 1600 50  0001 C CNN
 F 1 "+5V" H 3050 1890 50  0000 C CNN
 F 2 "" H 3050 1750 60  0000 C CNN
@@
 $EndComp
 $Comp
-L R R79
+L R R?
 U 1 1 5618A152
 P 2750 2250
-F 0 "R79" V 2830 2250 50  0000 C CNN
+F 0 "R?" V 2830 2250 50  0000 C CNN
 F 1 "51K" V 2750 2250 50  0000 C CNN
 F 2 "Resistors_SMD:R_0603" V 2680 2250 30  0001 C CNN
@@
 $EndComp
 $Comp
-L +3V3 #PWR0115
+L +3V3 #PWR?
 U 1 1 5618A158
 P 2750 1750
-F 0 "#PWR0115" H 2750 1600 50  0001 C CNN
+F 0 "#PWR?" H 2750 1600 50  0001 C CNN
 F 1 "+3V3" H 2750 1890 50  0000 C CNN
 F 2 "" H 2750 1750 60  0000 C CNN
@@
 Connection ~ 3350 4300
 $Comp
-L GND #PWR0116
+L GND #PWR?
 U 1 1 5618AE70
 P 4500 5550
-F 0 "#PWR0116" H 4500 5300 50  0001 C CNN
+F 0 "#PWR?" H 4500 5300 50  0001 C CNN
 F 1 "GND" H 4500 5400 50  0000 C CNN
 F 2 "" H 4500 5550 60  0000 C CNN

Commit message: Work on the Cortex sheet
Parts:
- removed C? (x4): 100n, symbol C
- removed R? (x2): 1.7K, Resistors_SMD:R_0603, symbol R
- removed R?: 27K, Resistors_SMD:R_0603, symbol R
- removed R?: 10K, Resistors_SMD:R_0603, symbol R
- removed R? (x2): 2.2K, Resistors_SMD:R_0603, symbol R
- removed R?: 51K, Resistors_SMD:R_0603, symbol R
- added C? (x4): 100nF/50V/X7R, Capacitors_SMD:C_0603, symbol C_SMT
- added D?: BAS316, Diodes_SMD:SOD-323, symbol D_SMT
- added R?: 10K/5%, Resistors_SMD:R_0603, symbol R_SMT
- added R? (x2): 2k2/5%, Resistors_SMD:R_0603, symbol R_SMT
- added R?: 1K/5%, Resistors_SMD:R_0603, symbol R_SMT
- added R? (x2): 1k8/5%, Resistors_SMD:R_0603, symbol R_SMT
- added R?: 27K/5%, Resistors_SMD:R_0603, symbol R_SMT
Connections:
- net +3V3: now also D?.2 (A), R?.1, R?.1
- net +5V: now also C?.2, R?.1, R?.1, R?.1, R?.1
- net DDC_SCL(5V): now also R?.2
- net DDC_SDA(5V): now also R?.2
- net GND: now also C?.1, C?.1, C?.1, C?.1
- net HDMI_CEC_IN: now also R?.2
- net at U?.2 (LV_SUPPLY): now also C?.2, R?.2
- net at CN?.16 (DDC_DATA), U?.21 (DDC_DAT_OUT): now also R?.2
- net at CN?.15 (DDC_CLK), U?.22 (DDC_CLK_OUT): now also R?.2
- net at CN?.13 (CE_REMOTE), U?.23 (CE_REMOTE_OUT): now also R?.2
- net at U?.37 (ESD_BYP): now also C?.2
- net at CN?.18 (+5V), U?.38 (5V_OUT): now also C?.2
- new net: D?.1 (K), R?.1
