File: hardware/colibri-v2/wnd_hdmi.sch (KiCad schematic (older format))
At the start: 14 parts, among them CN4 685_119_136_923, U8 TPD12S521DBTR

Commit message: Added MOLEX_500254_1927.kicad_mod
Parts:
- removed CN4: 685_119_136_923, symbol 685_119_136_923
- added CN4: HDMI_A, Sigmadrone:MOLEX_500254_1927, symbol HDMI_A
Connections:
- no-connect marks 0 -> 1
Changed lines of the file:
@@
 $Descr A4 11693 8268
 encoding utf-8
-Sheet 15 28
+Sheet 14 28
 Title ""
 Date ""
@@
 F 3 "" H 8850 1300 60  0000 C CNN
 	1    8850 1300
-	1    0    0    -1
-$EndComp
-$Comp
-L 685_119_136_923 CN4
-U 1 1 56188483
-P 10150 4000
-F 0 "CN4" H 10450 5550 60  0000 C CNN
-F 1 "685_119_136_923" H 10150 2650 60  0000 C CNN
-F 2 "" H 10000 4200 60  0001 C CNN
-F 3 "" H 10000 4200 60  0000 C CNN
-	1    10150 4000
 	1    0    0    -1
 $EndComp
@@
 	3800 2400 3650 2400
 Connection ~ 3650 2400
+$Comp
+L HDMI_A CN4
+U 1 1 56CE83E2
+P 10150 4000
+F 0 "CN4" H 10450 5550 60  0000 C CNN
+F 1 "HDMI_A" H 10150 2650 60  0000 C CNN
+F 2 "Sigmadrone:MOLEX_500254_1927" H 10000 4200 60  0001 C CNN
+F 3 "" H 10000 4200 60  0000 C CNN
+	1    10150 4000
+	1    0    0    -1
+$EndComp
+NoConn ~ 9550 4500
 $EndSCHEMATC

Commit message: Added footprints
Parts:
- U8: footprint (none) -> Housings_SSOP:TSSOP-38_4.4x9.7mm_Pitch0.5mm
Changed lines of the file:
@@
 F 0 "U8" H 6450 4550 60  0000 C CNN
 F 1 "TPD12S521DBTR" H 6250 2450 60  0000 C CNN
-F 2 "" H 5750 3000 60  0001 C CNN
+F 2 "Housings_SSOP:TSSOP-38_4.4x9.7mm_Pitch0.5mm" H 5750 3000 60  0001 C CNN
 F 3 "" H 5750 3000 60  0000 C CNN
 	1    5750 3500
