File: hardware/colibri-v2/wnd_usb_host.sch (KiCad schematic (older format))
At the start: 12 parts

Commit message: added wnd_lcd.sch
Changed lines of the file:
@@
 $Descr A4 11693 8268
 encoding utf-8
-Sheet 17 22
+Sheet 17 23
 Title ""
 Date ""
@@
 $EndComp
 Wire Wire Line
-	1900 2000 2750 2000
-Wire Wire Line
-	2750 2000 3100 2000
-Wire Wire Line
-	3100 2000 4100 2000
+	1900 2000 4100 2000
 Wire Wire Line
 	2750 1000 2750 1050
@@
 	5100 1800 5800 1800
 Wire Wire Line
-	6400 1800 6900 1800
-Wire Wire Line
-	6900 1800 7600 1800
-Wire Wire Line
-	7600 1800 8300 1800
+	6400 1800 8300 1800
 Wire Wire Line
 	8300 1800 8300 3350
 Wire Wire Line
-	3200 3350 8300 3350
-Wire Wire Line
-	8300 3350 9300 3350
-Wire Wire Line
-	1900 3550 3100 3550
-Wire Wire Line
-	3100 3550 9300 3550
-Wire Wire Line
-	1900 3650 3000 3650
-Wire Wire Line
-	3000 3650 9300 3650
-Wire Wire Line
-	1900 3750 5300 3750
-Wire Wire Line
-	5300 3750 7500 3750
-Wire Wire Line
-	7500 3750 9300 3750
-Wire Wire Line
-	1900 3850 5400 3850
-Wire Wire Line
-	5400 3850 7400 3850
-Wire Wire Line
-	7400 3850 9300 3850
-Wire Wire Line
-	1900 3950 8300 3950
-Wire Wire Line
-	8300 3950 9300 3950
-Wire Wire Line
-	1900 4050 5500 4050
-Wire Wire Line
-	5500 4050 7300 4050
-Wire Wire Line
-	7300 4050 9300 4050
-Wire Wire Line
-	1900 4150 5600 4150
-Wire Wire Line
-	5600 4150 7200 4150
-Wire Wire Line
-	7200 4150 9300 4150
+	3200 3350 9300 3350
+Wire Wire Line
+	1900 3550 9300 3550
+Wire Wire Line
+	1900 3650 9300 3650
+Wire Wire Line
+	1900 3750 9300 3750
+Wire Wire Line
+	1900 3850 9300 3850
+Wire Wire Line
+	1900 3950 9300 3950
+Wire Wire Line
+	1900 4050 9300 4050
+Wire Wire Line
+	1900 4150 9300 4150
 Wire Wire Line
 	6900 5500 7500 5500
@@
 	9300 4250 9100 4250
 Wire Wire Line
-	9100 4250 9100 4450
-Wire Wire Line
-	9100 4450 9100 4550
-Wire Wire Line
-	9100 4550 9100 6100
+	9100 4250 9100 6100
 Wire Wire Line
 	9300 4450 9100 4450

Commit message: Annotated Components
Parts:
- gave numbers to parts that had none: 12
Changed lines of the file:
@@
 $EndDescr
 $Comp
-L VBUS053CZ-HAF-G-08 U?
+L VBUS053CZ-HAF-G-08 U12
 U 1 1 5619F269
 P 3850 5150
-F 0 "U?" H 4000 5450 60  0000 C CNN
+F 0 "U12" H 4000 5450 60  0000 C CNN
 F 1 "VBUS053CZ-HAF-G-08" H 3850 4850 60  0000 C CNN
 F 2 "" H 3800 5850 60  0000 C CNN
@@
 $EndComp
 $Comp
-L VBUS054CD-FHI-GS08 U?
+L VBUS054CD-FHI-GS08 U14
 U 1 1 5619FC64
 P 6400 5300
-F 0 "U?" H 6600 5650 60  0000 C CNN
+F 0 "U14" H 6600 5650 60  0000 C CNN
 F 1 "VBUS054CD-FHI-GS08" H 6500 4950 60  0000 C CNN
 F 2 "" H 6350 6000 60  0000 C CNN
@@
 $EndComp
 $Comp
-L 692_121_030_100 CN?
+L 692_121_030_100 CN3
 U 1 1 561A064E
 P 9850 3950
-F 0 "CN?" H 10100 4700 60  0000 C CNN
+F 0 "CN3" H 10100 4700 60  0000 C CNN
 F 1 "692_121_030_100" H 9850 3200 60  0000 C CNN
 F 2 "" H 9850 3950 60  0000 C CNN
@@
 USB_H1_OC
 $Comp
-L +3V3 #PWR?
+L +3V3 #PWR118
 U 1 1 561A1B20
 P 2750 1000
-F 0 "#PWR?" H 2750 850 50  0001 C CNN
+F 0 "#PWR118" H 2750 850 50  0001 C CNN
 F 1 "+3V3" H 2750 1140 50  0000 C CNN
 F 2 "" H 2750 1000 60  0000 C CNN
@@
 $EndComp
 $Comp
-L R R?
+L R R85
 U 1 1 561A1B26
 P 2750 1200
-F 0 "R?" V 2830 1200 50  0000 C CNN
+F 0 "R85" V 2830 1200 50  0000 C CNN
 F 1 "47K" V 2750 1200 50  0000 C CNN
 F 2 "" V 2680 1200 30  0000 C CNN
@@
 $EndComp
 $Comp
-L LED D?
+L LED D15
 U 1 1 561A1B2D
 P 3100 1600
-F 0 "D?" H 3100 1700 50  0000 C CNN
+F 0 "D15" H 3100 1700 50  0000 C CNN
 F 1 "RED" H 3100 1500 50  0000 C CNN
 F 2 "" H 3100 1600 60  0000 C CNN
@@
 $EndComp
 $Comp
-L R R?
+L R R86
 U 1 1 561A1B34
 P 3100 1200
-F 0 "R?" V 3180 1200 50  0000 C CNN
+F 0 "R86" V 3180 1200 50  0000 C CNN
 F 1 "620" V 3100 1200 50  0000 C CNN
 F 2 "" V 3030 1200 30  0000 C CNN
@@
 $EndComp
 $Comp
-L +3V3 #PWR?
+L +3V3 #PWR119
 U 1 1 561A1B3B
 P 3100 1000
-F 0 "#PWR?" H 3100 850 50  0001 C CNN
+F 0 "#PWR119" H 3100 850 50  0001 C CNN
 F 1 "+3V3" H 3100 1140 50  0000 C CNN
 F 2 "" H 3100 1000 60  0000 C CNN
@@
 $EndComp
 $Comp
-L C C?
+L C C72
 U 1 1 561A1B41
 P 6900 2050
-F 0 "C?" H 6925 2150 50  0000 L CNN
+F 0 "C72" H 6925 2150 50  0000 L CNN
 F 1 "220u/6V3_T" H 6925 1950 50  0000 L CNN
 F 2 "" H 6938 1900 30  0000 C CNN
@@
 $EndComp
 $Comp
-L GND #PWR?
+L GND #PWR125
 U 1 1 561A1B48
 P 6900 2600
-F 0 "#PWR?" H 6900 2350 50  0001 C CNN
+F 0 "#PWR125" H 6900 2350 50  0001 C CNN
 F 1 "GND" H 6900 2450 50  0000 C CNN
 F 2 "" H 6900 2600 60  0000 C CNN
@@
 $EndComp
 $Comp
-L GND #PWR?
+L GND #PWR124
 U 1 1 561A1B4E
 P 5400 2600
-F 0 "#PWR?" H 5400 2350 50  0001 C CNN
+F 0 "#PWR124" H 5400 2350 50  0001 C CNN
 F 1 "GND" H 5400 2450 50  0000 C CNN
 F 2 "" H 5400 2600 60  0000 C CNN
@@
 $EndComp
 $Comp
-L +5V #PWR?
+L +5V #PWR120
 U 1 1 561A1B64
 P 3450 1000
-F 0 "#PWR?" H 3450 850 50  0001 C CNN
+F 0 "#PWR120" H 3450 850 50  0001 C CNN
 F 1 "+5V" H 3450 1140 50  0000 C CNN
 F 2 "" H 3450 1000 60  0000 C CNN
@@
 $EndComp
 $Comp
-L TPS2061CDBVT U?
+L TPS2061CDBVT U13
 U 1 1 561A1B6A
 P 4600 1900
-F 0 "U?" H 4850 2150 60  0000 C CNN
+F 0 "U13" H 4850 2150 60  0000 C CNN
 F 1 "TPS2061CDBVT" H 4600 1650 60  0000 C CNN
 F 2 "" H 4600 1700 60  0000 C CNN
@@
 $EndComp
 $Comp
-L R R?
+L R R87
 U 1 1 561A1B19
 P 3950 2300
-F 0 "R?" V 4030 2300 50  0000 C CNN
+F 0 "R87" V 4030 2300 50  0000 C CNN
 F 1 "10K" V 3950 2300 50  0000 C CNN
 F 2 "" V 3880 2300 30  0000 C CNN
@@
 $EndComp
 $Comp
-L GND #PWR?
+L GND #PWR121
 U 1 1 561A1E1C
 P 3950 2600
-F 0 "#PWR?" H 3950 2350 50  0001 C CNN
+F 0 "#PWR121" H 3950 2350 50  0001 C CNN
 F 1 "GND" H 3950 2450 50  0000 C CNN
 F 2 "" H 3950 2600 60  0000 C CNN
@@
 $EndComp
 $Comp
-L INDUCTOR L?
+L INDUCTOR L4
 U 1 1 561A2098
 P 6100 1800
-F 0 "L?" V 6050 1800 50  0000 C CNN
+F 0 "L4" V 6050 1800 50  0000 C CNN
 F 1 "BLM18EG101TN1D" V 6200 1800 50  0000 C CNN
 F 2 "" H 6100 1800 60  0000 C CNN
@@
 $EndComp
 $Comp
-L C C?
+L C C73
 U 1 1 561A223E
 P 7600 2050
-F 0 "C?" H 7625 2150 50  0000 L CNN
+F 0 "C73" H 7625 2150 50  0000 L CNN
 F 1 "100n/50V" H 7625 1950 50  0000 L CNN
 F 2 "" H 7638 1900 30  0000 C CNN
@@
 $EndComp
 $Comp
-L GND #PWR?
+L GND #PWR127
 U 1 1 561A2244
 P 7600 2600
-F 0 "#PWR?" H 7600 2350 50  0001 C CNN
+F 0 "#PWR127" H 7600 2350 50  0001 C CNN
 F 1 "GND" H 7600 2450 50  0000 C CNN
 F 2 "" H 7600 2600 60  0000 C CNN
@@
 StdA_SSTX+
 $Comp
-L INDUCTOR L?
+L INDUCTOR L5
 U 1 1 561A3280
 P 8300 4850
-F 0 "L?" V 8250 4850 50  0000 C CNN
+F 0 "L5" V 8250 4850 50  0000 C CNN
 F 1 "BLM18EG101TN1D" V 8400 4850 50  0000 C CNN
 F 2 "" H 8300 4850 60  0000 C CNN
@@
 $EndComp
 $Comp
-L GND #PWR?
+L GND #PWR128
 U 1 1 561A3388
 P 8300 6100
-F 0 "#PWR?" H 8300 5850 50  0001 C CNN
+F 0 "#PWR128" H 8300 5850 50  0001 C CNN
 F 1 "GND" H 8300 5950 50  0000 C CNN
 F 2 "" H 8300 6100 60  0000 C CNN
@@
 $EndComp
 $Comp
-L GND #PWR?
+L GND #PWR126
 U 1 1 561A33B7
 P 7500 6100
-F 0 "#PWR?" H 7500 5850 50  0001 C CNN
+F 0 "#PWR126" H 7500 5850 50  0001 C CNN
 F 1 "GND" H 7500 5950 50  0000 C CNN
 F 2 "" H 7500 6100 60  0000 C CNN
@@
 $EndComp
 $Comp
-L GND #PWR?
+L GND #PWR123
 U 1 1 561A3438
 P 5300 6100
-F 0 "#PWR?" H 5300 5850 50  0001 C CNN
+F 0 "#PWR123" H 5300 5850 50  0001 C CNN
 F 1 "GND" H 5300 5950 50  0000 C CNN
 F 2 "" H 5300 6100 60  0000 C CNN
@@
 	3200 5000 3200 3350
 $Comp
-L GND #PWR?
+L GND #PWR122
 U 1 1 561A6CE3
 P 4500 6100
-F 0 "#PWR?" H 4500 5850 50  0001 C CNN
+F 0 "#PWR122" H 4500 5850 50  0001 C CNN
 F 1 "GND" H 4500 5950 50  0000 C CNN
 F 2 "" H 4500 6100 60  0000 C CNN
@@
 NoConn ~ 3350 5300
 $Comp
-L GND #PWR?
+L GND #PWR129
 U 1 1 561A74D9
 P 9100 6100
-F 0 "#PWR?" H 9100 5850 50  0001 C CNN
+F 0 "#PWR129" H 9100 5850 50  0001 C CNN
 F 1 "GND" H 9100 5950 50  0000 C CNN
 F 2 "" H 9100 6100 60  0000 C CNN

Commit message: Re-annotated schematic
Parts:
- renumbered C72 to C70, C73 to C71, R85 to R86, R86 to R87, R87 to R88
Changed lines of the file:
@@
 USB_H1_OC
 $Comp
-L +3V3 #PWR0120
+L +3V3 #PWR115
 U 1 1 561A1B20
 P 2750 1000
-F 0 "#PWR0120" H 2750 850 50  0001 C CNN
+F 0 "#PWR115" H 2750 850 50  0001 C CNN
 F 1 "+3V3" H 2750 1140 50  0000 C CNN
 F 2 "" H 2750 1000 60  0000 C CNN
@@
 $EndComp
 $Comp
-L R R85
+L R R86
 U 1 1 561A1B26
 P 2750 1200
-F 0 "R85" V 2830 1200 50  0000 C CNN
+F 0 "R86" V 2830 1200 50  0000 C CNN
 F 1 "47K" V 2750 1200 50  0000 C CNN
 F 2 "" V 2680 1200 30  0000 C CNN
@@
 $EndComp
 $Comp
-L R R86
+L R R87
 U 1 1 561A1B34
 P 3100 1200
-F 0 "R86" V 3180 1200 50  0000 C CNN
+F 0 "R87" V 3180 1200 50  0000 C CNN
 F 1 "620" V 3100 1200 50  0000 C CNN
 F 2 "" V 3030 1200 30  0000 C CNN
@@
 $EndComp
 $Comp
-L +3V3 #PWR0121
+L +3V3 #PWR116
 U 1 1 561A1B3B
 P 3100 1000
-F 0 "#PWR0121" H 3100 850 50  0001 C CNN
+F 0 "#PWR116" H 3100 850 50  0001 C CNN
 F 1 "+3V3" H 3100 1140 50  0000 C CNN
 F 2 "" H 3100 1000 60  0000 C CNN
@@
 $EndComp
 $Comp
-L C C72
+L C C70
 U 1 1 561A1B41
 P 6900 2050
-F 0 "C72" H 6925 2150 50  0000 L CNN
+F 0 "C70" H 6925 2150 50  0000 L CNN
 F 1 "220u/6V3_T" H 6925 1950 50  0000 L CNN
 F 2 "" H 6938 1900 30  0000 C CNN
@@
 $EndComp
 $Comp
-L GND #PWR0122
+L GND #PWR122
 U 1 1 561A1B48
 P 6900 2600
-F 0 "#PWR0122" H 6900 2350 50  0001 C CNN
+F 0 "#PWR122" H 6900 2350 50  0001 C CNN
 F 1 "GND" H 6900 2450 50  0000 C CNN
 F 2 "" H 6900 2600 60  0000 C CNN
@@
 $EndComp
 $Comp
-L GND #PWR0123
+L GND #PWR121
 U 1 1 561A1B4E
 P 5400 2600
-F 0 "#PWR0123" H 5400 2350 50  0001 C CNN
+F 0 "#PWR121" H 5400 2350 50  0001 C CNN
 F 1 "GND" H 5400 2450 50  0000 C CNN
 F 2 "" H 5400 2600 60  0000 C CNN
@@
 $EndComp
 $Comp
-L +5V #PWR0124
+L +5V #PWR117
 U 1 1 561A1B64
 P 3450 1000
-F 0 "#PWR0124" H 3450 850 50  0001 C CNN
+F 0 "#PWR117" H 3450 850 50  0001 C CNN
 F 1 "+5V" H 3450 1140 50  0000 C CNN
 F 2 "" H 3450 1000 60  0000 C CNN
@@
 $EndComp
 $Comp
-L R R87
+L R R88
 U 1 1 561A1B19
 P 3950 2300
-F 0 "R87" V 4030 2300 50  0000 C CNN
+F 0 "R88" V 4030 2300 50  0000 C CNN
 F 1 "10K" V 3950 2300 50  0000 C CNN
 F 2 "" V 3880 2300 30  0000 C CNN
@@
 $EndComp
 $Comp
-L GND #PWR0125
+L GND #PWR118
 U 1 1 561A1E1C
 P 3950 2600
-F 0 "#PWR0125" H 3950 2350 50  0001 C CNN
+F 0 "#PWR118" H 3950 2350 50  0001 C CNN
 F 1 "GND" H 3950 2450 50  0000 C CNN
 F 2 "" H 3950 2600 60  0000 C CNN
@@
 $EndComp
 $Comp
-L C C73
+L C C71
 U 1 1 561A223E
 P 7600 2050
-F 0 "C73" H 7625 2150 50  0000 L CNN
+F 0 "C71" H 7625 2150 50  0000 L CNN
 F 1 "100n/50V" H 7625 1950 50  0000 L CNN
 F 2 "" H 7638 1900 30  0000 C CNN
@@
 $EndComp
 $Comp
-L GND #PWR0126
+L GND #PWR124
 U 1 1 561A2244
 P 7600 2600
-F 0 "#PWR0126" H 7600 2350 50  0001 C CNN
+F 0 "#PWR124" H 7600 2350 50  0001 C CNN
 F 1 "GND" H 7600 2450 50  0000 C CNN
 F 2 "" H 7600 2600 60  0000 C CNN
@@
 $EndComp
 $Comp
-L GND #PWR0127
+L GND #PWR125
 U 1 1 561A3388
 P 8300 6100
-F 0 "#PWR0127" H 8300 5850 50  0001 C CNN
+F 0 "#PWR125" H 8300 5850 50  0001 C CNN
 F 1 "GND" H 8300 5950 50  0000 C CNN
 F 2 "" H 8300 6100 60  0000 C CNN
@@
 $EndComp
 $Comp
-L GND #PWR0128
+L GND #PWR123
 U 1 1 561A33B7
 P 7500 6100
-F 0 "#PWR0128" H 7500 5850 50  0001 C CNN
+F 0 "#PWR123" H 7500 5850 50  0001 C CNN
 F 1 "GND" H 7500 5950 50  0000 C CNN
 F 2 "" H 7500 6100 60  0000 C CNN
@@
 $EndComp
 $Comp
-L GND #PWR0129
+L GND #PWR120
 U 1 1 561A3438
 P 5300 6100
-F 0 "#PWR0129" H 5300 5850 50  0001 C CNN
+F 0 "#PWR120" H 5300 5850 50  0001 C CNN
 F 1 "GND" H 5300 5950 50  0000 C CNN
 F 2 "" H 5300 6100 60  0000 C CNN
@@
 	3200 5000 3200 3350
 $Comp
-L GND #PWR0130
+L GND #PWR119
 U 1 1 561A6CE3
 P 4500 6100
-F 0 "#PWR0130" H 4500 5850 50  0001 C CNN
+F 0 "#PWR119" H 4500 5850 50  0001 C CNN
 F 1 "GND" H 4500 5950 50  0000 C CNN
 F 2 "" H 4500 6100 60  0000 C CNN
@@
 NoConn ~ 3350 5300
 $Comp
-L GND #PWR0131
+L GND #PWR126
 U 1 1 561A74D9
 P 9100 6100
-F 0 "#PWR0131" H 9100 5850 50  0001 C CNN
+F 0 "#PWR126" H 9100 5850 50  0001 C CNN
 F 1 "GND" H 9100 5950 50  0000 C CNN
 F 2 "" H 9100 6100 60  0000 C CNN

Commit message: Associated footprints for R and some of the C
Parts:
- R86, R87, R88: footprint (none) -> Resistors_SMD:R_0603
Changed lines of the file:
@@
 F 0 "U12" H 4000 5450 60  0000 C CNN
 F 1 "VBUS053CZ-HAF-G-08" H 3850 4850 60  0000 C CNN
-F 2 "" H 3800 5850 60  0000 C CNN
+F 2 "" H 3800 5850 60  0001 C CNN
 F 3 "" H 3800 5850 60  0000 C CNN
 	1    3850 5150
@@
 F 0 "U14" H 6600 5650 60  0000 C CNN
 F 1 "VBUS054CD-FHI-GS08" H 6500 4950 60  0000 C CNN
-F 2 "" H 6350 6000 60  0000 C CNN
+F 2 "" H 6350 6000 60  0001 C CNN
 F 3 "" H 6350 6000 60  0000 C CNN
 	1    6400 5300
@@
 F 0 "CN3" H 10100 4700 60  0000 C CNN
 F 1 "692_121_030_100" H 9850 3200 60  0000 C CNN
-F 2 "" H 9850 3950 60  0000 C CNN
+F 2 "" H 9850 3950 60  0001 C CNN
 F 3 "" H 9850 3950 60  0000 C CNN
 	1    9850 3950
@@
 USB_H1_OC
 $Comp
-L +3V3 #PWR115
+L +3V3 #PWR0117
 U 1 1 561A1B20
 P 2750 1000
-F 0 "#PWR115" H 2750 850 50  0001 C CNN
+F 0 "#PWR0117" H 2750 850 50  0001 C CNN
 F 1 "+3V3" H 2750 1140 50  0000 C CNN
 F 2 "" H 2750 1000 60  0000 C CNN
@@
 F 0 "R86" V 2830 1200 50  0000 C CNN
 F 1 "47K" V 2750 1200 50  0000 C CNN
-F 2 "" V 2680 1200 30  0000 C CNN
+F 2 "Resistors_SMD:R_0603" V 2680 1200 30  0001 C CNN
 F 3 "" H 2750 1200 30  0000 C CNN
 	1    2750 1200
@@
 F 0 "D15" H 3100 1700 50  0000 C CNN
 F 1 "RED" H 3100 1500 50  0000 C CNN
-F 2 "" H 3100 1600 60  0000 C CNN
+F 2 "" H 3100 1600 60  0001 C CNN
 F 3 "" H 3100 1600 60  0000 C CNN
 	1    3100 1600
@@
 F 0 "R87" V 3180 1200 50  0000 C CNN
 F 1 "620" V 3100 1200 50  0000 C CNN
-F 2 "" V 3030 1200 30  0000 C CNN
+F 2 "Resistors_SMD:R_0603" V 3030 1200 30  0001 C CNN
 F 3 "" H 3100 1200 30  0000 C CNN
 	1    3100 1200
@@
 $EndComp
 $Comp
-L +3V3 #PWR116
+L +3V3 #PWR0118
 U 1 1 561A1B3B
 P 3100 1000
-F 0 "#PWR116" H 3100 850 50  0001 C CNN
+F 0 "#PWR0118" H 3100 850 50  0001 C CNN
 F 1 "+3V3" H 3100 1140 50  0000 C CNN
 F 2 "" H 3100 1000 60  0000 C CNN
@@
 F 0 "C70" H 6925 2150 50  0000 L CNN
 F 1 "220u/6V3_T" H 6925 1950 50  0000 L CNN
-F 2 "" H 6938 1900 30  0000 C CNN
+F 2 "" H 6938 1900 30  0001 C CNN
 F 3 "" H 6900 2050 60  0000 C CNN
 	1    6900 2050
@@
 $EndComp
 $Comp
-L GND #PWR122
+L GND #PWR0119
 U 1 1 561A1B48
 P 6900 2600
-F 0 "#PWR122" H 6900 2350 50  0001 C CNN
+F 0 "#PWR0119" H 6900 2350 50  0001 C CNN
 F 1 "GND" H 6900 2450 50  0000 C CNN
 F 2 "" H 6900 2600 60  0000 C CNN
@@
 $EndComp
 $Comp
-L GND #PWR121
+L GND #PWR0120
 U 1 1 561A1B4E
 P 5400 2600
-F 0 "#PWR121" H 5400 2350 50  0001 C CNN
+F 0 "#PWR0120" H 5400 2350 50  0001 C CNN
 F 1 "GND" H 5400 2450 50  0000 C CNN
 F 2 "" H 5400 2600 60  0000 C CNN
@@
 $EndComp
 $Comp
-L +5V #PWR117
+L +5V #PWR0121
 U 1 1 561A1B64
 P 3450 1000
-F 0 "#PWR117" H 3450 850 50  0001 C CNN
+F 0 "#PWR0121" H 3450 850 50  0001 C CNN
 F 1 "+5V" H 3450 1140 50  0000 C CNN
 F 2 "" H 3450 1000 60  0000 C CNN
@@
 F 0 "U13" H 4850 2150 60  0000 C CNN
 F 1 "TPS2061CDBVT" H 4600 1650 60  0000 C CNN
-F 2 "" H 4600 1700 60  0000 C CNN
+F 2 "" H 4600 1700 60  0001 C CNN
 F 3 "" H 4600 1700 60  0000 C CNN
 	1    4600 1900
@@
 F 0 "R88" V 4030 2300 50  0000 C CNN
 F 1 "10K" V 3950 2300 50  0000 C CNN
-F 2 "" V 3880 2300 30  0000 C CNN
+F 2 "Resistors_SMD:R_0603" V 3880 2300 30  0001 C CNN
 F 3 "" H 3950 2300 30  0000 C CNN
 	1    3950 2300
@@
 $EndComp
 $Comp
-L GND #PWR118
+L GND #PWR0122
 U 1 1 561A1E1C
 P 3950 2600
-F 0 "#PWR118" H 3950 2350 50  0001 C CNN
+F 0 "#PWR0122" H 3950 2350 50  0001 C CNN
 F 1 "GND" H 3950 2450 50  0000 C CNN
 F 2 "" H 3950 2600 60  0000 C CNN
@@
 F 0 "L4" V 6050 1800 50  0000 C CNN
 F 1 "BLM18EG101TN1D" V 6200 1800 50  0000 C CNN
-F 2 "" H 6100 1800 60  0000 C CNN
+F 2 "" H 6100 1800 60  0001 C CNN
 F 3 "" H 6100 1800 60  0000 C CNN
 	1    6100 1800
@@
 F 0 "C71" H 7625 2150 50  0000 L CNN
 F 1 "100n/50V" H 7625 1950 50  0000 L CNN
-F 2 "" H 7638 1900 30  0000 C CNN
+F 2 "" H 7638 1900 30  0001 C CNN
 F 3 "" H 7600 2050 60  0000 C CNN
 	1    7600 2050
@@
 $EndComp
 $Comp
-L GND #PWR124
+L GND #PWR0123
 U 1 1 561A2244
 P 7600 2600
-F 0 "#PWR124" H 7600 2350 50  0001 C CNN
+F 0 "#PWR0123" H 7600 2350 50  0001 C CNN
 F 1 "GND" H 7600 2450 50  0000 C CNN
 F 2 "" H 7600 2600 60  0000 C CNN
@@
 F 0 "L5" V 8250 4850 50  0000 C CNN
 F 1 "BLM18EG101TN1D" V 8400 4850 50  0000 C CNN
-F 2 "" H 8300 4850 60  0000 C CNN
+F 2 "" H 8300 4850 60  0001 C CNN
 F 3 "" H 8300 4850 60  0000 C CNN
 	1    8300 4850
@@
 $EndComp
 $Comp
-L GND #PWR125
+L GND #PWR0124
 U 1 1 561A3388
 P 8300 6100
-F 0 "#PWR125" H 8300 5850 50  0001 C CNN
+F 0 "#PWR0124" H 8300 5850 50  0001 C CNN
 F 1 "GND" H 8300 5950 50  0000 C CNN
 F 2 "" H 8300 6100 60  0000 C CNN
@@
 $EndComp
 $Comp
-L GND #PWR123
+L GND #PWR0125
 U 1 1 561A33B7
 P 7500 6100
-F 0 "#PWR123" H 7500 5850 50  0001 C CNN
+F 0 "#PWR0125" H 7500 5850 50  0001 C CNN
 F 1 "GND" H 7500 5950 50  0000 C CNN
 F 2 "" H 7500 6100 60  0000 C CNN
@@
 $EndComp
 $Comp
-L GND #PWR120
+L GND #PWR0126
 U 1 1 561A3438
 P 5300 6100
-F 0 "#PWR120" H 5300 5850 50  0001 C CNN
+F 0 "#PWR0126" H 5300 5850 50  0001 C CNN
 F 1 "GND" H 5300 5950 50  0000 C CNN
 F 2 "" H 5300 6100 60  0000 C CNN
@@
 	3200 5000 3200 3350
 $Comp
-L GND #PWR119
+L GND #PWR0127
 U 1 1 561A6CE3
 P 4500 6100
-F 0 "#PWR119" H 4500 5850 50  0001 C CNN
+F 0 "#PWR0127" H 4500 5850 50  0001 C CNN
 F 1 "GND" H 4500 5950 50  0000 C CNN
 F 2 "" H 4500 6100 60  0000 C CNN
@@
 NoConn ~ 3350 5300
 $Comp
-L GND #PWR126
+L GND #PWR0128
 U 1 1 561A74D9
 P 9100 6100
-F 0 "#PWR126" H 9100 5850 50  0001 C CNN
+F 0 "#PWR0128" H 9100 5850 50  0001 C CNN
 F 1 "GND" H 9100 5950 50  0000 C CNN
 F 2 "" H 9100 6100 60  0000 C CNN

Commit message: Work on cortex USB connection.
Parts:
- renumbered C70 to C?, C71 to C?, CN3 to CN?, D15 to D?, L4 to L?, L5 to L?, R88 to R?, R86 to R?, R87 to R?, U12 to U?, U14 to U?, U13 to U?
Changed lines of the file:
@@
 $EndDescr
 $Comp
-L VBUS053CZ-HAF-G-08 U12
+L VBUS053CZ-HAF-G-08 U?
 U 1 1 5619F269
 P 3850 5150
-F 0 "U12" H 4000 5450 60  0000 C CNN
+F 0 "U?" H 4000 5450 60  0000 C CNN
 F 1 "VBUS053CZ-HAF-G-08" H 3850 4850 60  0000 C CNN
 F 2 "" H 3800 5850 60  0001 C CNN
@@
 $EndComp
 $Comp
-L VBUS054CD-FHI-GS08 U14
+L VBUS054CD-FHI-GS08 U?
 U 1 1 5619FC64
 P 6400 5300
-F 0 "U14" H 6600 5650 60  0000 C CNN
+F 0 "U?" H 6600 5650 60  0000 C CNN
 F 1 "VBUS054CD-FHI-GS08" H 6500 4950 60  0000 C CNN
 F 2 "" H 6350 6000 60  0001 C CNN
@@
 $EndComp
 $Comp
-L 692_121_030_100 CN3
+L 692_121_030_100 CN?
 U 1 1 561A064E
 P 9850 3950
-F 0 "CN3" H 10100 4700 60  0000 C CNN
+F 0 "CN?" H 10100 4700 60  0000 C CNN
 F 1 "692_121_030_100" H 9850 3200 60  0000 C CNN
 F 2 "" H 9850 3950 60  0001 C CNN
@@
 USB_H1_OC
 $Comp
-L +3V3 #PWR0117
+L +3V3 #PWR?
 U 1 1 561A1B20
 P 2750 1000
-F 0 "#PWR0117" H 2750 850 50  0001 C CNN
+F 0 "#PWR?" H 2750 850 50  0001 C CNN
 F 1 "+3V3" H 2750 1140 50  0000 C CNN
 F 2 "" H 2750 1000 60  0000 C CNN
@@
 $EndComp
 $Comp
-L R R86
+L R R?
 U 1 1 561A1B26
 P 2750 1200
-F 0 "R86" V 2830 1200 50  0000 C CNN
+F 0 "R?" V 2830 1200 50  0000 C CNN
 F 1 "47K" V 2750 1200 50  0000 C CNN
 F 2 "Resistors_SMD:R_0603" V 2680 1200 30  0001 C CNN
@@
 $EndComp
 $Comp
-L LED D15
+L LED D?
 U 1 1 561A1B2D
 P 3100 1600
-F 0 "D15" H 3100 1700 50  0000 C CNN
+F 0 "D?" H 3100 1700 50  0000 C CNN
 F 1 "RED" H 3100 1500 50  0000 C CNN
 F 2 "" H 3100 1600 60  0001 C CNN
@@
 $EndComp
 $Comp
-L R R87
+L R R?
 U 1 1 561A1B34
 P 3100 1200
-F 0 "R87" V 3180 1200 50  0000 C CNN
+F 0 "R?" V 3180 1200 50  0000 C CNN
 F 1 "620" V 3100 1200 50  0000 C CNN
 F 2 "Resistors_SMD:R_0603" V 3030 1200 30  0001 C CNN
@@
 $EndComp
 $Comp
-L +3V3 #PWR0118
+L +3V3 #PWR?
 U 1 1 561A1B3B
 P 3100 1000
-F 0 "#PWR0118" H 3100 850 50  0001 C CNN
+F 0 "#PWR?" H 3100 850 50  0001 C CNN
 F 1 "+3V3" H 3100 1140 50  0000 C CNN
 F 2 "" H 3100 1000 60  0000 C CNN
@@
 $EndComp
 $Comp
-L C C70
+L C C?
 U 1 1 561A1B41
 P 6900 2050
-F 0 "C70" H 6925 2150 50  0000 L CNN
+F 0 "C?" H 6925 2150 50  0000 L CNN
 F 1 "220u/6V3_T" H 6925 1950 50  0000 L CNN
 F 2 "" H 6938 1900 30  0001 C CNN
@@
 $EndComp
 $Comp
-L GND #PWR0119
+L GND #PWR?
 U 1 1 561A1B48
 P 6900 2600
-F 0 "#PWR0119" H 6900 2350 50  0001 C CNN
+F 0 "#PWR?" H 6900 2350 50  0001 C CNN
 F 1 "GND" H 6900 2450 50  0000 C CNN
 F 2 "" H 6900 2600 60  0000 C CNN
@@
 $EndComp
 $Comp
-L GND #PWR0120
+L GND #PWR?
 U 1 1 561A1B4E
 P 5400 2600
-F 0 "#PWR0120" H 5400 2350 50  0001 C CNN
+F 0 "#PWR?" H 5400 2350 50  0001 C CNN
 F 1 "GND" H 5400 2450 50  0000 C CNN
 F 2 "" H 5400 2600 60  0000 C CNN
@@
 $EndComp
 $Comp
-L +5V #PWR0121
+L +5V #PWR?
 U 1 1 561A1B64
 P 3450 1000
-F 0 "#PWR0121" H 3450 850 50  0001 C CNN
+F 0 "#PWR?" H 3450 850 50  0001 C CNN
 F 1 "+5V" H 3450 1140 50  0000 C CNN
 F 2 "" H 3450 1000 60  0000 C CNN
@@
 $EndComp
 $Comp
-L TPS2061CDBVT U13
+L TPS2061CDBVT U?
 U 1 1 561A1B6A
 P 4600 1900
-F 0 "U13" H 4850 2150 60  0000 C CNN
+F 0 "U?" H 4850 2150 60  0000 C CNN
 F 1 "TPS2061CDBVT" H 4600 1650 60  0000 C CNN
 F 2 "" H 4600 1700 60  0001 C CNN
@@
 $EndComp
 $Comp
-L R R88
+L R R?
 U 1 1 561A1B19
 P 3950 2300
-F 0 "R88" V 4030 2300 50  0000 C CNN
+F 0 "R?" V 4030 2300 50  0000 C CNN
 F 1 "10K" V 3950 2300 50  0000 C CNN
 F 2 "Resistors_SMD:R_0603" V 3880 2300 30  0001 C CNN
@@
 $EndComp
 $Comp
-L GND #PWR0122
+L GND #PWR?
 U 1 1 561A1E1C
 P 3950 2600
-F 0 "#PWR0122" H 3950 2350 50  0001 C CNN
+F 0 "#PWR?" H 3950 2350 50  0001 C CNN
 F 1 "GND" H 3950 2450 50  0000 C CNN
 F 2 "" H 3950 2600 60  0000 C CNN
@@
 $EndComp
 $Comp
-L INDUCTOR L4
+L INDUCTOR L?
 U 1 1 561A2098
 P 6100 1800
-F 0 "L4" V 6050 1800 50  0000 C CNN
+F 0 "L?" V 6050 1800 50  0000 C CNN
 F 1 "BLM18EG101TN1D" V 6200 1800 50  0000 C CNN
 F 2 "" H 6100 1800 60  0001 C CNN
@@
 $EndComp
 $Comp
-L C C71
+L C C?
 U 1 1 561A223E
 P 7600 2050
-F 0 "C71" H 7625 2150 50  0000 L CNN
+F 0 "C?" H 7625 2150 50  0000 L CNN
 F 1 "100n/50V" H 7625 1950 50  0000 L CNN
 F 2 "" H 7638 1900 30  0001 C CNN
@@
 $EndComp
 $Comp
-L GND #PWR0123
+L GND #PWR?
 U 1 1 561A2244
 P 7600 2600
-F 0 "#PWR0123" H 7600 2350 50  0001 C CNN
+F 0 "#PWR?" H 7600 2350 50  0001 C CNN
 F 1 "GND" H 7600 2450 50  0000 C CNN
 F 2 "" H 7600 2600 60  0000 C CNN
@@
 StdA_SSTX+
 $Comp
-L INDUCTOR L5
+L INDUCTOR L?
 U 1 1 561A3280
 P 8300 4850
-F 0 "L5" V 8250 4850 50  0000 C CNN
+F 0 "L?" V 8250 4850 50  0000 C CNN
 F 1 "BLM18EG101TN1D" V 8400 4850 50  0000 C CNN
 F 2 "" H 8300 4850 60  0001 C CNN
@@
 $EndComp
 $Comp
-L GND #PWR0124
+L GND #PWR?
 U 1 1 561A3388
 P 8300 6100
-F 0 "#PWR0124" H 8300 5850 50  0001 C CNN
+F 0 "#PWR?" H 8300 5850 50  0001 C CNN
 F 1 "GND" H 8300 5950 50  0000 C CNN
 F 2 "" H 8300 6100 60  0000 C CNN
@@
 $EndComp
 $Comp
-L GND #PWR0125
+L GND #PWR?
 U 1 1 561A33B7
 P 7500 6100
-F 0 "#PWR0125" H 7500 5850 50  0001 C CNN
+F 0 "#PWR?" H 7500 5850 50  0001 C CNN
 F 1 "GND" H 7500 5950 50  0000 C CNN
 F 2 "" H 7500 6100 60  0000 C CNN
@@
 $EndComp
 $Comp
-L GND #PWR0126
+L GND #PWR?
 U 1 1 561A3438
 P 5300 6100
-F 0 "#PWR0126" H 5300 5850 50  0001 C CNN
+F 0 "#PWR?" H 5300 5850 50  0001 C CNN
 F 1 "GND" H 5300 5950 50  0000 C CNN
 F 2 "" H 5300 6100 60  0000 C CNN
@@
 	3200 5000 3200 3350
 $Comp
-L GND #PWR0127
+L GND #PWR?
 U 1 1 561A6CE3
 P 4500 6100
-F 0 "#PWR0127" H 4500 5850 50  0001 C CNN
+F 0 "#PWR?" H 4500 5850 50  0001 C CNN
 F 1 "GND" H 4500 5950 50  0000 C CNN
 F 2 "" H 4500 6100 60  0000 C CNN
@@
 NoConn ~ 3350 5300
 $Comp
-L GND #PWR0128
+L GND #PWR?
 U 1 1 561A74D9
 P 9100 6100
-F 0 "#PWR0128" H 9100 5850 50  0001 C CNN
+F 0 "#PWR?" H 9100 5850 50  0001 C CNN
 F 1 "GND" H 9100 5950 50  0000 C CNN
 F 2 "" H 9100 6100 60  0000 C CNN
