File: hardware/colibri-v2/wnd_usb_host.sch (KiCad schematic (older format))
At the start: 12 parts

Commit message: Work on the Cortex sheet
Parts:
- removed C?: 220u/6V3_T, symbol C
- removed C?: 100n/50V, symbol C
- removed D?: RED, symbol LED
- removed L? (x2): BLM18EG101TN1D, symbol INDUCTOR
- removed R?: 10K, Resistors_SMD:R_0603, symbol R
- removed R?: 47K, Resistors_SMD:R_0603, symbol R
- removed R?: 620, Resistors_SMD:R_0603, symbol R
- added C?: 100nF/50V/X7R, Capacitors_SMD:C_0603, symbol C_SMT
- added C?: 220uF/10%/6V3, Capacitors_Tantalum_SMD:TantalC_SizeC_EIA-6032_Reflow, symbol CP_SMT
- added DL?: RED, LEDs:LED-0603, symbol LED_SMT
- added FB? (x2): BEAD/0.045OHM/2A, Resistors_SMD:R_0603, symbol FB_SMT
- added R?: 47K/5%, Resistors_SMD:R_0603, symbol R_SMT
- added R?: 620R/5%, Resistors_SMD:R_0603, symbol R_SMT
- added R?: 10K/5%, Resistors_SMD:R_0603, symbol R_SMT
Connections:
- net +3V3: now also R?.1, R?.1
- net GND: now also C?.2, C?.2, FB?.2, R?.2
- net GND_DRAIN: now also FB?.1
- net USB_H1_OC: now also DL?.1 (K), R?.2
- net at CN?.1 (VCC), U?.6 (VBUUS): now also C?.1, C?.1, FB?.2
- net at U?.4 (~EN): now also R?.1
- net at U?.1 (OUT): now also FB?.1
- new net: DL?.2 (A), R?.2
Changed lines of the file:
@@
-$EndComp
-$Comp
-L R R?
-U 1 1 561A1B26
-P 2750 1200
-F 0 "R?" V 2830 1200 50  0000 C CNN
-F 1 "47K" V 2750 1200 50  0000 C CNN
-F 2 "Resistors_SMD:R_0603" V 2680 1200 30  0001 C CNN
-F 3 "" H 2750 1200 30  0000 C CNN
-	1    2750 1200
-	1    0    0    -1
-$EndComp
-$Comp
-L LED D?
-U 1 1 561A1B2D
-P 3100 1600
-F 0 "D?" H 3100 1700 50  0000 C CNN
-F 1 "RED" H 3100 1500 50  0000 C CNN
-F 2 "" H 3100 1600 60  0001 C CNN
-F 3 "" H 3100 1600 60  0000 C CNN
-	1    3100 1600
-	0    -1   -1   0
-$EndComp
-$Comp
-L R R?
-U 1 1 561A1B34
-P 3100 1200
-F 0 "R?" V 3180 1200 50  0000 C CNN
-F 1 "620" V 3100 1200 50  0000 C CNN
-F 2 "Resistors_SMD:R_0603" V 3030 1200 30  0001 C CNN
-F 3 "" H 3100 1200 30  0000 C CNN
-	1    3100 1200
-	1    0    0    -1
 $EndComp
 $Comp
@@
 $EndComp
 $Comp
-L C C?
-U 1 1 561A1B41
-P 6900 2050
-F 0 "C?" H 6925 2150 50  0000 L CNN
-F 1 "220u/6V3_T" H 6925 1950 50  0000 L CNN
-F 2 "" H 6938 1900 30  0001 C CNN
-F 3 "" H 6900 2050 60  0000 C CNN
-	1    6900 2050
-	1    0    0    -1
-$EndComp
-$Comp
 L GND #PWR?
 U 1 1 561A1B48
@@
 $EndComp
 $Comp
-L R R?
-U 1 1 561A1B19
-P 3950 2300
-F 0 "R?" V 4030 2300 50  0000 C CNN
-F 1 "10K" V 3950 2300 50  0000 C CNN
-F 2 "Resistors_SMD:R_0603" V 3880 2300 30  0001 C CNN
-F 3 "" H 3950 2300 30  0000 C CNN
-	1    3950 2300
-	1    0    0    -1
-$EndComp
-$Comp
 L GND #PWR?
 U 1 1 561A1E1C
@@
 F 3 "" H 3950 2600 60  0000 C CNN
 	1    3950 2600
-	1    0    0    -1
-$EndComp
-$Comp
-L INDUCTOR L?
-U 1 1 561A2098
-P 6100 1800
-F 0 "L?" V 6050 1800 50  0000 C CNN
-F 1 "BLM18EG101TN1D" V 6200 1800 50  0000 C CNN
-F 2 "" H 6100 1800 60  0001 C CNN
-F 3 "" H 6100 1800 60  0000 C CNN
-	1    6100 1800
-	0    -1   -1   0
-$EndComp
-$Comp
-L C C?
-U 1 1 561A223E
-P 7600 2050
-F 0 "C?" H 7625 2150 50  0000 L CNN
-F 1 "100n/50V" H 7625 1950 50  0000 L CNN
-F 2 "" H 7638 1900 30  0001 C CNN
-F 3 "" H 7600 2050 60  0000 C CNN
-	1    7600 2050
 	1    0    0    -1
 $EndComp
@@
 StdA_SSTX+
 $Comp
-L INDUCTOR L?
-U 1 1 561A3280
-P 8300 4850
-F 0 "L?" V 8250 4850 50  0000 C CNN
-F 1 "BLM18EG101TN1D" V 8400 4850 50  0000 C CNN
-F 2 "" H 8300 4850 60  0001 C CNN
-F 3 "" H 8300 4850 60  0000 C CNN
-	1    8300 4850
-	-1   0    0    1
-$EndComp
-$Comp
 L GND #PWR?
 U 1 1 561A3388
@@
 $EndComp
 Wire Wire Line
-	1900 2000 4100 2000
+	1900 2000 2750 2000
+Wire Wire Line
+	2750 2000 3100 2000
+Wire Wire Line
+	3100 2000 4100 2000
 Wire Wire Line
 	2750 1000 2750 1050
@@
 	5100 1800 5800 1800
 Wire Wire Line
-	6400 1800 8300 1800
+	6200 1800 6900 1800
+Wire Wire Line
+	6900 1800 7600 1800
+Wire Wire Line
+	7600 1800 8300 1800
 Wire Wire Line
 	8300 1800 8300 3350
 Wire Wire Line
-	3200 3350 9300 3350
-Wire Wire Line
-	1900 3550 9300 3550
-Wire Wire Line
-	1900 3650 9300 3650
-Wire Wire Line
-	1900 3750 9300 3750
-Wire Wire Line
-	1900 3850 9300 3850
-Wire Wire Line
-	1900 3950 9300 3950
-Wire Wire Line
-	1900 4050 9300 4050
-Wire Wire Line
-	1900 4150 9300 4150
+	3200 3350 8300 3350
+Wire Wire Line
+	8300 3350 9300 3350
+Wire Wire Line
+	1900 3550 3100 3550
+Wire Wire Line
+	3100 3550 9300 3550
+Wire Wire Line
+	1900 3650 3000 3650
+Wire Wire Line
+	3000 3650 9300 3650
+Wire Wire Line
+	1900 3750 5300 3750
+Wire Wire Line
+	5300 3750 7500 3750
+Wire Wire Line
+	7500 3750 9300 3750
+Wire Wire Line
+	1900 3850 5400 3850
+Wire Wire Line
+	5400 3850 7400 3850
+Wire Wire Line
+	7400 3850 9300 3850
+Wire Wire Line
+	1900 3950 8300 3950
+Wire Wire Line
+	8300 3950 9300 3950
+Wire Wire Line
+	1900 4050 5500 4050
+Wire Wire Line
+	5500 4050 7300 4050
+Wire Wire Line
+	7300 4050 9300 4050
+Wire Wire Line
+	1900 4150 5600 4150
+Wire Wire Line
+	5600 4150 7200 4150
+Wire Wire Line
+	7200 4150 9300 4150
 Wire Wire Line
 	6900 5500 7500 5500
@@
 	5300 5500 5300 6100
 Wire Wire Line
-	8300 5150 8300 6100
+	8300 4950 8300 6100
 Wire Wire Line
 	5900 5100 5600 5100
@@
 	9300 4250 9100 4250
 Wire Wire Line
-	9100 4250 9100 6100
+	9100 4250 9100 4450
+Wire Wire Line
+	9100 4450 9100 4550
+Wire Wire Line
+	9100 4550 9100 6100
 Wire Wire Line
 	9300 4450 9100 4450
@@
 	9300 4550 9100 4550
 Connection ~ 9100 4550
+$Comp
+L R_SMT R?
+U 1 1 56350B75
+P 2750 1200
+F 0 "R?" H 2800 1350 50  0000 C CNN
+F 1 "47K/5%" V 2680 1200 50  0000 C CNN
+F 2 "Resistors_SMD:R_0603" V 2900 1200 30  0001 C CNN
+F 3 "" V 2830 1200 30  0000 C CNN
+F 4 "0603" V 2750 1200 20  0000 C CNN "SMT"
+F 5 "9332162" V 2950 1200 30  0001 C CNN "Part"
+F 6 "Farnell" V 3000 1200 30  0001 C CNN "Provider"
+	1    2750 1200
+	1    0    0    -1
+$EndComp
+$Comp
+L R_SMT R?
+U 1 1 563513C2
+P 3100 1200
+F 0 "R?" H 3150 1350 50  0000 C CNN
+F 1 "620R/5%" V 3030 1200 50  0000 C CNN
+F 2 "Resistors_SMD:R_0603" V 3250 1200 30  0001 C CNN
+F 3 "" V 3180 1200 30  0000 C CNN
+F 4 "0603" V 3100 1200 20  0000 C CNN "SMT"
+F 5 "2141352" V 3300 1200 30  0001 C CNN "Part"
+F 6 "Farnell" V 3350 1200 30  0001 C CNN "Provider"
+	1    3100 1200
+	1    0    0    -1
+$EndComp
+$Comp
+L LED_SMT DL?
+U 1 1 563518B5
+P 3100 1600
+F 0 "DL?" V 3200 1700 50  0000 C CNN
+F 1 "RED" H 3100 1500 50  0000 C CNN
+F 2 "LEDs:LED-0603" H 3100 1450 30  0001 C CNN
+F 3 "" H 3100 1600 60  0000 C CNN
+F 4 "0603" H 2985 1580 30  0000 C CNN "SMT"
+F 5 "2322071" H 3100 1400 30  0001 C CNN "Part"
+F 6 "Farnell" H 3100 1350 30  0001 C CNN "Provider"
+	1    3100 1600
+	0    1    -1   0
+$EndComp
+$Comp
+L R_SMT R?
+U 1 1 563526BF
+P 3950 2300
+F 0 "R?" H 4000 2450 50  0000 C CNN
+F 1 "10K/5%" V 3850 2300 50  0000 C CNN
+F 2 "Resistors_SMD:R_0603" V 4100 2300 30  0001 C CNN
+F 3 "" V 4030 2300 30  0000 C CNN
+F 4 "0603" V 3950 2300 20  0000 C CNN "SMT"
+F 5 "9331700" V 4150 2300 30  0001 C CNN "Part"
+F 6 "Farnell" V 4200 2300 30  0001 C CNN "Provider"
+	1    3950 2300
+	1    0    0    -1
+$EndComp
+$Comp
+L CP_SMT C?
+U 1 1 5635343E
+P 6900 2050
+F 0 "C?" H 6925 2150 50  0000 L CNN
+F 1 "220uF/10%/6V3" V 6750 1650 50  0000 L CNN
+F 2 "Capacitors_Tantalum_SMD:TantalC_SizeC_EIA-6032_Reflow" H 6938 1900 30  0001 C CNN
+F 3 "" H 6900 2050 60  0000 C CNN
+F 4 "2312" H 6900 2050 25  0000 C CNN "SMT"
+F 5 "1462420" H 6900 1850 30  0001 C CNN "Part"
+F 6 "Farnell" H 6900 1800 30  0001 C CNN "Provider"
+	1    6900 2050
+	1    0    0    -1
+$EndComp
+$Comp
+L C_SMT C?
+U 1 1 563526B5
+P 7600 2050
+F 0 "C?" H 7625 2150 50  0000 L CNN
+F 1 "100nF/50V/X7R" V 7450 1650 50  0000 L CNN
+F 2 "Capacitors_SMD:C_0603" H 7630 1900 30  0001 L CNN
+F 3 "" H 7625 2150 60  0000 L CNN
+F 4 "0603" H 7600 2050 20  0000 C CNN "SMT"
+F 5 "1414028" H 7630 1860 30  0001 L CNN "Part"
+F 6 "Farnell" H 7630 1820 30  0001 L CNN "Provider"
+	1    7600 2050
+	1    0    0    -1
+$EndComp
+$Comp
+L FB_SMT FB?
+U 1 1 56353A77
+P 6000 1800
+F 0 "FB?" H 6000 1900 50  0000 C CNN
+F 1 "BEAD/0.045OHM/2A" H 6000 1750 50  0000 C CNN
+F 2 "Resistors_SMD:R_0603" H 6000 1700 30  0001 C CNN
+F 3 "" H 6050 1800 60  0000 C CNN
+F 4 "0603" H 6000 1800 25  0000 C CNN "SMT"
+F 5 "1515714" H 6000 1650 30  0001 C CNN "Part"
+F 6 "Farnell" H 6000 1600 30  0001 C CNN "Provider"
+	1    6000 1800
+	1    0    0    -1
+$EndComp
+$Comp
+L FB_SMT FB?
+U 1 1 56354381
+P 8300 4750
+F 0 "FB?" H 8300 4850 50  0000 C CNN
+F 1 "BEAD/0.045OHM/2A" H 8300 4700 50  0000 C CNN
+F 2 "Resistors_SMD:R_0603" H 8300 4650 30  0001 C CNN
+F 3 "" H 8350 4750 60  0000 C CNN
+F 4 "0603" H 8300 4750 25  0000 C CNN "SMT"
+F 5 "1515714" H 8300 4600 30  0001 C CNN "Part"
+F 6 "Farnell" H 8300 4550 30  0001 C CNN "Provider"
+	1    8300 4750
+	0    1    1    0
+$EndComp
 $EndSCHEMATC

Commit message: Work on PWM, USB, MEMS, Power
Parts:
- removed R?: 47K/5%, Resistors_SMD:R_0603, symbol R_SMT
- removed U?: TPS2061CDBVT, symbol TPS2061CDBVT
- added DL?: GREEN, LEDs:LED-0603, symbol LED_SMT
- added R?: 10K/5%, Resistors_SMD:R_0603, symbol R_SMT
- added R?: 1k2/5%, Resistors_SMD:R_0603, symbol R_SMT
- added U?: TPS2065CDBVT, symbol TPS2065CDBVT
Connections:
- net +3V3: now also R?.1
- net +5V: now also R?.1, U?.5 (IN)
- net GND: now also DL?.1 (K), U?.2 (GND); no longer R?.2
- net USB_H1_OC: now also R?.2, U?.3 (~FLT)
- net at C?.1, C?.1, CN?.1 (VCC)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: now also R?.2
- net at FB?.1: now also U?.1 (OUT)
- net USB_HOST_DN renamed USB_HOST_DM
- new net: R?.2, U?.4 (EN)
- new net: DL?.2 (A), R?.1
Other:
- moved on the sheet: C?, DL?, FB?, R?
