File: hardware/colibri-v2/wb_connector.sch (KiCad schematic (older format))
At the start: 6 parts

Commit message: Added M25P32
Parts:
- added C?: 2u2/10V/X5R, Capacitors_SMD:C_0603, symbol C_SMT
- added C?: 100nF/50V/X7R, Capacitors_SMD:C_0603, symbol C_SMT
- added R? (x4): 22R/5%, Resistors_SMD:R_0603, symbol R_SMT
- added U?: M25P32-VME6G, symbol M25P32-VME6G
Connections:
- net +3V3: now also C?.1, C?.2, U?.3 (~W), U?.7 (~HOLD), U?.8 (VCC)
- net GND: now also CN?.1, CN?.100, CN?.101, CN?.12, CN?.121, CN?.124, CN?.13, CN?.148, CN?.153, CN?.154, CN?.166, CN?.177, CN?.18, CN?.184, CN?.185, CN?.19, CN?.198, CN?.201, CN?.204, CN?.217, CN?.220, CN?.229, CN?.232, CN?.239, CN?.24, CN?.249, CN?.25, CN?.250, CN?.265, CN?.266, CN?.30, CN?.3E1, CN?.3E4, CN?.3E8, CN?.41, CN?.42, CN?.47, CN?.48, CN?.4E1, CN?.4E10, CN?.4E4, CN?.4E7, CN?.53, CN?.54, CN?.59, CN?.6, CN?.60, CN?.65, CN?.66, CN?.7, CN?.77, CN?.83, CN?.88, CN?.89, CN?.94, CN?.95, CN?.P1, CN?.P2, C?.1, C?.2, U?.4 (VSS), U?.9 (EP)
- net R_NANDF_RB0: now reaches CN?.102
- net PCIEB_TXP: now reaches CN?.103
- net R_NANDF_WP: now reaches CN?.104
- net PCIEB_TXN: now reaches CN?.105
- net R_NANDF_CLE: now reaches CN?.106
- net EXCDA_nPREST: now reaches CN?.107
- net R_NANDF_ALE: now reaches CN?.108
- net PCIEB_RXP: now reaches CN?.109
- net LVDS0_TX2_P: now reaches CN?.11
- net R_NANDF_WE: now reaches CN?.110
- net PCIEB_RXN: now reaches CN?.111
- net R_NANDF_RE: now reaches CN?.112
- net PCIE_CLK_OEA: now reaches CN?.113
- net RSVD1: now reaches CN?.114
- net PCIE_CLK_OEB: now reaches CN?.115
- net R_NANDF_A10: now reaches CN?.116
- net PCIE_nWAKE: now reaches CN?.117
- net R_NANDF_A9: now reaches CN?.118
- net PCIE_nRST: now reaches CN?.119
- net R_NANDF_A8: now reaches CN?.120
- net R_NANDF_A7: now reaches CN?.122
- net SATA1_RXP: now reaches CN?.123
- net SATA1_RXN: now reaches CN?.125
- net LVDS0_TX3_N: now reaches CN?.15
- net LVDS0_TX3_P: now reaches CN?.17
- net +5V: now reaches CN?.1E10
- net +5V: now also CN?.1E2, CN?.1E3, CN?.1E4, CN?.1E5, CN?.1E6, CN?.1E7, CN?.1E8, CN?.1E9, CN?.2E10, CN?.2E2, CN?.2E3, CN?.2E4, CN?.2E5, CN?.2E6, CN?.2E7, CN?.2E8, CN?.2E9
- net LVDS0_CLK_N: now reaches CN?.21
- net LVDS0_CLK_P: now reaches CN?.23
- net LVDS0_BLT_CTRL: now reaches CN?.27
- net LVDS0_EN: now reaches CN?.29
- net LVDS0_TX1_N: now reaches CN?.3
- net LVDS0_VDDEN: now reaches CN?.31
- net eDP0_SELF_TEST: now reaches CN?.33
- net eDP0_HPD: now reaches CN?.35
- net I2C1_SDA: now reaches CN?.37
- net I2C1_SCL: now reaches CN?.39
- net LVDS0_TX0_P: now reaches CN?.3E10
- net ETHER1_D2P: now reaches CN?.3E2
- net ETHER1_D2N: now reaches CN?.3E3
- net ETHER1_D3P: now reaches CN?.3E5
- net ETHER1_D3N: now reaches CN?.3E6
- net LED1_ACT: now reaches CN?.3E7
- net LVDS0_TX0_N: now reaches CN?.3E9
- net HDMI_CLKP: now reaches CN?.43
- net HDMI_CLKM: now reaches CN?.45
- net HDMI_D0P: now reaches CN?.49
- net ETHER1_D0P: now reaches CN?.4E2
- net ETHER1_D0N: now reaches CN?.4E3
- net ETHER1_D1P: now reaches CN?.4E5
- net ETHER1_D1N: now reaches CN?.4E6
- net LED1_nLINK100: now reaches CN?.4E8
- net LED1_nLINK1000: now reaches CN?.4E9
- net LVDS0_TX1_P: now reaches CN?.5
- net HDMI_D0M: now reaches CN?.51
- net HDMI_D1P: now reaches CN?.55
- net HDMI_D1M: now reaches CN?.57
- net HDMI_D2P: now reaches CN?.61
- net HDMI_D2M: now reaches CN?.63
- net HDMI1_HPD: now reaches CN?.67
- net HDMI1_CAD: now reaches CN?.69
- net HDMI1_CEC: now reaches CN?.71
- net DDC_SCL: now reaches CN?.73
- net DDC_SDA: now reaches CN?.75
- net PCIEB_CLKP: now reaches CN?.79
- net PCIEB_CLKN: now reaches CN?.81
- net RSVD0: now reaches CN?.84
- net PCIEA_CLKP: now reaches CN?.85
- net R_NANDF_CS0: now reaches CN?.86
- net PCIEA_CLKN: now reaches CN?.87
- net LVDS0_TX2_N: now reaches CN?.9
- net R_NANDF_CS1: now reaches CN?.90
- net PCIEA_TXP: now reaches CN?.91
- net R_NANDF_CS2: now reaches CN?.92
- net PCIEA_TXN: now reaches CN?.93
- net R_NANDF_CS3: now reaches CN?.96
- net PCIEA_RXP: now reaches CN?.97
- net R_NANDF_CS4: now reaches CN?.98
- net PCIEA_RXN: now reaches CN?.99
- net EIM_WAIT: now reaches CN?.133
- net R_NANDF_A6: now reaches CN?.134
- net SATA1_TXP: now reaches CN?.135
- net R_NANDF_A5: now reaches CN?.136
- net SATA1_TXN: now reaches CN?.137
- net R_NANDF_A4: now reaches CN?.138
- net USB_HUB_RESET_B: now reaches CN?.139
- net R_NANDF_A3: now reaches CN?.140
- net USB_OTG_OC: now reaches CN?.141
- net R_NANDF_A2: now reaches CN?.142
- net StdB1_SSRXP: now reaches CN?.143
- net R_NANDF_A1: now reaches CN?.144
- net StdB1_SSRXN: now reaches CN?.145
- net R_NANDF_D15: now reaches CN?.146
- net GND_DRAIN1: now reaches CN?.147
- net StdB1_SSTXP: now reaches CN?.149
- net R_NANDF_D14: now reaches CN?.150
- net StdB1_SSTXN: now reaches CN?.151
- net R_NANDF_D13: now reaches CN?.152
- net USB_OTG_ID: now reaches CN?.155
- net R_NANDF_D12: now reaches CN?.156
- net USB_OTG_DP: now reaches CN?.157
- net R_NANDF_D11: now reaches CN?.158
- net USB_OTG_DN: now reaches CN?.159
- net R_NANDF_D10: now reaches CN?.160
- net USB_OTG_VBUS: now reaches CN?.161
- net R_NANDF_D9: now reaches CN?.162
- net USB_OTG_PWR_EN: now reaches CN?.163
- net R_NANDF_D8: now reaches CN?.164
- net USB_H1_OC: now reaches CN?.165
- net StdB2_SSRXP: now reaches CN?.167
- net R_NANDF_D7: now reaches CN?.168
- net StdB2_SSRXN: now reaches CN?.169
- net R_NANDF_D6: now reaches CN?.170
- net GND_DRAIN2: now reaches CN?.171
- net R_NANDF_D5: now reaches CN?.172
- net StdB2_SSTXP: now reaches CN?.173
- net R_NANDF_D4: now reaches CN?.174
- net StdB2_SSTXN: now reaches CN?.175
- net R_NANDF_D3: now reaches CN?.176
- net R_NANDF_D2: now reaches CN?.178
- net USB_HOST_DN: now reaches CN?.179
- net R_NANDF_D1: now reaches CN?.180
- net USB_HOST_DP: now reaches CN?.181
- net R_NANDF_D0: now reaches CN?.182
- net USB_H1_VBUS: now reaches CN?.183
- net AUD5_RXD: now reaches CN?.186
- net AUD3_RXD: now reaches CN?.187
- net AUD5_TXFS: now reaches CN?.188
- net AUD3_TXFS: now reaches CN?.189
- net AUD5_TXD: now reaches CN?.190
- net AUD3_TXC: now reaches CN?.191
- net AUD5_TXC: now reaches CN?.192
- net AUD3_: now reaches CN?.193
- net GPIO_1_CLK0: now reaches CN?.194
- net AUDIO_CLK: now reaches CN?.195
- net SPDIF_OUT: now reaches CN?.196
- net CAN2p: now reaches CN?.197
- net CAN2n: now reaches CN?.199
- net CAN1p: now reaches CN?.200
- net CAN1n: now reaches CN?.202
- net SD1_CD: now reaches CN?.203
- net SD1_CMD: now reaches CN?.205
- net SD1_CLK: now reaches CN?.206
- net SD1_WP: now reaches CN?.207
- net SD1_LED: now reaches CN?.208
- net SD1_DATA1: now reaches CN?.209
- net SD1_PWREN: now reaches CN?.210
- net SD1_DATA3: now reaches CN?.211
- net SD1_DATA0: now reaches CN?.212
- net SD1_DATA5: now reaches CN?.213
- net SD1_DATA2: now reaches CN?.214
- net SD1_DATA7: now reaches CN?.215
- net SD1_DATA4: now reaches CN?.216
- net SD1_DATA6: now reaches CN?.218
- net CSPI2_MOSI: now reaches CN?.219
- net CSPI2_MISO: now reaches CN?.221
- net WB_SPI_MOSI: now reaches CN?.222
- net WB_SPI_MOSI: now also R?.1
- net CSPI2_SCLK: now reaches CN?.223
- net WB_SPI_MISO: now reaches CN?.224
- net WB_SPI_MISO: now also R?.1
- net CSPI2_CS0: now reaches CN?.225
- net WB_SPI_CLK: now reaches CN?.226
- net WB_SPI_CLK: now also R?.1
- net CSPI2_CS1: now reaches CN?.227
- net WB_SPI_CS: now reaches CN?.228
- net CSPI1_CS1: now reaches CN?.230
- net CSPI1_CS1: now also R?.1
- net I2C2_SCL: now reaches CN?.231
- net I2C2_SDA: now reaches CN?.233
- net I2C3_SCL: now reaches CN?.235
- net I2C3_SDA: now reaches CN?.237
- net UART1_CTS: now reaches CN?.241
- net UART2_DCD: now reaches CN?.242
- net UART1_TXD: now reaches CN?.243
- net UART2_DSR: now reaches CN?.244
- net UART1_RXD: now reaches CN?.245
- net UART2_DTR: now reaches CN?.246
- net UART1_RTS: now reaches CN?.247
- net UART2_RI: now reaches CN?.248
- net S3: now reaches CN?.251
- net S5: now reaches CN?.253
- net AUX_5V_EN: now reaches CN?.257
- net MNF7: now reaches CN?.267
- net MNF8: now reaches CN?.269
- net MNF0: now reaches CN?.270
- net MNF9: now reaches CN?.271
- net MNF1: now reaches CN?.272
- net MNF10: now reaches CN?.273
- net MNF2: now reaches CN?.274
- net MNF11: now reaches CN?.275
- net MNF3: now reaches CN?.276
- net MNF12: now reaches CN?.277
- net MNF4: now reaches CN?.278
- net MNF13_WATCHDOG: now reaches CN?.279
- net MNF5: now reaches CN?.280
- net VCC_RTC: now reaches CN?.281
- net EIM_BCLK renamed WB_GPIO3
- net EIM_D27 renamed WB_GPIO2
- net EIM_DA11 renamed WB_GPIO1
- net ENET_RX_ER renamed WB_GPIO4
- net GPIO7_IO08 renamed WB_GPIO5
- new net: R?.2, U?.1 (~s)
- new net: R?.2, U?.2 (DQ1)
- new net: R?.2, U?.5 (DQ0)
- new net: R?.2, U?.6 (C)
- no-connect marks 0 -> 3
Other:
- moved on the sheet: CN?A, CN?B, Q?, R?

Commit message: Added ext_sensors.sch sheet
Parts:
- added R? (x8): 2k2/5%, Resistors_SMD:R_0603, symbol R_SMT
- added R?: 0R/5%, Resistors_SMD:R_0603, symbol R_SMT
Connections:
- net DISP0_CLK is gone; now on net DISP0_BKLEN: CN?.70
- net +3V3: now also R?.1, R?.1, R?.1, R?.1, R?.1, R?.1
- net +5V: now also R?.1, R?.1
- net DDC_SCL: now also R?.2
- net DDC_SDA: now also R?.2
- net I2C1_SCL: now also R?.2
- net I2C1_SDA: now also R?.2
- net I2C2_SCL: now also R?.2
- net I2C2_SDA: now also R?.2
- net I2C3_SCL: now also R?.2
- net I2C3_SDA: now also R?.2
- net R_NANDF_CS2: now also R?.1
- net Wandboard LCD/TP_PENIRQ: now also R?.2
- net R_NANDF_CS3 renamed RTC_INT
