File: hardware/colibri-v2/wnd_ethernet.sch (KiCad schematic (older format))
At the start: 6 parts

Commit message: Added footprints
Parts:
- LAN1: footprint (none) -> Sigmadrone:WURTH_7499111446
Changed lines of the file:
@@
 	3100 4150 5650 4150
 $Comp
-L GND #PWR0118
+L GND #PWR0119
 U 1 1 561772BC
 P 3100 4150
-F 0 "#PWR0118" H 3100 3900 50  0001 C CNN
+F 0 "#PWR0119" H 3100 3900 50  0001 C CNN
 F 1 "GND" H 3100 4000 50  0000 C CNN
 F 2 "" H 3100 4150 60  0000 C CNN
@@
 $EndComp
 $Comp
-L GND #PWR0119
+L GND #PWR0120
 U 1 1 56CB1E1A
 P 6350 5350
-F 0 "#PWR0119" H 6350 5100 50  0001 C CNN
+F 0 "#PWR0120" H 6350 5100 50  0001 C CNN
 F 1 "GND" H 6350 5200 50  0000 C CNN
 F 2 "" H 6350 5350 60  0000 C CNN
@@
 F 0 "LAN1" H 6877 3747 60  0000 L CNN
 F 1 "7499111446" H 6877 3641 60  0000 L CNN
-F 2 "" H 6350 4250 60  0001 C CNN
+F 2 "Sigmadrone:WURTH_7499111446" H 6350 4250 60  0001 C CNN
 F 3 "" H 6350 4250 60  0000 C CNN
 	1    6350 3800
@@
 	6450 5250 6450 5050
 $Comp
-L PWR_FLAG #FLG0120
+L PWR_FLAG #FLG0121
 U 1 1 56CDF282
 P 5300 2550
-F 0 "#FLG0120" H 5300 2645 50  0001 C CNN
+F 0 "#FLG0121" H 5300 2645 50  0001 C CNN
 F 1 "PWR_FLAG" H 5300 2774 50  0000 C CNN
 F 2 "" H 5300 2550 50  0000 C CNN
