File: hardware/colibri-v2/ext_sensors.sch (KiCad schematic (older format))
At the start: 21 parts, among them CN9 Wurth-68711814522, P32 CONN_02X10

Commit message: Adding and assigning footprints
Parts:
- P32: footprint (none) -> Pin_Headers:Pin_Header_Straight_2x10
Changed lines of the file:
@@
 F 0 "P32" H 5450 3566 50  0000 C CNN
 F 1 "CONN_02X10" H 5450 3474 50  0000 C CNN
-F 2 "" H 5450 1700 50  0001 C CNN
+F 2 "Pin_Headers:Pin_Header_Straight_2x10" H 5450 1700 50  0001 C CNN
 F 3 "" H 5450 1700 50  0000 C CNN
 	1    5450 2900

Commit message: Added new footprints
Parts:
- CN9: footprint (none) -> Sigmadrone:68711814522
Changed lines of the file:
@@
 $Descr A4 11693 8268
 encoding utf-8
-Sheet 28 28
+Sheet 27 28
 Title ""
 Date ""
@@
 F 0 "CN9" V 5090 7328 60  0000 L CNN
 F 1 "Wurth-68711814522" V 5196 7328 60  0000 L CNN
-F 2 "" H 5250 4900 60  0001 C CNN
+F 2 "Sigmadrone:68711814522" H 5250 4900 60  0001 C CNN
 F 3 "" H 5250 4900 60  0000 C CNN
 	1    5250 6150
