File: hardware/colibri-v2/c_ftdi_interface.sch (KiCad schematic (older format))
At the start: 13 parts, among them P4 USB_B, U4 FT232RL

Commit message: Added and assigned footprints.
Parts:
- removed D1: RED, symbol LED
- added DL17: RED, LEDs:LED-0603, symbol LED_SMT
Changed lines of the file:
@@
-$EndComp
-$Comp
-L LED D1
-U 1 1 563260D3
-P 9250 4250
-F 0 "D1" H 9250 4350 50  0000 C CNN
-F 1 "RED" H 9250 4150 50  0000 C CNN
-F 2 "" H 9250 4250 60  0001 C CNN
-F 3 "" H 9250 4250 60  0000 C CNN
-	1    9250 4250
-	1    0    0    -1
 $EndComp
 $Comp
@@
 	4350 2000 4350 3000
 Connection ~ 4350 3000
+$Comp
+L LED_SMT DL17
+U 1 1 56CFEF69
+P 9250 4250
+F 0 "DL17" H 9250 4350 50  0000 C CNN
+F 1 "RED" H 9250 4150 50  0000 C CNN
+F 2 "LEDs:LED-0603" H 9250 4100 30  0001 C CNN
+F 3 "" H 9250 4250 60  0000 C CNN
+F 4 "0603" H 9135 4230 30  0000 C CNN "SMT"
+F 5 "2322071" H 9250 4050 30  0001 C CNN "Part"
+F 6 "Farnell" H 9250 4000 30  0001 C CNN "Provider"
+	1    9250 4250
+	1    0    0    -1
+$EndComp
 $EndSCHEMATC

Commit message: Added footprints
Parts:
- removed P4: USB_B, symbol USB_B
- added CN10: 629_105_150_921, Sigmadrone:WURTH_629105150921, symbol 629_105_150_921
Connections:
- wire segments 46 -> 52
- no-connect marks 10 -> 11
Changed lines of the file:
@@
 	1    0    0    -1
 $EndComp
-$Comp
-L USB_B P4
-U 1 1 558F3BFF
-P 2000 3200
-F 0 "P4" H 2200 3000 50  0000 C CNN
-F 1 "USB_B" H 1950 3400 50  0000 C CNN
-F 2 "" V 1950 3100 60  0001 C CNN
-F 3 "" V 1950 3100 60  0000 C CNN
-	1    2000 3200
-	0    -1   1    0
-$EndComp
-Wire Wire Line
-	2300 3000 3550 3000
+Wire Wire Line
+	1950 3000 3550 3000
 Wire Wire Line
 	3950 3000 6550 3000
 Wire Wire Line
-	2300 3100 6550 3100
-Wire Wire Line
-	2300 3200 6550 3200
+	1950 3100 6550 3100
+Wire Wire Line
+	1950 3200 6550 3200
 $Comp
 L GND #PWR033
@@
 $Comp
 L GND #PWR040
-U 1 1 558F7AED
-P 2650 5000
-F 0 "#PWR040" H 2650 4750 50  0001 C CNN
-F 1 "GND" H 2650 4850 50  0000 C CNN
-F 2 "" H 2650 5000 60  0000 C CNN
-F 3 "" H 2650 5000 60  0000 C CNN
-	1    2650 5000
-	1    0    0    -1
-$EndComp
-Wire Wire Line
-	2300 3300 2650 3300
-Wire Wire Line
-	2650 3300 2650 5000
-$Comp
-L GND #PWR041
 U 1 1 558F7BAB
-P 1900 5000
-F 0 "#PWR041" H 1900 4750 50  0001 C CNN
-F 1 "GND" H 1900 4850 50  0000 C CNN
-F 2 "" H 1900 5000 60  0000 C CNN
-F 3 "" H 1900 5000 60  0000 C CNN
-	1    1900 5000
-	1    0    0    -1
-$EndComp
-Wire Wire Line
-	1900 3500 1900 5000
+P 2150 5000
+F 0 "#PWR040" H 2150 4750 50  0001 C CNN
+F 1 "GND" H 2150 4850 50  0000 C CNN
+F 2 "" H 2150 5000 60  0000 C CNN
+F 3 "" H 2150 5000 60  0000 C CNN
+	1    2150 5000
+	1    0    0    -1
+$EndComp
+Wire Wire Line
+	2150 3400 2150 5000
 NoConn ~ 6550 3400
 NoConn ~ 6550 4000
@@
 	7950 3200 9500 3200
 $Comp
-L +3V3 #PWR042
+L +3V3 #PWR041
 U 1 1 558F916C
 P 9650 3900
-F 0 "#PWR042" H 9650 3750 50  0001 C CNN
+F 0 "#PWR041" H 9650 3750 50  0001 C CNN
 F 1 "+3V3" H 9650 4040 50  0000 C CNN
 F 2 "" H 9650 3900 60  0000 C CNN
@@
 	9450 3900 9650 3900
 $Comp
-L +3V3 #PWR043
+L +3V3 #PWR042
 U 1 1 558F926F
 P 9650 4250
-F 0 "#PWR043" H 9650 4100 50  0001 C CNN
+F 0 "#PWR042" H 9650 4100 50  0001 C CNN
 F 1 "+3V3" H 9650 4390 50  0000 C CNN
 F 2 "" H 9650 4250 60  0000 C CNN
@@
 NoConn ~ 7950 3200
 $Comp
-L PWR_FLAG #FLG044
+L PWR_FLAG #FLG043
 U 1 1 56CC9B04
 P 4350 2000
-F 0 "#FLG044" H 4350 2095 50  0001 C CNN
+F 0 "#FLG043" H 4350 2095 50  0001 C CNN
 F 1 "PWR_FLAG" H 4350 2224 50  0000 C CNN
 F 2 "" H 4350 2000 50  0000 C CNN
@@
 	1    0    0    -1
 $EndComp
+$Comp
+L 629_105_150_921 CN10
+U 1 1 56D2CFA0
+P 1550 3500
+F 0 "CN10" H 1700 4150 60  0000 C CNN
+F 1 "629_105_150_921" V 1800 3350 60  0000 C CNN
+F 2 "Sigmadrone:WURTH_629105150921" H 3100 4800 60  0001 C CNN
+F 3 "" H 3100 4800 60  0000 C CNN
+	1    1550 3500
+	-1   0    0    -1
+$EndComp
+NoConn ~ 1950 3300
+Wire Wire Line
+	1950 3500 2150 3500
+Wire Wire Line
+	1950 3600 2150 3600
+Wire Wire Line
+	1950 3700 2150 3700
+Wire Wire Line
+	1950 3800 2150 3800
+Wire Wire Line
+	1950 3900 2150 3900
+Wire Wire Line
+	1950 4000 2150 4000
+Connection ~ 2150 3600
+Connection ~ 2150 3700
+Connection ~ 2150 3800
+Connection ~ 2150 3900
+Connection ~ 2150 4000
+Connection ~ 2150 3500
+Wire Wire Line
+	1950 3400 2150 3400
+$Comp
+L PWR_FLAG #FLG044
+U 1 1 56D35204
+P 2150 2000
+F 0 "#FLG044" H 2150 2095 50  0001 C CNN
+F 1 "PWR_FLAG" H 2150 2224 50  0000 C CNN
+F 2 "" H 2150 2000 50  0000 C CNN
+F 3 "" H 2150 2000 50  0000 C CNN
+	1    2150 2000
+	1    0    0    -1
+$EndComp
+Wire Wire Line
+	2150 2000 2150 3000
+Connection ~ 2150 3000
 $EndSCHEMATC

Commit message: Added footprints
Parts:
- U4: footprint (none) -> Housings_SSOP:SSOP-28_5.3x10.2mm_Pitch0.65mm
Changed lines of the file:
@@
 F 0 "U4" H 7600 4850 60  0000 C CNN
 F 1 "FT232RL" H 7000 2750 60  0000 C CNN
-F 2 "" H 7250 3800 60  0001 C CNN
+F 2 "Housings_SSOP:SSOP-28_5.3x10.2mm_Pitch0.65mm" H 7250 3800 60  0001 C CNN
 F 3 "" H 7250 3800 60  0000 C CNN
 	1    7250 3800

Commit message: Added AP6681GMT-HF-3.kicad_mod. Fixed netlist errors
Parts:
- DL17, DL5: footprint LEDs:LED-0603 -> LEDs:LED_0603
Changed lines of the file:
@@
 F 0 "DL5" H 9250 4000 50  0000 C CNN
 F 1 "GREEN" H 9250 3800 50  0000 C CNN
-F 2 "LEDs:LED-0603" H 9250 3750 30  0001 C CNN
+F 2 "LEDs:LED_0603" H 9250 3750 30  0001 C CNN
 F 3 "" H 9250 3900 60  0000 C CNN
 F 4 "0603" H 9135 3880 30  0000 C CNN "SMT"
@@
 F 0 "DL17" H 9250 4350 50  0000 C CNN
 F 1 "RED" H 9250 4150 50  0000 C CNN
-F 2 "LEDs:LED-0603" H 9250 4100 30  0001 C CNN
+F 2 "LEDs:LED_0603" H 9250 4100 30  0001 C CNN
 F 3 "" H 9250 4250 60  0000 C CNN
 F 4 "0603" H 9135 4230 30  0000 C CNN "SMT"

Commit message: Working on placement.
Parts:
- removed U4: FT232RL, Housings_SSOP:SSOP-28_5.3x10.2mm_Pitch0.65mm, symbol FT232RL
- added U4: FT232RQ, Housings_DFN_QFN:QFN-32-1EP_5x5mm_Pitch0.5mm, symbol FT232RQ
Connections:
- net +3V3: now also U4.1 (VCCIO)
- net C_FTDI_CTS: now also U4.8 (~CTS)
- net C_FTDI_RI: now also U4.3 (~RI)
- net C_FTDI_RTS: now also U4.32 (~RTS)
- net C_FTDI_RXD: now also U4.2 (RXD)
- net C_FTDI_TXD: now also U4.30 (TXD)
- net GND: now also U4.17 (GND), U4.20 (GND), U4.24 (AGND), U4.26 (TEST), U4.33 (Epad_GND), U4.4 (GND)
- net at CN10.3 (DP): now also U4.14 (USBDP)
- net at CN10.2 (DM): now also U4.15 (USBDM)
- net at C24.1: now also U4.16 (3V3OUT)
- net at R31.2: now also U4.31 (~DTR)
- net at C21.2, FB1.2: now also U4.19 (VCC)
- net at R33.2: now also U4.21 (CBUS1)
- net at R32.2: now also U4.22 (CBUS0)
- net at R31.1: now also U4.6 (~DSR)
- no-connect marks 11 -> 8
Changed lines of the file:
@@
 Comment4 ""
 $EndDescr
-$Comp
-L FT232RL U4
-U 1 1 558F3BD7
-P 7250 3800
-F 0 "U4" H 7600 4850 60  0000 C CNN
-F 1 "FT232RL" H 7000 2750 60  0000 C CNN
-F 2 "Housings_SSOP:SSOP-28_5.3x10.2mm_Pitch0.65mm" H 7250 3800 60  0001 C CNN
-F 3 "" H 7250 3800 60  0000 C CNN
-	1    7250 3800
-	1    0    0    -1
-$EndComp
 Wire Wire Line
 	1950 3000 3550 3000
@@
 Wire Wire Line
 	2150 3400 2150 5000
-NoConn ~ 6550 3400
-NoConn ~ 6550 4000
-NoConn ~ 6550 4100
-NoConn ~ 7950 4100
-NoConn ~ 7950 4000
-NoConn ~ 7950 3900
 Wire Wire Line
 	6350 2900 6350 2000
@@
 Text HLabel 9500 3600 2    60   Output ~ 0
 C_FTDI_RI
-NoConn ~ 7950 3500
 Wire Wire Line
 	8650 3300 8950 3300
@@
 	1    0    0    -1
 $EndComp
-NoConn ~ 7950 3600
 Wire Wire Line
 	7950 3600 9500 3600
-NoConn ~ 7950 3100
-NoConn ~ 7950 3200
 $Comp
 L PWR_FLAG #FLG044
@@
 	2150 2000 2150 3000
 Connection ~ 2150 3000
+$Comp
+L FT232RQ U4
+U 1 1 56DAB925
+P 7250 3800
+F 0 "U4" H 7600 4850 60  0000 C CNN
+F 1 "FT232RQ" H 7000 2750 60  0000 C CNN
+F 2 "Housings_DFN_QFN:QFN-32-1EP_5x5mm_Pitch0.5mm" H 7250 2675 60  0001 C CNN
+F 3 "" H 7250 3800 60  0000 C CNN
+F 4 "1146033" H 7250 2525 60  0001 C CNN "Part"
+F 5 "Farnell" H 7250 2600 60  0001 C CNN "Provider"
+	1    7250 3800
+	1    0    0    -1
+$EndComp
+NoConn ~ 6550 3800
+NoConn ~ 6550 4000
+NoConn ~ 6550 4100
+NoConn ~ 7950 3500
+NoConn ~ 7950 3900
+NoConn ~ 7950 4000
+NoConn ~ 7950 4100
+$Comp
+L GND #PWR046
+U 1 1 56DAC442
+P 8100 5000
+F 0 "#PWR046" H 8100 4750 50  0001 C CNN
+F 1 "GND" H 8100 4850 50  0000 C CNN
+F 2 "" H 8100 5000 60  0000 C CNN
+F 3 "" H 8100 5000 60  0000 C CNN
+	1    8100 5000
+	1    0    0    -1
+$EndComp
+Wire Wire Line
+	7950 4700 8100 4700
+Wire Wire Line
+	8100 4700 8100 5000
 $EndSCHEMATC
