File: hardware/colibri-v2/sensors_pwr_ctrl.sch (KiCad schematic (older format))
At the start: 3 parts, among them Q12 IRLML6402TRPBF

Commit message: Adding and assigning footprints
Parts:
- Q12: footprint (none) -> Sigmadrone:SOT23_IRLML6402
Changed lines of the file:
@@
 F 0 "Q12" H 6700 4000 50  0000 R CNN
 F 1 "IRLML6402TRPBF" H 7250 3900 50  0000 R CNN
-F 2 "" H 6600 4050 29  0001 C CNN
+F 2 "Sigmadrone:SOT23_IRLML6402" H 6600 4050 29  0001 C CNN
 F 3 "" H 6400 3950 60  0000 C CNN
 	1    6400 3950
