File: hardware/colibri-v2/pca9685pw_led_ctrl.sch (KiCad schematic (older format))
At the start: 17 parts, among them P24 CONN_01X03, P25 CONN_01X03, P26 CONN_01X03, P27 CONN_01X03, P28 CONN_01X03, P29 CONN_01X03, P30 CONN_01X03, P31 CONN_01X03, U24 PCA9685PW

Commit message: Adding and assigning footprints
Parts:
- P24, P25, P26, P27, P28, P29, P30, P31: footprint (none) -> Pin_Headers:Pin_Header_Straight_1x03
Changed lines of the file:
@@
 F 0 "P28" H 6700 4750 50  0000 C CNN
 F 1 "CONN_01X03" V 6800 4550 50  0000 C CNN
-F 2 "" H 6700 4550 60  0001 C CNN
+F 2 "Pin_Headers:Pin_Header_Straight_1x03" H 6700 4550 60  0001 C CNN
 F 3 "" H 6700 4550 60  0000 C CNN
 	1    6700 4550
@@
 F 0 "P29" H 6700 5650 50  0000 C CNN
 F 1 "CONN_01X03" V 6800 5450 50  0000 C CNN
-F 2 "" H 6700 5450 60  0001 C CNN
+F 2 "Pin_Headers:Pin_Header_Straight_1x03" H 6700 5450 60  0001 C CNN
 F 3 "" H 6700 5450 60  0000 C CNN
 	1    6700 5450
@@
 F 0 "P30" H 6700 6550 50  0000 C CNN
 F 1 "CONN_01X03" V 6800 6350 50  0000 C CNN
-F 2 "" H 6700 6350 60  0001 C CNN
+F 2 "Pin_Headers:Pin_Header_Straight_1x03" H 6700 6350 60  0001 C CNN
 F 3 "" H 6700 6350 60  0000 C CNN
 	1    6700 6350
@@
 F 0 "P31" H 6700 7450 50  0000 C CNN
 F 1 "CONN_01X03" V 6800 7250 50  0000 C CNN
-F 2 "" H 6700 7250 60  0001 C CNN
+F 2 "Pin_Headers:Pin_Header_Straight_1x03" H 6700 7250 60  0001 C CNN
 F 3 "" H 6700 7250 60  0000 C CNN
 	1    6700 7250
@@
 F 0 "P24" H 6700 1200 50  0000 C CNN
 F 1 "CONN_01X03" V 6800 1000 50  0000 C CNN
-F 2 "" H 6700 1000 60  0001 C CNN
+F 2 "Pin_Headers:Pin_Header_Straight_1x03" H 6700 1000 60  0001 C CNN
 F 3 "" H 6700 1000 60  0000 C CNN
 	1    6700 1000
@@
 F 0 "P25" H 6700 2100 50  0000 C CNN
 F 1 "CONN_01X03" V 6800 1900 50  0000 C CNN
-F 2 "" H 6700 1900 60  0001 C CNN
+F 2 "Pin_Headers:Pin_Header_Straight_1x03" H 6700 1900 60  0001 C CNN
 F 3 "" H 6700 1900 60  0000 C CNN
 	1    6700 1900
@@
 F 0 "P26" H 6700 3000 50  0000 C CNN
 F 1 "CONN_01X03" V 6800 2800 50  0000 C CNN
-F 2 "" H 6700 2800 60  0001 C CNN
+F 2 "Pin_Headers:Pin_Header_Straight_1x03" H 6700 2800 60  0001 C CNN
 F 3 "" H 6700 2800 60  0000 C CNN
 	1    6700 2800
@@
 F 0 "P27" H 6700 3900 50  0000 C CNN
 F 1 "CONN_01X03" V 6800 3700 50  0000 C CNN
-F 2 "" H 6700 3700 60  0001 C CNN
+F 2 "Pin_Headers:Pin_Header_Straight_1x03" H 6700 3700 60  0001 C CNN
 F 3 "" H 6700 3700 60  0000 C CNN
 	1    6700 3700

Commit message: Added new footprints
Parts:
- U24: footprint (none) -> Housings_SSOP:TSSOP-28_4.4x9.7mm_Pitch0.65mm
Changed lines of the file:
@@
 F 0 "U24" H 4550 5700 60  0000 C CNN
 F 1 "PCA9685PW" H 4250 3900 60  0000 C CNN
-F 2 "" H 4250 4800 60  0001 C CNN
+F 2 "Housings_SSOP:TSSOP-28_4.4x9.7mm_Pitch0.65mm" H 4250 4800 60  0001 C CNN
 F 3 "" H 4250 4800 60  0000 C CNN
 	1    4250 4800
