File: hardware/colibri-v2/wnd_usb_otg_to_cortex_usb_fs2.sch (KiCad schematic (older format))
At the start: 14 parts, among them Q14 PDTA123JU, U15 NTZD3155C

Commit message: Assigned footprints
Parts:
- U15: footprint (none) -> Sigmadrone:SOT-563_NTZD3155C
Changed lines of the file:
@@
 F 0 "U15" H 6100 3150 60  0000 C CNN
 F 1 "NTZD3155C" H 5900 2050 60  0000 C CNN
-F 2 "" H 5900 2600 60  0001 C CNN
+F 2 "Sigmadrone:SOT-563_NTZD3155C" H 5900 2600 60  0001 C CNN
 F 3 "" H 5900 2600 60  0000 C CNN
 	1    5900 2600

Commit message: Added AP6681GMT-HF-3.kicad_mod. Fixed netlist errors
Parts:
- DL10: footprint LEDs:LED-0603 -> LEDs:LED_0603
Changed lines of the file:
@@
 F 0 "DL10" H 7050 4100 50  0000 C CNN
 F 1 "GREEN" H 7050 3900 50  0000 C CNN
-F 2 "LEDs:LED-0603" H 7050 3850 30  0001 C CNN
+F 2 "LEDs:LED_0603" H 7050 3850 30  0001 C CNN
 F 3 "" H 7050 4000 60  0000 C CNN
 F 4 "0603" H 6935 3980 30  0000 C CNN "SMT"
