File: hardware/esc-power/esc-power.sch (KiCad schematic (older format))
At the start: 9 parts, among them P1 CONN_01X02, P2 CONN_01X02, P3 CONN_01X02, P4 CONN_01X02, P5 CONN_01X02, P6 CONN_01X02, P7 CONN_01X02, P8 CONN_01X02, P9 CONN_01X02

Commit message: Using components with 5mm pitch
Parts:
- P1, P2, P3, P4, P5, P6, P7, P8: footprint Terminal_Blocks:TerminalBlock_Pheonix_PT-3.5mm_2pol -> Sigmadrone:WURTH_691131710002; Provider (none) -> WURTH 691131710002
- P9: Provider (none) -> WURTH 691219610002; Provider2 (none) -> Mouser 651-1773976
Changed lines of the file:
@@
 F 2 "Sigmadrone:WURTH_691219610002" H 2700 1900 50  0001 C CNN
 F 3 "" H 2700 1900 50  0000 C CNN
+F 4 "WURTH 691219610002" H 2700 1900 60  0001 C CNN "Provider"
+F 5 "Mouser 651-1773976" H 2700 1900 60  0001 C CNN "Provider2"
 	1    2700 1900
 	1    0    0    -1
@@
 F 0 "P1" H 3200 2050 50  0000 C CNN
 F 1 "CONN_01X02" V 3300 1900 50  0000 C CNN
-F 2 "Terminal_Blocks:TerminalBlock_Pheonix_PT-3.5mm_2pol" H 3200 1900 50  0001 C CNN
+F 2 "Sigmadrone:WURTH_691131710002" H 3200 1900 50  0001 C CNN
 F 3 "" H 3200 1900 50  0000 C CNN
+F 4 "WURTH 691131710002" H 3200 1900 60  0001 C CNN "Provider"
 	1    3200 1900
 	1    0    0    -1
@@
 F 0 "P2" H 3700 2050 50  0000 C CNN
 F 1 "CONN_01X02" V 3800 1900 50  0000 C CNN
-F 2 "Terminal_Blocks:TerminalBlock_Pheonix_PT-3.5mm_2pol" H 3700 1900 50  0001 C CNN
+F 2 "Sigmadrone:WURTH_691131710002" H 3700 1900 50  0001 C CNN
 F 3 "" H 3700 1900 50  0000 C CNN
+F 4 "WURTH 691131710002" H 3700 1900 60  0001 C CNN "Provider"
 	1    3700 1900
 	1    0    0    -1
@@
 F 0 "P3" H 4250 2050 50  0000 C CNN
 F 1 "CONN_01X02" V 4350 1900 50  0000 C CNN
-F 2 "Terminal_Blocks:TerminalBlock_Pheonix_PT-3.5mm_2pol" H 4250 1900 50  0001 C CNN
+F 2 "Sigmadrone:WURTH_691131710002" H 4250 1900 50  0001 C CNN
 F 3 "" H 4250 1900 50  0000 C CNN
+F 4 "WURTH 691131710002" H 4250 1900 60  0001 C CNN "Provider"
 	1    4250 1900
 	1    0    0    -1
@@
 F 0 "P4" H 4750 2050 50  0000 C CNN
 F 1 "CONN_01X02" V 4850 1900 50  0000 C CNN
-F 2 "Terminal_Blocks:TerminalBlock_Pheonix_PT-3.5mm_2pol" H 4750 1900 50  0001 C CNN
+F 2 "Sigmadrone:WURTH_691131710002" H 4750 1900 50  0001 C CNN
 F 3 "" H 4750 1900 50  0000 C CNN
+F 4 "WURTH 691131710002" H 4750 1900 60  0001 C CNN "Provider"
 	1    4750 1900
 	1    0    0    -1
@@
 F 0 "P5" H 5200 2050 50  0000 C CNN
 F 1 "CONN_01X02" V 5300 1900 50  0000 C CNN
-F 2 "Terminal_Blocks:TerminalBlock_Pheonix_PT-3.5mm_2pol" H 5200 1900 50  0001 C CNN
+F 2 "Sigmadrone:WURTH_691131710002" H 5200 1900 50  0001 C CNN
 F 3 "" H 5200 1900 50  0000 C CNN
+F 4 "WURTH 691131710002" H 5200 1900 60  0001 C CNN "Provider"
 	1    5200 1900
 	1    0    0    -1
@@
 F 0 "P6" H 5650 2050 50  0000 C CNN
 F 1 "CONN_01X02" V 5750 1900 50  0000 C CNN
-F 2 "Terminal_Blocks:TerminalBlock_Pheonix_PT-3.5mm_2pol" H 5650 1900 50  0001 C CNN
+F 2 "Sigmadrone:WURTH_691131710002" H 5650 1900 50  0001 C CNN
 F 3 "" H 5650 1900 50  0000 C CNN
+F 4 "WURTH 691131710002" H 5650 1900 60  0001 C CNN "Provider"
 	1    5650 1900
 	1    0    0    -1
@@
 F 0 "P7" H 6150 2050 50  0000 C CNN
 F 1 "CONN_01X02" V 6250 1900 50  0000 C CNN
-F 2 "Terminal_Blocks:TerminalBlock_Pheonix_PT-3.5mm_2pol" H 6150 1900 50  0001 C CNN
+F 2 "Sigmadrone:WURTH_691131710002" H 6150 1900 50  0001 C CNN
 F 3 "" H 6150 1900 50  0000 C CNN
+F 4 "WURTH 691131710002" H 6150 1900 60  0001 C CNN "Provider"
 	1    6150 1900
 	1    0    0    -1
@@
 F 0 "P8" H 6650 2050 50  0000 C CNN
 F 1 "CONN_01X02" V 6750 1900 50  0000 C CNN
-F 2 "Terminal_Blocks:TerminalBlock_Pheonix_PT-3.5mm_2pol" H 6650 1900 50  0001 C CNN
+F 2 "Sigmadrone:WURTH_691131710002" H 6650 1900 50  0001 C CNN
 F 3 "" H 6650 1900 50  0000 C CNN
+F 4 "WURTH 691131710002" H 6650 1900 60  0001 C CNN "Provider"
 	1    6650 1900
 	1    0    0    -1
